File: teensy/eagle/BrushedBoard2/HackflightBrushed.brd (EAGLE design)
At the start: 33 x 48.3 mm, 12 parts, among them M1 53047-0210, M2 53047-0210, M3 53047-0210, M4 53047-0210

Commit message: Redesigned board
Parts:
- moved M3 5.08 mm to (11.4, 74.9)
- moved M4 5.08 mm to (11.4, 33.0)
- moved M1 5.08 mm to (26.7, 74.9)
- moved M2 5.08 mm to (26.7, 33.0)
Connections:
- removed net M1+: MTOP.3
- removed net M2+: MBOT.3
- removed net M3+: MTOP.2
- removed net M4+: MBOT.2
- removed net N$2: TNSBOT.4
- removed net N$3: TNSBOT.3
- removed net N$5: TNSBOT.1
- net 5VREG: now also TNSBOT.1; no longer TNSBOT.5
- net VBAT: now also MTOP.2; no longer TNSRGT.14
Routing:
- net GND: track 58.4 -> 0.00 mm
- net RX1: track 40.9 -> 66.2 mm
- net M2-: track 33.5 -> 27.8 mm
- net 3.3V: track 38.5 -> 42.1 mm
- net 5VREG: track 10.3 -> 7.39 mm
- net M1-: track 19.1 -> 21.4 mm
- net VBAT: track 95.3 -> 97.0 mm
- net M4-: track 29.0 -> 27.5 mm
- net M3-: track 19.7 -> 21.0 mm
- added copper zone on layer 1, net GND
Other:
- board size 33 x 48.3 mm -> 22.9 x 49.5 mm

Commit message: More board work
Parts:
- removed TNSBOT: (no value), SparkFun-Connectors:1X05
Connections:
- net 5VREG: now also TNSRGT.14; no longer TNSBOT.1
Routing:
- net 5VREG: track 7.39 -> 31.2 mm
Changed lines of the file:
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@@
 <element name="TNSLFT" library="SparkFun-Connectors" package="1X14" value="" x="11.43" y="36.83" rot="R90"/>
 <element name="TNSRGT" library="SparkFun-Connectors" package="1X14" value="" x="26.67" y="36.83" rot="R90"/>
-<element name="TNSBOT" library="SparkFun-Connectors" package="1X05" value="" x="13.97" y="36.83"/>
 </elements>
 <signals>
@@
 <signal name="5VREG">
 <contactref element="POLOLU" pad="3"/>
-<contactref element="TNSBOT" pad="1"/>
-<wire x1="14.1732" y1="40.6908" x2="14.1732" y2="37.0332" width="0.254" layer="16"/>
-<wire x1="16.4592" y1="42.9768" x2="14.1732" y2="40.6908" width="0.254" layer="16"/>
-<wire x1="14.1732" y1="37.0332" x2="13.97" y2="36.83" width="0.254" layer="16"/>
-<wire x1="16.4592" y1="42.9768" x2="16.51" y2="43.18" width="0.254" layer="16"/>
+<contactref element="TNSRGT" pad="14"/>
+<wire x1="16.6878" y1="43.6626" x2="16.6878" y2="43.2054" width="0.254" layer="1"/>
+<wire x1="17.145" y1="44.1198" x2="16.6878" y2="43.6626" width="0.254" layer="1"/>
+<wire x1="17.145" y1="44.3484" x2="17.145" y2="44.1198" width="0.254" layer="1"/>
+<wire x1="24.6888" y1="51.8922" x2="17.145" y2="44.3484" width="0.254" layer="1"/>
+<wire x1="24.6888" y1="68.1228" x2="24.6888" y2="51.8922" width="0.254" layer="1"/>
+<wire x1="26.5176" y1="69.9516" x2="24.6888" y2="68.1228" width="0.254" layer="1"/>
+<wire x1="16.6878" y1="43.2054" x2="16.51" y2="43.18" width="0.254" layer="1"/>
+<wire x1="26.5176" y1="69.9516" x2="26.67" y2="69.85" width="0.254" layer="1"/>
 </signal>
 <signal name="M4-">
