File: teensy/eagle/BrushedBoard2/HackflightBrushed.sch (EAGLE design)
At the start: 12 parts, among them M1 53047-0210, M2 53047-0210, M3 53047-0210, M4 53047-0210

Commit message: Redesigned board
Connections:
- removed net M1+: MTOP.3
- removed net M2+: MBOT.3
- removed net M3+: MTOP.2
- removed net M4+: MBOT.2
- removed net N$2: TNSBOT.4
- removed net N$3: TNSBOT.3
- removed net N$5: TNSBOT.1
- net 5VREG: now also TNSBOT.1; no longer TNSBOT.5
- net VBAT: now also MTOP.2; no longer TNSRGT.14
Changed lines of the file:
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@@
-</segment>
-<segment>
-<pinref part="TNSRGT" gate="G$1" pin="14"/>
-<wire x1="81.28" y1="63.5" x2="86.36" y2="63.5" width="0.1524" layer="91"/>
-<label x="81.28" y="63.5" size="1.778" layer="95"/>
 </segment>
 <segment>
@@
 <pinref part="M1" gate="G$1" pin="1"/>
 <wire x1="111.76" y1="7.62" x2="109.22" y2="7.62" width="0.1524" layer="91"/>
+<label x="106.68" y="7.62" size="1.778" layer="95"/>
+</segment>
+<segment>
+<pinref part="MTOP" gate="G$1" pin="2"/>
+<wire x1="22.86" y1="25.4" x2="27.94" y2="25.4" width="0.1524" layer="91"/>
+<label x="22.86" y="25.4" size="1.778" layer="95"/>
 </segment>
 </net>
@@
 <wire x1="58.42" y1="60.96" x2="66.04" y2="60.96" width="0.1524" layer="91"/>
 <label x="58.42" y="60.96" size="1.778" layer="95"/>
-</segment>
-</net>
-<net name="M3+" class="0">
-<segment>
-<pinref part="MTOP" gate="G$1" pin="2"/>
-<wire x1="22.86" y1="25.4" x2="27.94" y2="25.4" width="0.1524" layer="91"/>
-<label x="22.86" y="25.4" size="1.778" layer="95"/>
-</segment>
-</net>
-<net name="M4+" class="0">
-<segment>
-<pinref part="MBOT" gate="G$1" pin="2"/>
-<wire x1="22.86" y1="7.62" x2="27.94" y2="7.62" width="0.1524" layer="91"/>
-<label x="22.86" y="7.62" size="1.778" layer="95"/>
-</segment>
-</net>
-<net name="M2+" class="0">
-<segment>
-<pinref part="MBOT" gate="G$1" pin="3"/>
-<wire x1="22.86" y1="10.16" x2="27.94" y2="10.16" width="0.1524" layer="91"/>
-<label x="22.86" y="10.16" size="1.778" layer="95"/>
-</segment>
-</net>
-<net name="M1+" class="0">
-<segment>
-<pinref part="MTOP" gate="G$1" pin="3"/>
-<wire x1="22.86" y1="27.94" x2="27.94" y2="27.94" width="0.1524" layer="91"/>
-<label x="22.86" y="27.94" size="1.778" layer="95"/>
 </segment>
 </net>
@@
 </segment>
 <segment>
-<pinref part="TNSBOT" gate="G$1" pin="5"/>
-<wire x1="68.58" y1="20.32" x2="73.66" y2="20.32" width="0.1524" layer="91"/>
-<label x="68.58" y="20.32" size="1.778" layer="95"/>
+<pinref part="TNSBOT" gate="G$1" pin="1"/>
+<wire x1="68.58" y1="10.16" x2="73.66" y2="10.16" width="0.1524" layer="91"/>
+<label x="68.58" y="10.16" size="1.778" layer="95"/>
 </segment>
 </net>
@@
 </segment>
 </net>
-<net name="N$2" class="0">
-<segment>
-<pinref part="TNSBOT" gate="G$1" pin="4"/>
-<wire x1="68.58" y1="17.78" x2="73.66" y2="17.78" width="0.1524" layer="91"/>
-</segment>
-</net>
-<net name="N$3" class="0">
-<segment>
-<pinref part="TNSBOT" gate="G$1" pin="3"/>
-<wire x1="68.58" y1="15.24" x2="73.66" y2="15.24" width="0.1524" layer="91"/>
-</segment>
-</net>
-<net name="N$4" class="0">
-<segment>
-<wire x1="66.04" y1="12.7" x2="73.66" y2="12.7" width="0.1524" layer="91"/>
-</segment>
-</net>
-<net name="N$5" class="0">
-<segment>
-<pinref part="TNSBOT" gate="G$1" pin="1"/>
-<wire x1="68.58" y1="10.16" x2="73.66" y2="10.16" width="0.1524" layer="91"/>
-</segment>
-</net>

Commit message: More board work
Parts:
- removed TNSBOT: (no value), SparkFun-Connectors:CONN_05
Connections:
- net 5VREG: now also TNSRGT.14; no longer TNSBOT.1
Changed lines of the file:
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@@
 <part name="TNSRGT" library="SparkFun-Connectors" deviceset="CONN_14" device=""/>
 <part name="TNSLFT" library="SparkFun-Connectors" deviceset="CONN_14" device=""/>
-<part name="TNSBOT" library="SparkFun-Connectors" deviceset="CONN_05" device=""/>
 </parts>
 <sheets>
@@
 <instance part="TNSRGT" gate="G$1" x="71.12" y="48.26"/>
 <instance part="TNSLFT" gate="G$1" x="48.26" y="48.26"/>
-<instance part="TNSBOT" gate="G$1" x="60.96" y="15.24"/>
 </instances>
 <busses>
@@
 </segment>
 <segment>
-<pinref part="TNSBOT" gate="G$1" pin="1"/>
-<wire x1="68.58" y1="10.16" x2="73.66" y2="10.16" width="0.1524" layer="91"/>
-<label x="68.58" y="10.16" size="1.778" layer="95"/>
+<pinref part="TNSRGT" gate="G$1" pin="14"/>
+<wire x1="81.28" y1="63.5" x2="86.36" y2="63.5" width="0.1524" layer="91"/>
+<label x="81.28" y="63.5" size="1.778" layer="95"/>
 </segment>
 </net>
