File: extras/eagle-cad/loiterboard/loiterboard.sch (EAGLE design)
At the start: 5 parts

Commit message: Worked on Loiterboard
Parts:
- removed PMLFT, PMRGT: (no value), SparkFun-Connectors:CONN_04
- removed PWPWR: (no value), SparkFun-Connectors:CONN_02
- removed VLLFT, VLRGT2: (no value), SparkFun-Connectors:CONN_03
- added J1, J2: (no value), SparkFun-Connectors:CONN_041X04_NO_SILK
- added J3, J4: (no value), SparkFun-Connectors:CONN_031X03_NO_SILK
Connections:
- removed net 3.3V: PWPWR.1, VLLFT.1
- removed net A1/SCK: PMRGT.4
- removed net D10/CS: PMLFT.2
- removed net D4/MISO: PMLFT.4
- removed net D5/MOSI: PMLFT.3
- new net 3V3: J3.1
- new net CS: J1.2
- new net MISO: J1.4
- new net MOSI: J1.3
- new net SCK: J2.4
- net GND: now also J3.2; no longer PWPWR.2, VLLFT.2
- net INT: now also J3.3; no longer VLLFT.3
- net SCL: now also J4.2; no longer VLRGT2.2
- net SDA: now also J4.1; no longer VLRGT2.1
Changed lines of the file:
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@@
 <?xml version="1.0" encoding="utf-8"?>
 <!DOCTYPE eagle SYSTEM "eagle.dtd">
-<eagle version="9.1.1">
+<eagle version="9.6.2">
 <drawing>
 <settings>
@@
 <layer number="115" name="ReferenceISLANDS" color="7" fill="1" visible="yes" active="yes"/>
 <layer number="116" name="Patch_BOT" color="9" fill="4" visible="yes" active="yes"/>
+<layer number="117" name="PM_Ref" color="7" fill="1" visible="no" active="no"/>
 <layer number="118" name="Rect_Pads" color="7" fill="1" visible="yes" active="yes"/>
+<layer number="119" name="PF_Ref" color="7" fill="1" visible="no" active="no"/>
+<layer number="120" name="WFL_Ref" color="7" fill="1" visible="no" active="no"/>
 <layer number="121" name="_tsilk" color="7" fill="1" visible="yes" active="yes"/>
 <layer number="122" name="_bsilk" color="7" fill="1" visible="yes" active="yes"/>
@@
 </classes>
 <parts>
-<part name="VLLFT" library="SparkFun-Connectors" library_urn="urn:adsk.eagle:library:513" deviceset="CONN_03" device="" package3d_urn="urn:adsk.eagle:package:38063/1"/>
-<part name="VLRGT2" library="SparkFun-Connectors" library_urn="urn:adsk.eagle:library:513" deviceset="CONN_03" device="" package3d_urn="urn:adsk.eagle:package:38063/1"/>
-<part name="PMLFT" library="SparkFun-Connectors" library_urn="urn:adsk.eagle:library:513" deviceset="CONN_04" device="" package3d_urn="urn:adsk.eagle:package:38085/1"/>
-<part name="PMRGT" library="SparkFun-Connectors" library_urn="urn:adsk.eagle:library:513" deviceset="CONN_04" device="" package3d_urn="urn:adsk.eagle:package:38085/1"/>
-<part name="PWPWR" library="SparkFun-Connectors" library_urn="urn:adsk.eagle:library:513" deviceset="CONN_02" device="" package3d_urn="urn:adsk.eagle:package:38039/1"/>
+<part name="J1" library="SparkFun-Connectors" deviceset="CONN_04" device="1X04_NO_SILK"/>
+<part name="J2" library="SparkFun-Connectors" deviceset="CONN_04" device="1X04_NO_SILK"/>
+<part name="J3" library="SparkFun-Connectors" deviceset="CONN_03" device="1X03_NO_SILK"/>
+<part name="J4" library="SparkFun-Connectors" deviceset="CONN_03" device="1X03_NO_SILK"/>
 </parts>
 <sheets>
@@
 </plain>
 <instances>
-<instance part="VLLFT" gate="J$1" x="27.94" y="86.36"/>
-<instance part="VLRGT2" gate="J$1" x="48.26" y="86.36"/>
-<instance part="PMLFT" gate="G$1" x="30.48" y="58.42"/>
-<instance part="PMRGT" gate="G$1" x="55.88" y="58.42"/>
-<instance part="PWPWR" gate="G$1" x="40.64" y="71.12"/>
+<instance part="J1" gate="J1" x="-15.24" y="111.76" smashed="yes">
+<attribute name="VALUE" x="-20.32" y="104.394" size="1.778" layer="96" font="vector"/>
+</instance>
+<instance part="J2" gate="J1" x="20.32" y="111.76" smashed="yes">
+<attribute name="VALUE" x="15.24" y="104.394" size="1.778" layer="96" font="vector"/>
+</instance>
+<instance part="J3" gate="J$1" x="-17.78" y="93.98" smashed="yes">
+<attribute name="VALUE" x="-20.32" y="86.614" size="1.778" layer="96" font="vector"/>
+</instance>
+<instance part="J4" gate="J$1" x="17.78" y="93.98" smashed="yes">
+<attribute name="VALUE" x="15.24" y="86.614" size="1.778" layer="96" font="vector"/>
+</instance>
 </instances>
 <busses>
 </busses>
 <nets>
-<net name="A1/SCK" class="0">
-<segment>
-<pinref part="PMRGT" gate="G$1" pin="4"/>
-<wire x1="60.96" y1="63.5" x2="58.42" y2="63.5" width="0.1524" layer="91"/>
-<label x="60.96" y="63.5" size="1.778" layer="95"/>
-</segment>
-</net>
 <net name="GND" class="0">
 <segment>
-<pinref part="VLLFT" gate="J$1" pin="2"/>
-<wire x1="35.56" y1="86.36" x2="38.1" y2="86.36" width="0.1524" layer="91"/>
-<label x="35.56" y="86.36" size="1.778" layer="95"/>
-</segment>
-<segment>
-<pinref part="PWPWR" gate="G$1" pin="2"/>
-<wire x1="48.26" y1="73.66" x2="50.8" y2="73.66" width="0.1524" layer="91"/>
-<label x="48.26" y="73.66" size="1.778" layer="95"/>
-</segment>
-</net>
-<net name="3.3V" class="0">
-<segment>
-<pinref part="VLLFT" gate="J$1" pin="1"/>
-<wire x1="35.56" y1="83.82" x2="38.1" y2="83.82" width="0.1524" layer="91"/>
-<label x="35.56" y="83.82" size="1.778" layer="95"/>
-</segment>
-<segment>
-<pinref part="PWPWR" gate="G$1" pin="1"/>
-<wire x1="48.26" y1="71.12" x2="50.8" y2="71.12" width="0.1524" layer="91"/>
-<label x="48.26" y="71.12" size="1.778" layer="95"/>
+<pinref part="J3" gate="J$1" pin="2"/>
+<wire x1="-10.16" y1="93.98" x2="-5.08" y2="93.98" width="0.1524" layer="91"/>
+<label x="-10.16" y="93.98" size="1.778" layer="95"/>
 </segment>
 </net>
 <net name="SDA" class="0">
 <segment>
-<pinref part="VLRGT2" gate="J$1" pin="1"/>
-<wire x1="55.88" y1="83.82" x2="58.42" y2="83.82" width="0.1524" layer="91"/>
-<label x="55.88" y="83.82" size="1.778" layer="95"/>
+<pinref part="J4" gate="J$1" pin="1"/>
+<wire x1="25.4" y1="91.44" x2="30.48" y2="91.44" width="0.1524" layer="91"/>
+<label x="25.4" y="91.44" size="1.778" layer="95"/>
 </segment>
 </net>
 <net name="SCL" class="0">
 <segment>
-<pinref part="VLRGT2" gate="J$1" pin="2"/>
-<wire x1="55.88" y1="86.36" x2="58.42" y2="86.36" width="0.1524" layer="91"/>
-<label x="55.88" y="86.36" size="1.778" layer="95"/>
+<pinref part="J4" gate="J$1" pin="2"/>
+<wire x1="25.4" y1="93.98" x2="30.48" y2="93.98" width="0.1524" layer="91"/>
+<label x="25.4" y="93.98" size="1.778" layer="95"/>
 </segment>
 </net>
 <net name="INT" class="0">
 <segment>
-<pinref part="VLLFT" gate="J$1" pin="3"/>
-<wire x1="35.56" y1="88.9" x2="38.1" y2="88.9" width="0.1524" layer="91"/>
-<label x="35.56" y="88.9" size="1.778" layer="95"/>
-</segment>
-</net>
-<net name="D5/MOSI" class="0">
-<segment>
-<pinref part="PMLFT" gate="G$1" pin="3"/>
-<wire x1="35.56" y1="60.96" x2="38.1" y2="60.96" width="0.1524" layer="91"/>
-<label x="35.56" y="60.96" size="1.778" layer="95"/>
-</segment>
-</net>
-<net name="D4/MISO" class="0">
-<segment>
-<pinref part="PMLFT" gate="G$1" pin="4"/>
-<wire x1="35.56" y1="63.5" x2="38.1" y2="63.5" width="0.1524" layer="91"/>
-<label x="35.56" y="63.5" size="1.778" layer="95"/>
-</segment>
-</net>
-<net name="D10/CS" class="0">
-<segment>
-<pinref part="PMLFT" gate="G$1" pin="2"/>
-<wire x1="35.56" y1="58.42" x2="38.1" y2="58.42" width="0.1524" layer="91"/>
-<label x="35.56" y="58.42" size="1.778" layer="95"/>
+<pinref part="J3" gate="J$1" pin="3"/>
+<wire x1="-10.16" y1="96.52" x2="-5.08" y2="96.52" width="0.1524" layer="91"/>
+<label x="-10.16" y="96.52" size="1.778" layer="95"/>
+</segment>
+</net>
+<net name="MISO" class="0">
+<segment>
+<pinref part="J1" gate="J1" pin="4"/>
+<wire x1="-10.16" y1="116.84" x2="-5.08" y2="116.84" width="0.1524" layer="91"/>
+<label x="-10.16" y="116.84" size="1.778" layer="95"/>
+</segment>
+</net>
+<net name="MOSI" class="0">
+<segment>
+<pinref part="J1" gate="J1" pin="3"/>
+<wire x1="-10.16" y1="114.3" x2="-5.08" y2="114.3" width="0.1524" layer="91"/>
+<label x="-10.16" y="114.3" size="1.778" layer="95"/>
+</segment>
+</net>
+<net name="CS" class="0">
+<segment>
+<pinref part="J1" gate="J1" pin="2"/>
+<wire x1="-10.16" y1="111.76" x2="-5.08" y2="111.76" width="0.1524" layer="91"/>
+<label x="-10.16" y="111.76" size="1.778" layer="95"/>
+</segment>
+</net>
+<net name="SCK" class="0">
+<segment>
+<pinref part="J2" gate="J1" pin="4"/>
+<wire x1="25.4" y1="116.84" x2="30.48" y2="116.84" width="0.1524" layer="91"/>
+<label x="25.4" y="116.84" size="1.778" layer="95"/>
+</segment>
+</net>
+<net name="3V3" class="0">
+<segment>
+<pinref part="J3" gate="J$1" pin="1"/>
+<wire x1="-10.16" y1="91.44" x2="-5.08" y2="91.44" width="0.1524" layer="91"/>
+<label x="-10.16" y="91.44" size="1.778" layer="95"/>
 </segment>
 </net>
@@
 </schematic>
 </drawing>
-<compatibility>
-<note version="8.2" severity="warning">
-Since Version 8.2, EAGLE supports online libraries. The ids
-of those online libraries will not be understood (or retained)
-with this version.
-</note>
-<note version="8.3" severity="warning">
-Since Version 8.3, EAGLE supports URNs for individual library
-assets (packages, symbols, and devices). The URNs of those assets
-will not be understood (or retained) with this version.
-</note>
-<note version="8.3" severity="warning">
-Since Version 8.3, EAGLE supports the association of 3D packages
-with devices in libraries, schematics, and board files. Those 3D
-packages will not be understood (or retained) with this version.
-</note>
-</compatibility>
 </eagle>
