File: cad/combo/combo.sch (EAGLE design)
At the start: 5 parts

Commit message: modified:   cad/combo/combo.brd
Parts:
- added PMW1, PMW2: (no value), SparkFun-Connectors:CONN_041X04_NO_SILK
- added PMW3: (no value), SparkFun-Connectors:CONN_021X02_NO_SILK
- added VL1, VL2: (no value), SparkFun-Connectors:CONN_031X03_NO_SILK
Connections:
- new net EN: PMW1.2
- new net INT: VL2.3
- new net LED: PMW2.4
- new net MOSI: PMW2.2
- new net MOT: PMW1.3
- new net RST: PMW1.4
- new net SCK: PMW1.1
- net 3V3: now also PMW3.1, VL2.1
- net CS: now also PMW2.3
- net GND: now also PMW3.2, VL2.2
- net MISO: now also PMW2.1
- net SCL: now also VL1.2
- net SDA: now also VL1.1
Changed lines of the file:
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@@
 <part name="U$2" library="headers(2mm)" deviceset="1X6" device=""/>
 <part name="U$5" library="headers(2mm)" deviceset="1X3" device=""/>
+<part name="VL1" library="SparkFun-Connectors" deviceset="CONN_03" device="1X03_NO_SILK"/>
+<part name="VL2" library="SparkFun-Connectors" deviceset="CONN_03" device="1X03_NO_SILK"/>
+<part name="PMW1" library="SparkFun-Connectors" deviceset="CONN_04" device="1X04_NO_SILK"/>
+<part name="PMW2" library="SparkFun-Connectors" deviceset="CONN_04" device="1X04_NO_SILK"/>
+<part name="PMW3" library="SparkFun-Connectors" deviceset="CONN_02" device="1X02_NO_SILK"/>
 </parts>
 <sheets>
@@
 <instance part="U$2" gate="G$1" x="7.62" y="-5.08"/>
 <instance part="U$5" gate="G$1" x="48.26" y="88.9"/>
+<instance part="VL1" gate="J$1" x="-40.64" y="86.36"/>
+<instance part="VL2" gate="J$1" x="-40.64" y="66.04"/>
+<instance part="PMW1" gate="J1" x="-58.42" y="33.02"/>
+<instance part="PMW2" gate="J1" x="-58.42" y="15.24"/>
+<instance part="PMW3" gate="G$1" x="-60.96" y="-2.54"/>
 </instances>
 <busses>
@@
 <label x="53.34" y="88.9" size="1.778" layer="95"/>
 </segment>
+<segment>
+<pinref part="VL2" gate="J$1" pin="1"/>
+<wire x1="-33.02" y1="63.5" x2="-27.94" y2="63.5" width="0.1524" layer="91"/>
+<label x="-33.02" y="63.5" size="1.778" layer="95"/>
+</segment>
+<segment>
+<pinref part="PMW3" gate="G$1" pin="1"/>
+<wire x1="-53.34" y1="-2.54" x2="-48.26" y2="-2.54" width="0.1524" layer="91"/>
+<label x="-53.34" y="-2.54" size="1.778" layer="95"/>
+</segment>
 </net>
 <net name="GND" class="0">
@@
 <label x="73.66" y="2.54" size="1.778" layer="95"/>
 </segment>
+<segment>
+<pinref part="VL2" gate="J$1" pin="2"/>
+<wire x1="-33.02" y1="66.04" x2="-27.94" y2="66.04" width="0.1524" layer="91"/>
+<label x="-33.02" y="66.04" size="1.778" layer="95"/>
+</segment>
+<segment>
+<pinref part="PMW3" gate="G$1" pin="2"/>
+<wire x1="-53.34" y1="0" x2="-48.26" y2="0" width="0.1524" layer="91"/>
+<label x="-53.34" y="0" size="1.778" layer="95"/>
+</segment>
 </net>
 <net name="SDA" class="0">
@@
 <label x="93.98" y="43.18" size="1.778" layer="95"/>
 </segment>
+<segment>
+<pinref part="VL1" gate="J$1" pin="1"/>
+<wire x1="-33.02" y1="83.82" x2="-27.94" y2="83.82" width="0.1524" layer="91"/>
+<label x="-33.02" y="83.82" size="1.778" layer="95"/>
+</segment>
 </net>
 <net name="SCL" class="0">
@@
 <label x="93.98" y="45.72" size="1.778" layer="95"/>
 </segment>
+<segment>
+<pinref part="VL1" gate="J$1" pin="2"/>
+<wire x1="-33.02" y1="86.36" x2="-27.94" y2="86.36" width="0.1524" layer="91"/>
+<label x="-33.02" y="86.36" size="1.778" layer="95"/>
+</segment>
 </net>
 <net name="5V" class="0">
@@
 <label x="48.26" y="60.96" size="1.778" layer="95"/>
 </segment>
+<segment>
+<pinref part="PMW2" gate="J1" pin="3"/>
+<wire x1="-53.34" y1="17.78" x2="-48.26" y2="17.78" width="0.1524" layer="91"/>
+<label x="-53.34" y="17.78" size="1.778" layer="95"/>
+</segment>
 </net>
 <net name="MISO" class="0">
@@
 <label x="48.26" y="58.42" size="1.778" layer="95"/>
 </segment>
+<segment>
+<pinref part="PMW2" gate="J1" pin="1"/>
+<wire x1="-48.26" y1="12.7" x2="-53.34" y2="12.7" width="0.1524" layer="91"/>
+<label x="-53.34" y="12.7" size="1.778" layer="95"/>
+</segment>
 </net>
 <net name="RX" class="0">
@@
 </segment>
 </net>
+<net name="INT" class="0">
+<segment>
+<pinref part="VL2" gate="J$1" pin="3"/>
+<wire x1="-33.02" y1="68.58" x2="-27.94" y2="68.58" width="0.1524" layer="91"/>
+<label x="-33.02" y="68.58" size="1.778" layer="95"/>
+</segment>
+</net>
+<net name="MOSI" class="0">
+<segment>
+<pinref part="PMW2" gate="J1" pin="2"/>
+<wire x1="-53.34" y1="15.24" x2="-48.26" y2="15.24" width="0.1524" layer="91"/>
+<label x="-53.34" y="15.24" size="1.778" layer="95"/>
+</segment>
+</net>
+<net name="LED" class="0">
+<segment>
+<pinref part="PMW2" gate="J1" pin="4"/>
+<wire x1="-53.34" y1="20.32" x2="-48.26" y2="20.32" width="0.1524" layer="91"/>
+<label x="-53.34" y="20.32" size="1.778" layer="95"/>
+</segment>
+</net>
+<net name="SCK" class="0">
+<segment>
+<pinref part="PMW1" gate="J1" pin="1"/>
+<wire x1="-53.34" y1="30.48" x2="-48.26" y2="30.48" width="0.1524" layer="91"/>
+<label x="-53.34" y="30.48" size="1.778" layer="95"/>
+</segment>
+</net>
+<net name="EN" class="0">
+<segment>
+<pinref part="PMW1" gate="J1" pin="2"/>
+<wire x1="-53.34" y1="33.02" x2="-48.26" y2="33.02" width="0.1524" layer="91"/>
+<label x="-53.34" y="33.02" size="1.778" layer="95"/>
+</segment>
+</net>
+<net name="MOT" class="0">
+<segment>
+<pinref part="PMW1" gate="J1" pin="3"/>
+<wire x1="-53.34" y1="35.56" x2="-48.26" y2="35.56" width="0.1524" layer="91"/>
+<label x="-53.34" y="35.56" size="1.778" layer="95"/>
+</segment>
+</net>
+<net name="RST" class="0">
+<segment>
+<pinref part="PMW1" gate="J1" pin="4"/>
+<wire x1="-53.34" y1="38.1" x2="-48.26" y2="38.1" width="0.1524" layer="91"/>
+<label x="-53.34" y="38.1" size="1.778" layer="95"/>
+</segment>
+</net>

Commit message: modified:   cad/combo/combo.brd
Parts:
- added SPI2: 1X2, headers(2mm):1X2
Connections:
- net MOSI: now also SPI2.1
- net SCK: now also SPI2.2
Changed lines of the file:
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@@
 <part name="PMW2" library="SparkFun-Connectors" deviceset="CONN_04" device="1X04_NO_SILK"/>
 <part name="PMW3" library="SparkFun-Connectors" deviceset="CONN_02" device="1X02_NO_SILK"/>
+<part name="SPI2" library="headers(2mm)" deviceset="1X2" device=""/>
 </parts>
 <sheets>
@@
 <instance part="PMW2" gate="J1" x="-58.42" y="15.24"/>
 <instance part="PMW3" gate="G$1" x="-60.96" y="-2.54"/>
+<instance part="SPI2" gate="G$1" x="-60.96" y="-22.86" smashed="yes">
+<attribute name="NAME" x="-63.5" y="-19.685" size="1.27" layer="95" font="vector"/>
+</instance>
 </instances>
 <busses>
@@
 <label x="-53.34" y="15.24" size="1.778" layer="95"/>
 </segment>
+<segment>
+<pinref part="SPI2" gate="G$1" pin="1"/>
+<wire x1="-58.42" y1="-22.86" x2="-53.34" y2="-22.86" width="0.1524" layer="91"/>
+<label x="-55.88" y="-22.86" size="1.778" layer="95"/>
+</segment>
 </net>
 <net name="LED" class="0">
@@
 <label x="-53.34" y="30.48" size="1.778" layer="95"/>
 </segment>
-</net>
+<segment>
+<pinref part="SPI2" gate="G$1" pin="2"/>
+<wire x1="-58.42" y1="-25.4" x2="-53.34" y2="-25.4" width="0.1524" layer="91"/>
+<label x="-55.88" y="-25.4" size="1.778" layer="95"/>
+</segment>
+</net>

Commit message: modified:   cad/combo/combo.brd
Connections:
- net M1: now also U$1.5; no longer U$1.2
- net M2: now also U$1.4; no longer U$1.3
- net M3: now also U$1.3; no longer U$1.4
- net M4: now also U$1.2; no longer U$1.5
Changed lines of the file:
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@@
 </segment>
 <segment>
-<pinref part="U$1" gate="G$1" pin="5"/>
-<wire x1="53.34" y1="48.26" x2="48.26" y2="48.26" width="0.1524" layer="91"/>
-<label x="48.26" y="48.26" size="1.778" layer="95"/>
+<pinref part="U$1" gate="G$1" pin="2"/>
+<wire x1="53.34" y1="55.88" x2="48.26" y2="55.88" width="0.1524" layer="91"/>
+<label x="48.26" y="55.88" size="1.778" layer="95"/>
 </segment>
 </net>
@@
 </segment>
 <segment>
-<pinref part="U$1" gate="G$1" pin="2"/>
-<wire x1="53.34" y1="55.88" x2="48.26" y2="55.88" width="0.1524" layer="91"/>
-<label x="48.26" y="55.88" size="1.778" layer="95"/>
+<pinref part="U$1" gate="G$1" pin="5"/>
+<wire x1="53.34" y1="48.26" x2="48.26" y2="48.26" width="0.1524" layer="91"/>
+<label x="48.26" y="48.26" size="1.778" layer="95"/>
 </segment>
 </net>
@@
 </segment>
 <segment>
-<pinref part="U$1" gate="G$1" pin="3"/>
-<wire x1="53.34" y1="53.34" x2="48.26" y2="53.34" width="0.1524" layer="91"/>
-<label x="48.26" y="53.34" size="1.778" layer="95"/>
+<pinref part="U$1" gate="G$1" pin="4"/>
+<wire x1="53.34" y1="50.8" x2="48.26" y2="50.8" width="0.1524" layer="91"/>
+<label x="48.26" y="50.8" size="1.778" layer="95"/>
 </segment>
 </net>
@@
 </segment>
 <segment>
-<pinref part="U$1" gate="G$1" pin="4"/>
-<wire x1="53.34" y1="50.8" x2="48.26" y2="50.8" width="0.1524" layer="91"/>
-<label x="48.26" y="50.8" size="1.778" layer="95"/>
+<pinref part="U$1" gate="G$1" pin="3"/>
+<wire x1="53.34" y1="53.34" x2="48.26" y2="53.34" width="0.1524" layer="91"/>
+<label x="48.26" y="53.34" size="1.778" layer="95"/>
 </segment>
 </net>

Commit message: modified:   cad/combo/combo.brd
Parts:
- removed SPI2: 1X2, headers(2mm):1X2
- added U$3, U$4, U$6, U$7: 1X1, headers(2mm):1X1
Connections:
- new net G2: U$1.GND, U$7.1
- new net LED_R_IN: U$1.0/RX1, U$3.1
- new net LED_R_OUT: U$4.1, U$6.1
- net CS: now also U$1.10/CS; no longer U$1.0/RX1
- net GND: no longer U$1.GND
- net MISO: now also U$1.12/MISO; no longer U$1.1/TX1
- net MOSI: now also U$1.11/MOSI; no longer SPI2.1
- net SCK: now also U$1.13/SCK; no longer SPI2.2

Commit message: modified:   cad/combo/combo.brd
Parts:
- removed U$2: 1X6, headers(2mm):1X6
- added J1: BM06B-SRSS-TB, SparkFun-Connectors:JST_6_PIN_HORIZONTAL
Connections:
- net GND: now also J1A.6; no longer U$2.1
- net M1: now also J1A.1, U$1.3; no longer U$1.5, U$2.6
- net M2: now also J1A.2; no longer U$2.5
- net M3: now also J1A.3, U$1.5; no longer U$1.3, U$2.4
- net M4: now also J1A.4, U$1.6; no longer U$1.2, U$2.3
- net VBAT: now also J1A.5; no longer U$2.2
Changed lines of the file:
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@@
 <?xml version="1.0" encoding="utf-8"?>
 <!DOCTYPE eagle SYSTEM "eagle.dtd">
-<eagle version="9.1.1">
+<eagle version="9.6.2">
 <drawing>
 <settings>
@@
 <part name="MPU6050" library="SparkFun-Connectors" deviceset="CONN_05" device="NO_SILK"/>
 <part name="REG" library="SparkFun-Connectors" deviceset="CONN_04" device="1X04_NO_SILK"/>
-<part name="U$2" library="headers(2mm)" deviceset="1X6" device=""/>
 <part name="U$5" library="headers(2mm)" deviceset="1X3" device=""/>
 <part name="VL1" library="SparkFun-Connectors" deviceset="CONN_03" device="1X03_NO_SILK"/>
@@
 <part name="U$6" library="headers(2mm)" deviceset="1X1" device=""/>
 <part name="U$7" library="headers(2mm)" deviceset="1X1" device=""/>
+<part name="J1" library="SparkFun-Connectors" deviceset="JST_6_PIN_HORIZONTAL" device="" value="BM06B-SRSS-TB"/>
 </parts>
 <sheets>
@@
 <attribute name="NAME" x="2.54" y="28.448" size="1.778" layer="95" font="vector"/>
 </instance>
-<instance part="REG" gate="J1" x="7.62" y="50.8"/>
-<instance part="U$2" gate="G$1" x="7.62" y="-5.08"/>
-<instance part="U$5" gate="G$1" x="48.26" y="88.9"/>
-<instance part="VL1" gate="J$1" x="-40.64" y="86.36"/>
-<instance part="VL2" gate="J$1" x="-40.64" y="66.04"/>
-<instance part="PMW1" gate="J1" x="-58.42" y="33.02"/>
-<instance part="PMW2" gate="J1" x="-58.42" y="15.24"/>
-<instance part="PMW3" gate="G$1" x="-60.96" y="-2.54"/>
+<instance part="REG" gate="J1" x="7.62" y="50.8" smashed="yes">
+<attribute name="VALUE" x="2.54" y="43.434" size="1.778" layer="96" font="vector"/>
+<attribute name="NAME" x="2.54" y="58.928" size="1.778" layer="95" font="vector"/>
+</instance>
+<instance part="U$5" gate="G$1" x="48.26" y="88.9" smashed="yes">
+<attribute name="NAME" x="45.72" y="94.615" size="1.27" layer="95" font="vector"/>
+<attribute name="VALUE" x="45.72" y="81.915" size="1.27" layer="96" font="vector"/>
+</instance>
+<instance part="VL1" gate="J$1" x="-40.64" y="86.36" smashed="yes">
+<attribute name="VALUE" x="-43.18" y="78.994" size="1.778" layer="96" font="vector"/>
+<attribute name="NAME" x="-43.18" y="91.948" size="1.778" layer="95" font="vector"/>
+</instance>
+<instance part="VL2" gate="J$1" x="-40.64" y="66.04" smashed="yes">
+<attribute name="VALUE" x="-43.18" y="58.674" size="1.778" layer="96" font="vector"/>
+<attribute name="NAME" x="-43.18" y="71.628" size="1.778" layer="95" font="vector"/>
+</instance>
+<instance part="PMW1" gate="J1" x="-58.42" y="33.02" smashed="yes">
+<attribute name="VALUE" x="-63.5" y="25.654" size="1.778" layer="96" font="vector"/>
+<attribute name="NAME" x="-63.5" y="41.148" size="1.778" layer="95" font="vector"/>
+</instance>
+<instance part="PMW2" gate="J1" x="-58.42" y="15.24" smashed="yes">
+<attribute name="VALUE" x="-63.5" y="7.874" size="1.778" layer="96" font="vector"/>
+<attribute name="NAME" x="-63.5" y="23.368" size="1.778" layer="95" font="vector"/>
+</instance>
+<instance part="PMW3" gate="G$1" x="-60.96" y="-2.54" smashed="yes">
+<attribute name="VALUE" x="-63.5" y="-7.366" size="1.778" layer="96" font="vector"/>
+<attribute name="NAME" x="-63.5" y="3.048" size="1.778" layer="95" font="vector"/>
+</instance>
 <instance part="U$3" gate="G$1" x="-27.94" y="25.4" smashed="yes"/>
 <instance part="U$4" gate="G$1" x="-27.94" y="17.78" smashed="yes"/>
 <instance part="U$6" gate="G$1" x="-27.94" y="-2.54" smashed="yes"/>
 <instance part="U$7" gate="G$1" x="-27.94" y="-10.16" smashed="yes"/>
+<instance part="J1" gate="A" x="0" y="83.82" smashed="yes">
+<attribute name="VALUE" x="-5.08" y="73.914" size="1.778" layer="96" font="vector"/>
+<attribute name="NAME" x="-5.08" y="94.488" size="1.778" layer="95" font="vector"/>
+</instance>
 </instances>
 <busses>
@@
 </segment>
 <segment>
-<pinref part="U$2" gate="G$1" pin="1"/>
-<wire x1="10.16" y1="2.54" x2="15.24" y2="2.54" width="0.1524" layer="91"/>
-<label x="12.7" y="2.54" size="1.778" layer="95"/>
-</segment>
-<segment>
 <pinref part="U$5" gate="G$1" pin="1"/>
 <wire x1="50.8" y1="91.44" x2="55.88" y2="91.44" width="0.1524" layer="91"/>
@@
 <label x="-53.34" y="0" size="1.778" layer="95"/>
 </segment>
+<segment>
+<pinref part="J1" gate="A" pin="6"/>
+<wire x1="5.08" y1="91.44" x2="10.16" y2="91.44" width="0.1524" layer="91"/>
+<label x="5.08" y="91.44" size="1.778" layer="95"/>
+</segment>
 </net>
 <net name="SDA" class="0">
@@
 <net name="M4" class="0">
 <segment>
-<pinref part="U$2" gate="G$1" pin="3"/>
-<wire x1="10.16" y1="-2.54" x2="15.24" y2="-2.54" width="0.1524" layer="91"/>
-<label x="12.7" y="-2.54" size="1.778" layer="95"/>
-</segment>
-<segment>
-<pinref part="U$1" gate="G$1" pin="2"/>
-<wire x1="53.34" y1="55.88" x2="48.26" y2="55.88" width="0.1524" layer="91"/>
-<label x="48.26" y="55.88" size="1.778" layer="95"/>
+<pinref part="J1" gate="A" pin="4"/>
+<wire x1="5.08" y1="86.36" x2="10.16" y2="86.36" width="0.1524" layer="91"/>
+<label x="5.08" y="86.36" size="1.778" layer="95"/>
+</segment>
+<segment>
+<pinref part="U$1" gate="G$1" pin="6"/>
+<wire x1="53.34" y1="45.72" x2="48.26" y2="45.72" width="0.1524" layer="91"/>
+<label x="48.26" y="45.72" size="1.778" layer="95"/>
 </segment>
 </net>
 <net name="M1" class="0">
 <segment>
-<pinref part="U$2" gate="G$1" pin="6"/>
-<wire x1="10.16" y1="-10.16" x2="15.24" y2="-10.16" width="0.1524" layer="91"/>
-<label x="12.7" y="-10.16" size="1.778" layer="95"/>
+<pinref part="J1" gate="A" pin="1"/>
+<wire x1="5.08" y1="78.74" x2="10.16" y2="78.74" width="0.1524" layer="91"/>
+<label x="5.08" y="78.74" size="1.778" layer="95"/>
+</segment>
+<segment>
+<pinref part="U$1" gate="G$1" pin="3"/>
+<wire x1="53.34" y1="53.34" x2="48.26" y2="53.34" width="0.1524" layer="91"/>
+<label x="48.26" y="53.34" size="1.778" layer="95"/>
+</segment>
+</net>
+<net name="M2" class="0">
+<segment>
+<pinref part="J1" gate="A" pin="2"/>
+<wire x1="5.08" y1="81.28" x2="10.16" y2="81.28" width="0.1524" layer="91"/>
+<label x="5.08" y="81.28" size="1.778" layer="95"/>
+</segment>
+<segment>
+<pinref part="U$1" gate="G$1" pin="4"/>
+<wire x1="53.34" y1="50.8" x2="48.26" y2="50.8" width="0.1524" layer="91"/>
+<label x="48.26" y="50.8" size="1.778" layer="95"/>
+</segment>
+</net>
+<net name="M3" class="0">
+<segment>
+<pinref part="J1" gate="A" pin="3"/>
+<wire x1="5.08" y1="83.82" x2="10.16" y2="83.82" width="0.1524" layer="91"/>
+<label x="5.08" y="83.82" size="1.778" layer="95"/>
 </segment>
 <segment>
@@
 </segment>
 </net>
-<net name="M2" class="0">
-<segment>
-<pinref part="U$2" gate="G$1" pin="5"/>
-<wire x1="10.16" y1="-7.62" x2="15.24" y2="-7.62" width="0.1524" layer="91"/>
-<label x="12.7" y="-7.62" size="1.778" layer="95"/>
-</segment>
-<segment>
-<pinref part="U$1" gate="G$1" pin="4"/>
-<wire x1="53.34" y1="50.8" x2="48.26" y2="50.8" width="0.1524" layer="91"/>
-<label x="48.26" y="50.8" size="1.778" layer="95"/>
-</segment>
-</net>
-<net name="M3" class="0">
-<segment>
-<pinref part="U$2" gate="G$1" pin="4"/>
-<wire x1="10.16" y1="-5.08" x2="15.24" y2="-5.08" width="0.1524" layer="91"/>
-<label x="12.7" y="-5.08" size="1.778" layer="95"/>
-</segment>
-<segment>
-<pinref part="U$1" gate="G$1" pin="3"/>
-<wire x1="53.34" y1="53.34" x2="48.26" y2="53.34" width="0.1524" layer="91"/>
-<label x="48.26" y="53.34" size="1.778" layer="95"/>
-</segment>
-</net>
 <net name="VBAT" class="0">
 <segment>
@@
 </segment>
 <segment>
-<pinref part="U$2" gate="G$1" pin="2"/>
-<wire x1="10.16" y1="0" x2="15.24" y2="0" width="0.1524" layer="91"/>
-<label x="12.7" y="0" size="1.778" layer="95"/>
-</segment>
-</net>
+<pinref part="J1" gate="A" pin="5"/>
+<wire x1="5.08" y1="88.9" x2="10.16" y2="88.9" width="0.1524" layer="91"/>
+<label x="5.08" y="88.9" size="1.778" layer="95"/>
+</segment>
+</net>
