File: cad/combo/combo.sch (EAGLE design)
At the start: 14 parts, among them J1 BM06B-SRSS-TB

Commit message: modified:   cad/combo/combo.brd
Parts:
- removed J1: BM06B-SRSS-TB, SparkFun-Connectors:JST_6_PIN_HORIZONTAL
- added GND, M1, M2, M3, M4, VBAT: (no value), wirepad:SMD2
Connections:
- net GND: now also GND.P; no longer J1A.6
- net M1: now also M1.P, U$1.6; no longer J1A.1, U$1.3
- net M2: now also M2.P, U$1.5; no longer J1A.2, U$1.4
- net M3: now also M3.P, U$1.4; no longer J1A.3, U$1.5
- net M4: now also M4.P, U$1.3; no longer J1A.4, U$1.6
- net VBAT: now also VBAT.P; no longer J1A.5
Changed lines of the file:
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@@
 <?xml version="1.0" encoding="utf-8"?>
 <!DOCTYPE eagle SYSTEM "eagle.dtd">
-<eagle version="9.6.2">
+<eagle version="9.1.1">
 <drawing>
 <settings>
@@
 <part name="U$6" library="headers(2mm)" deviceset="1X1" device=""/>
 <part name="U$7" library="headers(2mm)" deviceset="1X1" device=""/>
-<part name="J1" library="SparkFun-Connectors" deviceset="JST_6_PIN_HORIZONTAL" device="" value="BM06B-SRSS-TB"/>
+<part name="GND" library="wirepad" deviceset="SMD2" device=""/>
+<part name="VBAT" library="wirepad" deviceset="SMD2" device=""/>
+<part name="M4" library="wirepad" deviceset="SMD2" device=""/>
+<part name="M3" library="wirepad" deviceset="SMD2" device=""/>
+<part name="M2" library="wirepad" deviceset="SMD2" device=""/>
+<part name="M1" library="wirepad" deviceset="SMD2" device=""/>
 </parts>
 <sheets>
@@
 <instance part="U$6" gate="G$1" x="-27.94" y="-2.54" smashed="yes"/>
 <instance part="U$7" gate="G$1" x="-27.94" y="-10.16" smashed="yes"/>
-<instance part="J1" gate="A" x="0" y="83.82" smashed="yes">
-<attribute name="VALUE" x="-5.08" y="73.914" size="1.778" layer="96" font="vector"/>
-<attribute name="NAME" x="-5.08" y="94.488" size="1.778" layer="95" font="vector"/>
+<instance part="GND" gate="1" x="2.54" y="114.3" smashed="yes">
+<attribute name="VALUE" x="1.397" y="110.998" size="1.778" layer="96"/>
+</instance>
+<instance part="VBAT" gate="1" x="2.54" y="109.22" smashed="yes">
+<attribute name="VALUE" x="1.397" y="105.918" size="1.778" layer="96"/>
+</instance>
+<instance part="M4" gate="1" x="2.54" y="104.14" smashed="yes">
+<attribute name="VALUE" x="1.397" y="100.838" size="1.778" layer="96"/>
+</instance>
+<instance part="M3" gate="1" x="2.54" y="99.06" smashed="yes">
+<attribute name="VALUE" x="1.397" y="95.758" size="1.778" layer="96"/>
+</instance>
+<instance part="M2" gate="1" x="2.54" y="93.98" smashed="yes">
+<attribute name="VALUE" x="1.397" y="90.678" size="1.778" layer="96"/>
+</instance>
+<instance part="M1" gate="1" x="2.54" y="88.9" smashed="yes">
+<attribute name="VALUE" x="1.397" y="85.598" size="1.778" layer="96"/>
 </instance>
 </instances>
@@
 </segment>
 <segment>
-<pinref part="J1" gate="A" pin="6"/>
-<wire x1="5.08" y1="91.44" x2="10.16" y2="91.44" width="0.1524" layer="91"/>
-<label x="5.08" y="91.44" size="1.778" layer="95"/>
+<pinref part="GND" gate="1" pin="P"/>
+<wire x1="5.08" y1="114.3" x2="10.16" y2="114.3" width="0.1524" layer="91"/>
+<label x="5.08" y="114.3" size="1.778" layer="95"/>
 </segment>
 </net>
@@
 <net name="M4" class="0">
 <segment>
-<pinref part="J1" gate="A" pin="4"/>
-<wire x1="5.08" y1="86.36" x2="10.16" y2="86.36" width="0.1524" layer="91"/>
-<label x="5.08" y="86.36" size="1.778" layer="95"/>
+<pinref part="M4" gate="1" pin="P"/>
+<wire x1="5.08" y1="104.14" x2="10.16" y2="104.14" width="0.1524" layer="91"/>
+<label x="5.08" y="104.14" size="1.778" layer="95"/>
+</segment>
+<segment>
+<pinref part="U$1" gate="G$1" pin="3"/>
+<wire x1="53.34" y1="53.34" x2="48.26" y2="53.34" width="0.1524" layer="91"/>
+<label x="48.26" y="53.34" size="1.778" layer="95"/>
+</segment>
+</net>
+<net name="M1" class="0">
+<segment>
+<pinref part="M1" gate="1" pin="P"/>
+<wire x1="5.08" y1="88.9" x2="10.16" y2="88.9" width="0.1524" layer="91"/>
+<label x="5.08" y="88.9" size="1.778" layer="95"/>
 </segment>
 <segment>
@@
 </segment>
 </net>
-<net name="M1" class="0">
-<segment>
-<pinref part="J1" gate="A" pin="1"/>
-<wire x1="5.08" y1="78.74" x2="10.16" y2="78.74" width="0.1524" layer="91"/>
-<label x="5.08" y="78.74" size="1.778" layer="95"/>
-</segment>
-<segment>
-<pinref part="U$1" gate="G$1" pin="3"/>
-<wire x1="53.34" y1="53.34" x2="48.26" y2="53.34" width="0.1524" layer="91"/>
-<label x="48.26" y="53.34" size="1.778" layer="95"/>
-</segment>
-</net>
 <net name="M2" class="0">
 <segment>
-<pinref part="J1" gate="A" pin="2"/>
-<wire x1="5.08" y1="81.28" x2="10.16" y2="81.28" width="0.1524" layer="91"/>
-<label x="5.08" y="81.28" size="1.778" layer="95"/>
+<pinref part="M2" gate="1" pin="P"/>
+<wire x1="5.08" y1="93.98" x2="10.16" y2="93.98" width="0.1524" layer="91"/>
+<label x="5.08" y="93.98" size="1.778" layer="95"/>
+</segment>
+<segment>
+<pinref part="U$1" gate="G$1" pin="5"/>
+<wire x1="53.34" y1="48.26" x2="48.26" y2="48.26" width="0.1524" layer="91"/>
+<label x="48.26" y="48.26" size="1.778" layer="95"/>
+</segment>
+</net>
+<net name="M3" class="0">
+<segment>
+<pinref part="M3" gate="1" pin="P"/>
+<wire x1="5.08" y1="99.06" x2="10.16" y2="99.06" width="0.1524" layer="91"/>
+<label x="5.08" y="99.06" size="1.778" layer="95"/>
 </segment>
 <segment>
@@
 </segment>
 </net>
-<net name="M3" class="0">
-<segment>
-<pinref part="J1" gate="A" pin="3"/>
-<wire x1="5.08" y1="83.82" x2="10.16" y2="83.82" width="0.1524" layer="91"/>
-<label x="5.08" y="83.82" size="1.778" layer="95"/>
-</segment>
-<segment>
-<pinref part="U$1" gate="G$1" pin="5"/>
-<wire x1="53.34" y1="48.26" x2="48.26" y2="48.26" width="0.1524" layer="91"/>
-<label x="48.26" y="48.26" size="1.778" layer="95"/>
-</segment>
-</net>
 <net name="VBAT" class="0">
 <segment>
@@
 </segment>
 <segment>
-<pinref part="J1" gate="A" pin="5"/>
-<wire x1="5.08" y1="88.9" x2="10.16" y2="88.9" width="0.1524" layer="91"/>
-<label x="5.08" y="88.9" size="1.778" layer="95"/>
-</segment>
-</net>
+<pinref part="VBAT" gate="1" pin="P"/>
+<wire x1="5.08" y1="109.22" x2="10.16" y2="109.22" width="0.1524" layer="91"/>
+<label x="5.08" y="109.22" size="1.778" layer="95"/>
+</segment>
+</net>
