File: eagle/usfs/combo.sch (EAGLE design)
At the start: 21 parts

Commit message: modified:   eagle/usfs/combo.brd
Parts:
- added USFS1: (no value), SparkFun-Connectors:CONN_05NO_SILK
Connections:
- removed net EN: PMW1.2
- removed net INT: VL2.3
- removed net MOT: PMW1.3
- removed net RST: PMW1.4
Changed lines of the file:
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@@
 <?xml version="1.0" encoding="utf-8"?>
 <!DOCTYPE eagle SYSTEM "eagle.dtd">
-<eagle version="9.6.2">
+<eagle version="9.1.1">
 <drawing>
 <settings>
@@
 <part name="3V" library="wirepad" deviceset="SMD2" device=""/>
 <part name="RX" library="wirepad" deviceset="SMD2" device=""/>
+<part name="USFS1" library="SparkFun-Connectors" deviceset="CONN_05" device="NO_SILK"/>
 </parts>
 <sheets>
@@
 <attribute name="VALUE" x="75.057" y="80.518" size="1.778" layer="96"/>
 </instance>
+<instance part="USFS1" gate="G$1" x="25.4" y="20.32" smashed="yes">
+<attribute name="VALUE" x="22.86" y="10.414" size="1.778" layer="96" font="vector"/>
+<attribute name="NAME" x="22.86" y="28.448" size="1.778" layer="95" font="vector"/>
+</instance>
 </instances>
 <busses>
@@
 </segment>
 </net>
-<net name="INT" class="0">
-<segment>
-<pinref part="VL2" gate="J$1" pin="3"/>
-<wire x1="-33.02" y1="68.58" x2="-27.94" y2="68.58" width="0.1524" layer="91"/>
-<label x="-33.02" y="68.58" size="1.778" layer="95"/>
-</segment>
-</net>
 <net name="MOSI" class="0">
 <segment>
@@
 </segment>
 </net>
-<net name="EN" class="0">
-<segment>
-<pinref part="PMW1" gate="J1" pin="2"/>
-<wire x1="-53.34" y1="33.02" x2="-48.26" y2="33.02" width="0.1524" layer="91"/>
-<label x="-53.34" y="33.02" size="1.778" layer="95"/>
-</segment>
-</net>
-<net name="MOT" class="0">
-<segment>
-<pinref part="PMW1" gate="J1" pin="3"/>
-<wire x1="-53.34" y1="35.56" x2="-48.26" y2="35.56" width="0.1524" layer="91"/>
-<label x="-53.34" y="35.56" size="1.778" layer="95"/>
-</segment>
-</net>
-<net name="RST" class="0">
-<segment>
-<pinref part="PMW1" gate="J1" pin="4"/>
-<wire x1="-53.34" y1="38.1" x2="-48.26" y2="38.1" width="0.1524" layer="91"/>
-<label x="-53.34" y="38.1" size="1.778" layer="95"/>
-</segment>
-</net>
