File: eagle/mpu6050/combo.brd (EAGLE design)
At the start: 35.8 x 76.9 mm, 21 parts

Commit message: modified:   eagle/mpu6050/combo.brd
Parts:
- moved PMW3 2.80 mm to (21.5, 64.5), turned to 0 degrees
Routing:
- net GND: track 106.9 -> 83.5 mm
- net 3V3: track 92.9 -> 83.8 mm
Changed lines of the file:
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@@
 <?xml version="1.0" encoding="utf-8"?>
 <!DOCTYPE eagle SYSTEM "eagle.dtd">
-<eagle version="9.1.1">
+<eagle version="9.6.2">
 <drawing>
 <settings>
@@
 <text x="33" y="59.4858" size="0.8128" layer="25">CS</text>
 <text x="33" y="64.1858" size="0.8128" layer="25">SO</text>
-<text x="23.7" y="65.771775" size="0.8128" layer="25">3V3</text>
-<text x="21.1" y="65.871775" size="0.8128" layer="25">GD</text>
+<text x="20.6" y="65.771775" size="0.8128" layer="25">3V3</text>
+<text x="23.5" y="65.771775" size="0.8128" layer="25">GD</text>
 <text x="12.9858" y="64.1858" size="0.8128" layer="25">SCK</text>
 <text x="33" y="61.7858" size="0.8128" layer="25">SI</text>
@@
 <attribute name="VALUE" x="29.568" y="65.77" size="0.6096" layer="27" font="vector" ratio="20" rot="R270"/>
 </element>
-<element name="PMW3" library="SparkFun-Connectors" package="1X02_NO_SILK" value="" x="24.3" y="64.5" smashed="yes" rot="R180">
-<attribute name="VALUE" x="25.57" y="66.532" size="0.6096" layer="27" font="vector" ratio="20" rot="R180"/>
+<element name="PMW3" library="SparkFun-Connectors" package="1X02_NO_SILK" value="" x="21.5" y="64.5" smashed="yes">
+<attribute name="VALUE" x="20.23" y="62.468" size="0.6096" layer="27" font="vector" ratio="20"/>
 </element>
 <element name="U$3" library="headers(2mm)" package="1X1" value="1X1" x="36" y="50.40281875" smashed="yes"/>
@@
 <wire x1="14" y1="65.5" x2="16.4" y2="67.5" width="0.3048" layer="1"/>
 <wire x1="7.9304" y1="41.56" x2="11.7286" y2="45.3582" width="0.3048" layer="1"/>
-<wire x1="16.4" y1="67.5" x2="18.1554" y2="65.7446" width="0.3048" layer="1"/>
-<wire x1="23.52013125" y1="64.5" x2="24.3" y2="64.5" width="0.3048" layer="1"/>
-<wire x1="18.1554" y1="65.7446" x2="22.27553125" y2="65.7446" width="0.3048" layer="1"/>
-<wire x1="22.27553125" y1="65.7446" x2="23.52013125" y2="64.5" width="0.3048" layer="1"/>
 <contactref element="3V" pad="1"/>
 <wire x1="13.8114" y1="30.9686375" x2="13.7" y2="30.8572375" width="0.3048" layer="1"/>
@@
 <wire x1="34.5627625" y1="31.4" x2="33.5213625" y2="30.3586" width="0.3048" layer="1"/>
 <wire x1="33.5213625" y1="30.3586" x2="26.3586" y2="30.3586" width="0.3048" layer="1"/>
-<wire x1="13.7" y1="30.8572375" x2="19" y2="23" width="0" layer="19" extent="1-1"/>
+<wire x1="16.4" y1="67.5" x2="21.5" y2="64.5" width="0" layer="19" extent="1-1"/>
 <wire x1="15.4" y1="11" x2="14.9" y2="10.8" width="0" layer="19" extent="1-1"/>
+<wire x1="19" y1="23" x2="15.4" y2="11" width="0" layer="19" extent="1-1"/>
 </signal>
 <signal name="GND">
@@
 <wire x1="9.1886" y1="51.6" x2="13.4" y2="67.9" width="0.3048" layer="16"/>
 <wire x1="13.4" y1="67.9" x2="16.4" y2="70.04" width="0.3048" layer="16"/>
-<wire x1="16.4" y1="70.04" x2="21.76" y2="64.5" width="0.3048" layer="16"/>
 <contactref element="GND" pad="1"/>
 <wire x1="38.17" y1="31.4" x2="31.7" y2="37.87" width="0.3048" layer="1"/>
@@
 <wire x1="38.17" y1="31.4" x2="27.23" y2="20.46" width="0.3048" layer="1"/>
 <wire x1="27.23" y1="20.46" x2="19" y2="20.46" width="0.3048" layer="1"/>
-<wire x1="21.76" y1="64.5" x2="24.96" y2="61.3" width="0.3048" layer="1"/>
-<wire x1="24.96" y1="61.3" x2="24.96" y2="50.2" width="0.3048" layer="1"/>
+<wire x1="16.4" y1="70.04" x2="24.04" y2="64.5" width="0" layer="19" extent="1-1"/>
+<wire x1="24.96" y1="50.2" x2="24.04" y2="64.5" width="0" layer="19" extent="1-1"/>
+<wire x1="29.5" y1="40.2" x2="24.96" y2="50.2" width="0" layer="19" extent="16-16"/>
+<wire x1="15.4" y1="9" x2="16.1" y2="8.7" width="0" layer="19" extent="1-1"/>
 </signal>
 <signal name="SDA">

Commit message: modified:   eagle/mpu6050/combo.brd
Parts:
- moved MPU6050 15.8 mm to (31.2, 12.9), turned to 90 degrees
- moved PMW1 15.2 mm to (31.6, 64.5)
- moved PMW2 15.2 mm to (16.4, 64.5)
Routing:
- net GND: track 83.5 -> 109.3 mm, vias 1 -> 2
- net 3V3: track 83.8 -> 106.9 mm
- net MISO: track 33.8 -> 21.5 mm
- net CS: track 25.8 -> 14.3 mm
- net MOSI: track 29.1 -> 17.7 mm
- net SCK: track 37.7 -> 42.5 mm, vias 1 -> 0
- net SCL: track 65.9 -> 62.5 mm
- net SDA: track 59.8 -> 62.0 mm
