File: eagle/1s/1s.brd (EAGLE design)
At the start: 52.5 x 76.5 mm, 13 parts

Commit message: modified:   eagle/1s/1s.brd
Parts:
- added ESC1: 455-1750-1-ND, SparkFun-Connectors:1X03
- added PAD1, PAD2: (no value), wirepad:SMD2,54-5,08
- moved J_REG_5V_1 4.30 mm to (34.4, 57.9)
Connections:
- removed net ESP_RX: U$1.7
- removed net SCL1: U$1.16/A2
- removed net SDA1: U$1.17/A3
- new net VBAT: ESC1.2, J_REG_5V_1.VIN, PAD1.1
- net 5V: now also J_REG_5V_1.VOUT
- net GND: now also ESC1.1, J_REG_5V_1.GND, PAD2.1
- net M1: now also ESC1.3, U$1.3/CANTX; no longer U$1.6
- net M2: now also U$1.4/CANRX; no longer U$1.5
- net M3: now also U$1.5; no longer U$1.4/CANRX
- net M4: now also U$1.6; no longer U$1.3/CANTX
Routing:
- net 3V3: track 41.7 -> 0.29 mm
- net 5V: track 37.0 -> 0.14 mm, vias 2 -> 0
- net GND: track 52.4 -> 21.5 mm
- net RX: track 26.8 -> 0.14 mm, vias 2 -> 0
- net SCL: track 20.6 -> 0.00 mm
- net SDA: track 17.1 -> 0.00 mm

Commit message: modified:   eagle/1s/1s.brd
Parts:
- added ESC2, ESC3, ESC4: 455-1750-1-ND, SparkFun-Connectors:1X03
- moved ESC1 9.02 mm to (51.5, 26.8), turned to 225 degrees
- moved U$3 2.27 mm to (41.3, 64.5)
- moved U$4 2.25 mm to (41.1, 72.8)
- moved MPU6050 1.90 mm to (41.6, 11.1)
- moved U$6 0.82 mm to (44.0, 69.2)
- moved U$7 0.54 mm to (44.9, 65.8)
Connections:
- net GND: now also ESC2.1, ESC3.1, ESC4.1
- net M2: now also ESC2.3
- net M3: now also ESC3.3
- net M4: now also ESC4.3
- net VBAT: now also ESC2.2, ESC3.2, ESC4.2
Routing:
- net GND: track 21.5 -> 0.64 mm
- net LED_R_IN: track 19.9 -> 0.00 mm
- net LED_R_OUT: track 5.80 -> 4.85 mm
Other:
- board size 52.5 x 76.5 mm -> 40.9 x 76.5 mm
- board text removed: "G"

Commit message: new file:   eagle/bottom/bottom.brd
Parts:
- removed FLOWDECK_1, FLOWDECK_2: 1X10, headers(2mm):1X10
- added J1, J2: (no value), SparkFun-Connectors:1X04_NO_SILK
- moved RX 5.71 mm to (27.1, 17.3)
- moved 3V3 5.71 mm to (27.1, 13.9)
- moved 5V 5.71 mm to (27.1, 15.6)
- moved GD 5.71 mm to (27.1, 12.2)
- moved MPU6050 1.40 mm to (43.0, 11.1)
Connections:
- net 3V3: now also J1.3; no longer FLOWDECK_1.1
- net CS: now also J2.4; no longer FLOWDECK_1.8
- net GND: now also J1.4; no longer FLOWDECK_1.10
- net MISO: now also J2.1; no longer FLOWDECK_2.4
- net MOSI: now also J2.2; no longer FLOWDECK_2.5
- net SCK: now also J2.3; no longer FLOWDECK_2.3
- net SCL: now also J1.2; no longer FLOWDECK_1.5
- net SDA: now also J1.1; no longer FLOWDECK_1.4
Routing:
- net SCK: track 0.73 -> 0.00 mm
Other:
- board text added: "SK"
- board text removed: "3V3"
- board text removed: "CL1"
- board text removed: "DA1"
- board text removed: "ESP_RX"
- board text removed: "GND"
- board text removed: "SCK"

Commit message: modified:   eagle/1s/1s.brd
Parts:
- removed PAD1, PAD2: (no value), wirepad:SMD2,54-5,08
- added +, -: (no value), wirepad:SMD2,54-5,08
- moved MPU6050 47.4 mm to (38.5, 58.3)
- moved J_REG_5V_1 40.4 mm to (34.5, 17.5)
- moved ESC4 6.72 mm to (21.3, 56.7), turned to 225 degrees
- moved ESC1 6.16 mm to (47.4, 22.2), turned to 45 degrees
- moved ESC3 2.12 mm to (18.0, 25.3)
- moved J1 1.00 mm to (31.0, 29.0)
- moved J2 1.00 mm to (31.0, 51.0)
- moved U$7 0.61 mm to (44.2, 65.9)
- moved U$4 0.59 mm to (41.4, 72.3)
- moved U$6 0.20 mm to (43.8, 69.2)
Connections:
- net GND: now also -.1; no longer PAD2.1
- net M1: now also U$1.23/A9; no longer U$1.3/CANTX
- net M3: now also U$1.15/A1; no longer U$1.5
- net VBAT: now also +.1; no longer PAD1.1
Routing:
- net GND: track 0.64 -> 159.7 mm, vias 0 -> 2
- net VBAT: track 0.00 -> 112.7 mm, vias 0 -> 2
- net 3V3: track 0.00 -> 73.6 mm, vias 0 -> 1
- net SDA: track 0.00 -> 50.9 mm, vias 0 -> 1
- net SCL: track 0.00 -> 50.8 mm, vias 0 -> 4
- net 5V: track 0.14 -> 45.7 mm, vias 0 -> 2
- net SCK: track 0.00 -> 36.9 mm
- net RX: track 0.14 -> 26.3 mm, vias 0 -> 3
- net LED_R_IN: track 0.00 -> 22.7 mm, vias 0 -> 2
- net M4: track 0.00 -> 18.5 mm, vias 0 -> 1
- net CS: track 0.00 -> 18.4 mm
- net MOSI: track 0.00 -> 18.1 mm
- net M2: track 0.00 -> 17.5 mm, vias 0 -> 1
- net M3: track 0.00 -> 14.3 mm
- net MISO: track 0.00 -> 14.2 mm
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Other:
- outline, holes or cut-outs redrawn
- board text added: "-"
