File: cad/biggity/biggity.brd (EAGLE design)
At the start: 94.1 x 88.7 mm, 12 parts

Commit message: modified:   cad/biggity/biggity.brd
Parts:
- removed J1, J2: (no value), SparkFun-Connectors:1X04_NO_SILK
- removed TP_1, TP_2: (no value), SparkFun-Connectors:1X10_NO_SILK
- added U$1: TEENSY_4.0, TEENSY 4.0:TEENSY_4.0
- renumbered J3 to REG, USFS to MPU6050
Connections:
- removed net CS: J2.4, TP_1.7
- removed net MISO: J2.1, TP_1.9
- removed net MOSI: J2.2, TP_1.10
- removed net RESET: TP_1.2
- removed net SCK: J2.3, TP_1.8
- net 3V3: now also MPU6050.1; no longer J1.3, MPU6050.4, TP_2.7
- net 5V: no longer TP_2.8
- net GND: now also MPU6050.2; no longer J1.4, MPU6050.5, TP_1.1, TP_2.9
- net M1: no longer TP_2.6
- net M2: no longer TP_2.5
- net M3: no longer TP_2.4
- net M4: no longer TP_2.3
- net SCL: now also MPU6050.4; no longer J1.2, MPU6050.2, TP_1.6
- net SDA: now also MPU6050.3; no longer J1.1, MPU6050.1, TP_1.5
Other:
- board text removed: "M1"
- board text removed: "M2"
- board text removed: "M3"
- board text removed: "M4"
- board text removed: "TinyPICO"
- board text removed: "USB"
Changed lines of the file:
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@@
 <hole x="48.6" y="15.9" drill="2.4"/>
 <hole x="58.9" y="16" drill="2.4"/>
-<text x="46.59185" y="57.791396875" size="1.016" layer="25">SK</text>
-<text x="48.660890625" y="57.78270625" size="1.016" layer="25">CL</text>
-<text x="41.73169375" y="57.7" size="1.016" layer="25">SI</text>
-<text x="43.958071875" y="57.682709375" size="1.016" layer="25">SO</text>
-<text x="50.7666" y="40.4" size="1.016" layer="25" rot="R180">DA</text>
 <wire x1="71.3" y1="63.3" x2="71.2" y2="41.2" width="0.1524" layer="20"/>
 <wire x1="43.6" y1="90.3" x2="63" y2="90.3" width="0.1524" layer="20"/>
@@
 <wire x1="43.6" y1="90.3" x2="40.9" y2="72.8" width="0.1524" layer="20"/>
 <wire x1="63" y1="90.2" x2="65.8" y2="72.8" width="0.1524" layer="20"/>
-<text x="49.1432" y="46.6048" size="1.016" layer="25">M1</text>
-<text x="49.1" y="64.9" size="1.016" layer="25">SO</text>
-<text x="51.8" y="64.9" size="1.016" layer="25">SI</text>
-<text x="54.1" y="64.9" size="1.016" layer="25">SK</text>
-<text x="56.6" y="64.9" size="1.016" layer="25">CS</text>
-<text x="53.3706" y="40.4" size="1.016" layer="25" rot="R180">CL</text>
-<text x="55.7738" y="40.5" size="1.016" layer="25" rot="R180">3V</text>
-<text x="58.5738" y="40.6" size="1.016" layer="25" rot="R180">GD</text>
-<text x="56.4738" y="40.6" size="1.016" layer="26" rot="MR180">GD</text>
+<text x="35.9" y="40.7" size="1.016" layer="25">SO</text>
+<text x="38.9" y="40.9" size="1.016" layer="25">SI</text>
+<text x="36.1" y="60.5" size="1.016" layer="25">SK</text>
+<text x="41.1" y="41" size="1.016" layer="25">CS</text>
 <wire x1="65.8" y1="72.8" x2="83.1" y2="87.3" width="0.1524" layer="20"/>
 <wire x1="71.3" y1="63.3" x2="89.5" y2="79" width="0.1524" layer="20"/>
@@
 <text x="47.3" y="21.6" size="1.016" layer="25">DA</text>
 <text x="47.4" y="24.3" size="1.016" layer="25">CL</text>
-<text x="39.195503125" y="55.793903125" size="1.778" layer="26" rot="SMR270">USB</text>
 <text x="60.4326" y="68.2508" size="1.016" layer="25" rot="R180">5V</text>
-<text x="58.795503125" y="52.293903125" size="1.778" layer="26" rot="SMR0">TinyPICO</text>
 <text x="57.695503125" y="70.193903125" size="1.778" layer="26" rot="SMR0">Reg</text>
-<text x="41.4432" y="46.6048" size="1.016" layer="25">GD</text>
-<text x="44.2432" y="46.6048" size="1.016" layer="25">5V</text>
-<text x="46.5432" y="46.6048" size="1.016" layer="25">3V</text>
-<text x="51.8432" y="46.7048" size="1.016" layer="25">M2</text>
-<text x="54.2432" y="46.7048" size="1.016" layer="25">M3</text>
-<text x="56.9432" y="46.8048" size="1.016" layer="25">M4</text>
-<text x="51.360890625" y="57.68270625" size="1.016" layer="25">DA</text>
 <text x="60.4326" y="70.9508" size="1.016" layer="25" rot="R180">GD</text>
+<text x="66.6" y="60.7" size="1.016" layer="25">GD</text>
+<text x="63.8" y="60.6" size="1.016" layer="25">3V</text>
+<text x="69.1" y="60.7" size="1.016" layer="25">5V</text>
+<text x="48.5" y="60.5" size="1.016" layer="25">DA</text>
+<text x="51.5" y="60.5" size="1.016" layer="25">CL</text>
 </plain>
 <attributes>
@@
 </autorouter>
 <elements>
-<element name="J1" library="SparkFun-Connectors" package="1X04_NO_SILK" value="" x="49.8" y="41.6" smashed="yes">
-<attribute name="PROD_ID" value="CONN-09696" x="49.8" y="41.6" size="1.778" layer="27" display="off"/>
-<attribute name="VALUE" x="48.53" y="39.568" size="0.6096" layer="27" font="vector" ratio="20"/>
-</element>
-<element name="J2" library="SparkFun-Connectors" package="1X04_NO_SILK" value="" x="49.8" y="63.6" smashed="yes">
-<attribute name="PROD_ID" value="CONN-09696" x="49.8" y="63.6" size="1.778" layer="27" display="off"/>
-<attribute name="VALUE" x="48.53" y="61.568" size="0.6096" layer="27" font="vector" ratio="20"/>
-</element>
-<element name="USFS" library="SparkFun-Connectors" package="1X05_NO_SILK" value="" x="46" y="22" smashed="yes" rot="R90">
+<element name="MPU6050" library="SparkFun-Connectors" package="1X05_NO_SILK" value="" x="46" y="22" smashed="yes" rot="R90">
 <attribute name="VALUE" x="48.032" y="20.73" size="0.6096" layer="27" font="vector" ratio="20" rot="R90"/>
 </element>
-<element name="J3" library="SparkFun-Connectors" package="1X04_NO_SILK" value="" x="61.8" y="68" smashed="yes" rot="R90">
+<element name="REG" library="SparkFun-Connectors" package="1X04_NO_SILK" value="" x="61.8" y="68" smashed="yes" rot="R90">
 <attribute name="PROD_ID" value="CONN-09696" x="61.8" y="68" size="1.778" layer="27" rot="R90" display="off"/>
 <attribute name="VALUE" x="63.832" y="66.73" size="0.6096" layer="27" font="vector" ratio="20" rot="R90"/>
 </element>
-<element name="TP_1" library="SparkFun-Connectors" package="1X10_NO_SILK" value="" x="62.5" y="60" rot="R180"/>
-<element name="TP_2" library="SparkFun-Connectors" package="1X10_NO_SILK" value="" x="62.5" y="45" rot="R180"/>
 <element name="GD" library="wirepad" package="SMD1,27-2,54" value="" x="46.9" y="81.6" rot="R180"/>
 <element name="VB" library="wirepad" package="SMD1,27-2,54" value="" x="49.4" y="81.6" rot="R180"/>
@@
 <element name="M3" library="wirepad" package="SMD1,27-2,54" value="" x="56.9" y="81.6" rot="R180"/>
 <element name="M4" library="wirepad" package="SMD1,27-2,54" value="" x="59.4" y="81.6" rot="R180"/>
+<element name="U$1" library="TEENSY 4.0" package="TEENSY_4.0" value="TEENSY_4.0" x="53.4" y="51.1" rot="SMR0"/>
 </elements>
 <signals>
 <signal name="3V3">
-<contactref element="J1" pad="3"/>
-<contactref element="USFS" pad="4"/>
-<contactref element="TP_2" pad="7"/>
-<wire x1="54.88" y1="41.6" x2="47.26" y2="45" width="0" layer="19" extent="1-1"/>
-<wire x1="46" y1="29.62" x2="54.88" y2="41.6" width="0" layer="19" extent="1-1"/>
+<contactref element="MPU6050" pad="1"/>
 </signal>
 <signal name="GND">
 <polygon width="0.3048" layer="1">
-<vertex x="83.65" y="90.456"/>
-<vertex x="83.65" y="13.65"/>
-<vertex x="23.6" y="13.65"/>
-<vertex x="23.6" y="90.456"/>
+<vertex x="71.15" y="90.456"/>
+<vertex x="71.15" y="13.65"/>
+<vertex x="35.5" y="13.65"/>
+<vertex x="35.5" y="90.456"/>
 </polygon>
-<contactref element="J1" pad="4"/>
-<contactref element="USFS" pad="5"/>
-<contactref element="J3" pad="2"/>
-<contactref element="TP_2" pad="9"/>
+<contactref element="REG" pad="2"/>
 <contactref element="GD" pad="1"/>
-<contactref element="TP_1" pad="1"/>
-<wire x1="61.8" y1="70.54" x2="46.9" y2="81.6" width="0" layer="19" extent="1-1"/>
-<wire x1="62.5" y1="60" x2="61.8" y2="70.54" width="0" layer="19" extent="1-1"/>
-<wire x1="57.42" y1="41.6" x2="62.5" y2="60" width="0" layer="19" extent="1-1"/>
-<wire x1="42.18" y1="45" x2="57.42" y2="41.6" width="0" layer="19" extent="1-1"/>
-<wire x1="46" y1="32.16" x2="42.18" y2="45" width="0" layer="19" extent="1-1"/>
+<contactref element="MPU6050" pad="2"/>
+<wire x1="46.9" y1="81.6" x2="61.8" y2="70.54" width="0" layer="19" extent="1-1"/>
+<wire x1="46" y1="24.54" x2="61.8" y2="70.54" width="0" layer="19" extent="1-1"/>
 </signal>
 <signal name="SDA">
-<contactref element="J1" pad="1"/>
-<contactref element="USFS" pad="1"/>
-<contactref element="TP_1" pad="5"/>
-<wire x1="49.8" y1="41.6" x2="52.34" y2="60" width="0" layer="19" extent="1-1"/>
-<wire x1="46" y1="22" x2="49.8" y2="41.6" width="0" layer="19" extent="1-1"/>
+<contactref element="MPU6050" pad="3"/>
 </signal>
 <signal name="SCL">
-<contactref element="J1" pad="2"/>
-<contactref element="USFS" pad="2"/>
-<contactref element="TP_1" pad="6"/>
-<wire x1="52.34" y1="41.6" x2="49.8" y2="60" width="0" layer="19" extent="1-1"/>
-<wire x1="46" y1="24.54" x2="52.34" y2="41.6" width="0" layer="19" extent="1-1"/>
+<contactref element="MPU6050" pad="4"/>
 </signal>
 <signal name="5V">
-<contactref element="J3" pad="1"/>
-<contactref element="TP_2" pad="8"/>
-<wire x1="44.72" y1="45" x2="61.8" y2="68" width="0" layer="19" extent="1-1"/>
-</signal>
-<signal name="CS">
-<contactref element="J2" pad="4"/>
-<contactref element="TP_1" pad="7"/>
-<wire x1="47.26" y1="60" x2="57.42" y2="63.6" width="0" layer="19" extent="1-1"/>
-</signal>
-<signal name="MISO">
-<contactref element="J2" pad="1"/>
-<contactref element="TP_1" pad="9"/>
-<wire x1="49.8" y1="63.6" x2="42.18" y2="60" width="0" layer="19" extent="1-1"/>
-</signal>
-<signal name="MOSI">
-<contactref element="J2" pad="2"/>
-<contactref element="TP_1" pad="10"/>
-<wire x1="52.34" y1="63.6" x2="39.64" y2="60" width="0" layer="19" extent="1-1"/>
-</signal>
-<signal name="SCK">
-<contactref element="J2" pad="3"/>
-<contactref element="TP_1" pad="8"/>
-<wire x1="44.72" y1="60" x2="54.88" y2="63.6" width="0" layer="19" extent="1-1"/>
+<contactref element="REG" pad="1"/>
 </signal>
 <signal name="VBAT">
-<contactref element="J3" pad="3"/>
+<contactref element="REG" pad="3"/>
 <contactref element="VB" pad="1"/>
 <wire x1="49.4" y1="81.6" x2="61.8" y2="73.08" width="0" layer="19" extent="1-1"/>
@@
 <signal name="M1">
 <contactref element="M1" pad="1"/>
-<contactref element="TP_2" pad="6"/>
-<wire x1="49.8" y1="45" x2="51.9" y2="81.6" width="0" layer="19" extent="1-1"/>
 </signal>
 <signal name="M2">
 <contactref element="M2" pad="1"/>
-<contactref element="TP_2" pad="5"/>
-<wire x1="52.34" y1="45" x2="54.4" y2="81.6" width="0" layer="19" extent="1-1"/>
 </signal>
 <signal name="M3">
 <contactref element="M3" pad="1"/>
-<contactref element="TP_2" pad="4"/>
-<wire x1="54.88" y1="45" x2="56.9" y2="81.6" width="0" layer="19" extent="1-1"/>
 </signal>
 <signal name="M4">
 <contactref element="M4" pad="1"/>
-<contactref element="TP_2" pad="3"/>
-<wire x1="57.42" y1="45" x2="59.4" y2="81.6" width="0" layer="19" extent="1-1"/>
-</signal>
-<signal name="RESET">
-<contactref element="TP_1" pad="2"/>
 </signal>
 </signals>
@@
 </board>
 </drawing>
+<compatibility>
+<note version="6.3" minversion="6.2.2" severity="warning">
+Since Version 6.2.2 text objects can contain more than one line,
+which will not be processed correctly with this version.
+</note>
+</compatibility>
 </eagle>
