File: kicad/teensypi_v91/teensypi_v91.kicad_sch (KiCad schematic)
At the start: 18 parts

Commit message: =More KiCAD PCB
Parts:
- added M2_center1, M3_center1, M4_center1: MountingHole, MountingHole:MountingHole_5.5mm, symbol Mechanical:MountingHole
- added M_1_2, M_1_3, M_1_4, M_2_1, M_2_2, M_2_3, M_2_4, M_3_1, M_3_2, M_3_3, M_3_4, M_4_1, M_4_2, M_4_3, M_4_4: MountingHole, MountingHole:MountingHole_2.2mm_M2, symbol Mechanical:MountingHole
- renumbered H1 to M1_center1, H2 to M_1_1
Other:
- moved on the sheet: M1_center1

Commit message: modified:   kicad/teensypi_v91/teensypi_v91.kicad_pcb
Parts:
- added GND_PAD10, GND_PAD11, GND_PAD12, GND_PAD13, GND_PAD14, GND_PAD15, GND_PAD16, GND_PAD17, GND_PAD2, GND_PAD3, GND_PAD4, GND_PAD5, GND_PAD6, GND_PAD7, GND_PAD8, GND_PAD9: Conn_01x01, Connector_Wire:SolderWirePad_1x01_SMD_5x10mm, symbol Connector_Generic:Conn_01x01
Connections:
- net 3V3: now also GND_PAD2.1 (Pin_1)
- net GND: now also GND_PAD3.1 (Pin_1)

Commit message: modified:   kicad/teensypi_v91/teensypi_v91.kicad_pcb
Parts:
- added GND_PAD18, GND_PAD19, GND_PAD20, GND_PAD21: Conn_01x01, Connector_Wire:SolderWirePad_1x01_SMD_5x10mm, symbol Connector_Generic:Conn_01x01

Commit message: modified:   teensypi_v91/teensypi_v91.kicad_pcb
Connections:
- net 3V3: now also GND_PAD10.1 (Pin_1), GND_PAD16.1 (Pin_1); no longer GND_PAD2.1 (Pin_1)
- net 5V: now also GND_PAD19.1 (Pin_1)
- net GND: now also GND_PAD11.1 (Pin_1), GND_PAD18.1 (Pin_1); no longer GND_PAD3.1 (Pin_1)
- net INT: now also GND_PAD13.1 (Pin_1)
- net LED_MCU: now also Teensy_bottom1.12 (Pin_12)
- net M3: now also Motor3.2 (Pin_2), Teensy_bottom1.13 (Pin_13); no longer Motor4.2 (Pin_2)
- net M4: now also Motor4.2 (Pin_2); no longer Motor3.2 (Pin_2)
- net RX5: now also GND_PAD20.1 (Pin_1)
- net SCL0: now also GND_PAD14.1 (Pin_1)
- net SDA0: now also GND_PAD15.1 (Pin_1)
- net TX5: now also GND_PAD21.1 (Pin_1)
- net VBAT: now also Motor1.1 (Pin_1), Motor2.1 (Pin_1), Motor3.1 (Pin_1), Motor4.1 (Pin_1)
Other:
- moved on the sheet: Motor3, Motor4

Commit message: =More board routing
Connections:
- net CS: now also Teensy_top1.5 (Pin_5); no longer Teensy_top1.12 (Pin_12)
Changed lines of the file:
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@@
-	(wire
-		(pts
-			(xy 152.4 173.99) (xy 157.48 173.99)
-		)
-		(stroke
-			(width 0)
-			(type default)
-		)
-	)
 	(wire
 		(pts
@@
 		(pts
 			(xy 186.69 173.99) (xy 191.77 173.99)
+		)
+		(stroke
+			(width 0)
+			(type default)
+		)
+	)
+	(wire
+		(pts
+			(xy 152.4 156.21) (xy 157.48 156.21)
 		)
 		(stroke
@@
 		)
 	)
-	(label "CS"
-		(at 153.67 173.99 0)
-		(effects
-			(font
-				(size 1.27 1.27)
-			)
-			(justify left bottom)
-		)
-	)
 	(label "SCL0"
 		(at 151.13 38.1 0)
@@
 		(effects
 			(font
+				(size 1.27 1.27)
+			)
+			(justify left bottom)
+		)
+	)
+	(label "CS"
+		(at 152.4 156.21 0)
+		(effects
+			(font

Commit message: modified:   kicad/teensypi_v91/teensypi_v91.kicad_pcb
Changed lines of the file:
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@@
 	(wire
 		(pts
-			(xy 83.82 44.45) (xy 87.63 44.45)
+			(xy 115.57 44.45) (xy 119.38 44.45)
 		)
 		(stroke
@@
 	(wire
 		(pts
-			(xy 83.82 39.37) (xy 87.63 39.37)
+			(xy 115.57 39.37) (xy 119.38 39.37)
 		)
 		(stroke
@@
 	(wire
 		(pts
-			(xy 83.82 54.61) (xy 87.63 54.61)
+			(xy 115.57 54.61) (xy 119.38 54.61)
 		)
 		(stroke
@@
 	)
 	(label "GND"
-		(at 85.09 44.45 0)
+		(at 116.84 44.45 0)
 		(effects
 			(font
@@
 	)
 	(label "3V3"
-		(at 85.09 39.37 0)
+		(at 116.84 39.37 0)
 		(effects
 			(font
@@
 	)
 	(label "INT"
-		(at 85.09 54.61 0)
+		(at 116.84 54.61 0)
 		(effects
 			(font
@@
 	(symbol
 		(lib_id "Connector_Generic:Conn_01x01")
-		(at 121.92 55.88 0)
+		(at 95.25 52.07 0)
 		(unit 1)
 		(exclude_from_sim no)
@@
 		(fields_autoplaced yes)
 		(property "Reference" "GND_PAD5"
-			(at 124.46 54.6099 0)
+			(at 97.79 50.7999 0)
 			(effects
 				(font
@@
 		)
 		(property "Value" "Conn_01x01"
-			(at 124.46 57.1499 0)
+			(at 97.79 53.3399 0)
 			(effects
 				(font
@@
 		)
 		(property "Footprint" "Connector_Wire:SolderWirePad_1x01_SMD_5x10mm"
-			(at 121.92 55.88 0)
+			(at 95.25 52.07 0)
 			(effects
 				(font
@@
 		)
 		(property "Datasheet" "~"
-			(at 121.92 55.88 0)
+			(at 95.25 52.07 0)
 			(effects
 				(font
@@
 		)
 		(property "Description" "Generic connector, single row, 01x01, script generated (kicad-library-utils/schlib/autogen/connector/)"
-			(at 121.92 55.88 0)
+			(at 95.25 52.07 0)
 			(effects
 				(font
@@
 	(symbol
 		(lib_id "Connector_Generic:Conn_01x01")
-		(at 92.71 54.61 0)
+		(at 124.46 54.61 0)
 		(unit 1)
 		(exclude_from_sim no)
@@
 		(fields_autoplaced yes)
 		(property "Reference" "GND_PAD13"
-			(at 95.25 53.3399 0)
+			(at 127 53.3399 0)
 			(effects
 				(font
@@
 		)
 		(property "Value" "Conn_01x01"
-			(at 95.25 55.8799 0)
+			(at 127 55.8799 0)
 			(effects
 				(font
@@
 		)
 		(property "Footprint" "Connector_Wire:SolderWirePad_1x01_SMD_5x10mm"
-			(at 92.71 54.61 0)
+			(at 124.46 54.61 0)
 			(effects
 				(font
@@
 		)
 		(property "Datasheet" "~"
-			(at 92.71 54.61 0)
+			(at 124.46 54.61 0)
 			(effects
 				(font
@@
 		)
 		(property "Description" "Generic connector, single row, 01x01, script generated (kicad-library-utils/schlib/autogen/connector/)"
-			(at 92.71 54.61 0)
+			(at 124.46 54.61 0)
 			(effects
 				(font
@@
 	(symbol
 		(lib_id "Connector_Generic:Conn_01x01")
-		(at 92.71 49.53 0)
+		(at 124.46 49.53 0)
 		(unit 1)
 		(exclude_from_sim no)
@@
 		(fields_autoplaced yes)
 		(property "Reference" "GND_PAD12"
-			(at 95.25 48.2599 0)
+			(at 127 48.2599 0)
 			(effects
 				(font
@@
 		)
 		(property "Value" "Conn_01x01"
-			(at 95.25 50.7999 0)
+			(at 127 50.7999 0)
 			(effects
 				(font
@@
 		)
 		(property "Footprint" "Connector_Wire:SolderWirePad_1x01_SMD_5x10mm"
-			(at 92.71 49.53 0)
+			(at 124.46 49.53 0)
 			(effects
 				(font
@@
 		)
 		(property "Datasheet" "~"
-			(at 92.71 49.53 0)
+			(at 124.46 49.53 0)
 			(effects
 				(font
@@
 		)
 		(property "Description" "Generic connector, single row, 01x01, script generated (kicad-library-utils/schlib/autogen/connector/)"
-			(at 92.71 49.53 0)
+			(at 124.46 49.53 0)
 			(effects
 				(font
@@
 	(symbol
 		(lib_id "Connector_Generic:Conn_01x01")
-		(at 121.92 40.64 0)
+		(at 95.25 36.83 0)
 		(unit 1)
 		(exclude_from_sim no)
@@
 		(fields_autoplaced yes)
 		(property "Reference" "GND_PAD2"
-			(at 124.46 39.3699 0)
+			(at 97.79 35.5599 0)
 			(effects
 				(font
@@
 		)
 		(property "Value" "Conn_01x01"
-			(at 124.46 41.9099 0)
+			(at 97.79 38.0999 0)
 			(effects
 				(font
@@
 		)
 		(property "Footprint" "Connector_Wire:SolderWirePad_1x01_SMD_5x10mm"
-			(at 121.92 40.64 0)
+			(at 95.25 36.83 0)
 			(effects
 				(font
@@
 		)
 		(property "Datasheet" "~"
-			(at 121.92 40.64 0)
+			(at 95.25 36.83 0)
 			(effects
 				(font
@@
 		)
 		(property "Description" "Generic connector, single row, 01x01, script generated (kicad-library-utils/schlib/autogen/connector/)"
-			(at 121.92 40.64 0)
+			(at 95.25 36.83 0)
 			(effects
 				(font
@@
 	(symbol
 		(lib_id "Connector_Generic:Conn_01x01")
-		(at 121.92 45.72 0)
+		(at 95.25 41.91 0)
 		(unit 1)
 		(exclude_from_sim no)
@@
 		(fields_autoplaced yes)
 		(property "Reference" "GND_PAD3"
-			(at 124.46 44.4499 0)
+			(at 97.79 40.6399 0)
 			(effects
 				(font
@@
 		)
 		(property "Value" "Conn_01x01"
-			(at 124.46 46.9899 0)
+			(at 97.79 43.1799 0)
 			(effects
 				(font
@@
 		)
 		(property "Footprint" "Connector_Wire:SolderWirePad_1x01_SMD_5x10mm"
-			(at 121.92 45.72 0)
+			(at 95.25 41.91 0)
 			(effects
 				(font
@@
 		)
 		(property "Datasheet" "~"
-			(at 121.92 45.72 0)
+			(at 95.25 41.91 0)
 			(effects
 				(font
@@
 		)
 		(property "Description" "Generic connector, single row, 01x01, script generated (kicad-library-utils/schlib/autogen/connector/)"
-			(at 121.92 45.72 0)
+			(at 95.25 41.91 0)
 			(effects
 				(font
@@
 	(symbol
 		(lib_id "Connector_Generic:Conn_01x01")
-		(at 92.71 39.37 0)
+		(at 124.46 39.37 0)
 		(unit 1)
 		(exclude_from_sim no)
@@
 		(fields_autoplaced yes)
 		(property "Reference" "GND_PAD10"
-			(at 95.25 38.0999 0)
+			(at 127 38.0999 0)
 			(effects
 				(font
@@
 		)
 		(property "Value" "Conn_01x01"
-			(at 95.25 40.6399 0)
+			(at 127 40.6399 0)
 			(effects
 				(font
@@
 		)
 		(property "Footprint" "Connector_Wire:SolderWirePad_1x01_SMD_5x10mm"
-			(at 92.71 39.37 0)
+			(at 124.46 39.37 0)
 			(effects
 				(font
@@
 		)
 		(property "Datasheet" "~"
-			(at 92.71 39.37 0)
+			(at 124.46 39.37 0)
 			(effects
 				(font
@@
 		)
 		(property "Description" "Generic connector, single row, 01x01, script generated (kicad-library-utils/schlib/autogen/connector/)"
-			(at 92.71 39.37 0)
+			(at 124.46 39.37 0)
 			(effects
 				(font
@@
 	(symbol
 		(lib_id "Connector_Generic:Conn_01x01")
-		(at 92.71 44.45 0)
+		(at 124.46 44.45 0)
 		(unit 1)
 		(exclude_from_sim no)
@@
 		(fields_autoplaced yes)
 		(property "Reference" "GND_PAD11"
-			(at 95.25 43.1799 0)
+			(at 127 43.1799 0)
 			(effects
 				(font
@@
 		)
 		(property "Value" "Conn_01x01"
-			(at 95.25 45.7199 0)
+			(at 127 45.7199 0)
 			(effects
 				(font
@@
 		)
 		(property "Footprint" "Connector_Wire:SolderWirePad_1x01_SMD_5x10mm"
-			(at 92.71 44.45 0)
+			(at 124.46 44.45 0)
 			(effects
 				(font
@@
 		)
 		(property "Datasheet" "~"
-			(at 92.71 44.45 0)
+			(at 124.46 44.45 0)
 			(effects
 				(font
@@
 		)
 		(property "Description" "Generic connector, single row, 01x01, script generated (kicad-library-utils/schlib/autogen/connector/)"
-			(at 92.71 44.45 0)
+			(at 124.46 44.45 0)
 			(effects
 				(font
@@
 	(symbol
 		(lib_id "Connector_Generic:Conn_01x01")
-		(at 121.92 50.8 0)
+		(at 95.25 46.99 0)
 		(unit 1)
 		(exclude_from_sim no)
@@
 		(fields_autoplaced yes)
 		(property "Reference" "GND_PAD4"
-			(at 124.46 49.5299 0)
+			(at 97.79 45.7199 0)
 			(effects
 				(font
@@
 		)
 		(property "Value" "Conn_01x01"
-			(at 124.46 52.0699 0)
+			(at 97.79 48.2599 0)
 			(effects
 				(font
@@
 		)
 		(property "Footprint" "Connector_Wire:SolderWirePad_1x01_SMD_5x10mm"
-			(at 121.92 50.8 0)
+			(at 95.25 46.99 0)
 			(effects
 				(font
@@
 		)
 		(property "Datasheet" "~"
-			(at 121.92 50.8 0)
+			(at 95.25 46.99 0)
 			(effects
 				(font
@@
 		)
 		(property "Description" "Generic connector, single row, 01x01, script generated (kicad-library-utils/schlib/autogen/connector/)"
-			(at 121.92 50.8 0)
+			(at 95.25 46.99 0)
 			(effects
 				(font

Commit message: modified:   kicad/teensypi_v91/teensypi_v91.kicad_pcb
Parts:
- added POST_1, POST_2, POST_3, POST_4: MountingHole, MountingHole:MountingHole_2.2mm_M2, symbol Mechanical:MountingHole

Commit message: modified:   kicad/teensypi_v91/teensypi_v91.kicad_pcb
Parts:
- removed GND_PAD10, GND_PAD11, GND_PAD12, GND_PAD13, GND_PAD14, GND_PAD15, GND_PAD16, GND_PAD17, GND_PAD2, GND_PAD3, GND_PAD4, GND_PAD5, GND_PAD6, GND_PAD7, GND_PAD8, GND_PAD9: Conn_01x01, Connector_Wire:SolderWirePad_1x01_SMD_5x10mm, symbol Connector_Generic:Conn_01x01
- added J1: Conn_01x01_Socket, Connector_PinSocket_2.54mm:PinSocket_1x01_P2.54mm_Vertical, symbol Connector:Conn_01x01_Socket
- added Motor5: Conn_01x03_Female, Connector_PinHeader_2.54mm:PinHeader_1x03_P2.54mm_Vertical, symbol Connector:Conn_01x03_Female
- added PMW3901_PWR2: Conn_01x02_Female, Connector_PinHeader_2.54mm:PinHeader_1x02_P2.54mm_Vertical, symbol Connector:Conn_01x02_Female
Connections:
- net 3V3: now also Motor5.3 (Pin_3), PMW3901_PWR2.1 (Pin_1)
- net GND: now also PMW3901_PWR2.2 (Pin_2)
- net INT: now also J1.1 (Pin_1)
- net SCL0: now also Motor5.1 (Pin_1)
- net SDA0: now also Motor5.2 (Pin_2)
