File: kicad/feather/top/top.kicad_pcb (KiCad board)
At the start: 2 copper layers, 52 x 25.7 mm, 13 parts, among them J1 Conn_01x12_Socket, J2 Conn_01x16_Socket, J3 Conn_01x03_Socket

Commit message: modified:   kicad/feather/top/top.kicad_pro
Parts:
- added POST_5: MountingHole, MountingHole:MountingHole_4mm, F.Cu at (80.3, 116.3)
- moved J3 10.1 mm to (105.1, 113.9), turned to 180 degrees
- moved Motor5 2.84 mm to (101.5, 110.3)
- moved PMW3901_PWR2 2.84 mm to (87.2, 109.0)
- moved J2 2.00 mm to (70.0, 102.0)
- moved POST_2 1.33 mm to (65.1, 100.0)
- moved J1 1.00 mm to (70.0, 122.0)
- moved POST_3 0.65 mm to (112.0, 122.0)
Routing:
- net /3V3: track 65.3 -> 20.9 mm
- net /RX1: track 29.2 -> 7.28 mm
- net /TX1: track 25.3 -> 5.60 mm
- net /SCL: track 14.7 -> 0.00 mm
- net /SDA: track 12.1 -> 0.00 mm
- net /BOOT: track 4.13 -> 0.00 mm
- net /GND: track 32.2 -> 31.6 mm
Other:
- board text removed: "USB"

Commit message: modified:   kicad/feather/top/top.kicad_pro
Parts:
- moved POST_5 20.1 mm to (97.9, 106.6)
- moved Motor5 8.74 mm to (92.7, 109.9)
- moved PMW3901_PWR2 8.74 mm to (78.5, 108.7)
- moved J3 1.96 mm to (103.7, 112.6)
- moved POST_2 1.00 mm to (65.1, 101.0)
Connections:
- J3 pad 2: unconnected-(J3-Pin_2-Pad2) -> /3V3
- J3 pad 3: unconnected-(J3-Pin_3-Pad3) -> /BOOT
Routing:
- net /3V3: track 20.9 -> 41.0 mm
- net /SDA1: track 0.12 -> 18.8 mm
- net /SCL1: track 0.00 -> 15.7 mm
- net /GND: track 31.6 -> 18.3 mm, vias 1 -> 2
- net /BOOT: track 0.00 -> 7.39 mm
- net /RX1: track 7.28 -> 0.00 mm
- net /5V: track 8.74 -> 7.74 mm
- net /TX1: track 5.60 -> 4.96 mm, vias 0 -> 1
Other:
- outline, holes or cut-outs redrawn

Commit message: modified:   kicad/feather/top/top.kicad_pcb
Connections:
- GND_PAD20 pad 1: /RX1 -> /TX1
- GND_PAD21 pad 1: /TX1 -> /RX1
Routing:
- net /RX1: track 0.00 -> 28.9 mm, vias 0 -> 2
- net /TX1: track 4.96 -> 24.9 mm
- net /GND: track 18.3 -> 17.0 mm
- added copper zone on F.Cu, net /GND
Other:
- board size 52 x 25.7 mm -> 52 x 24.8 mm
Changed lines of the file:
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@@
 			(size 3 1.5)
 			(layers "F.Cu" "F.Mask" "F.Paste")
-			(net 2 "/RX1")
+			(net 3 "/TX1")
 			(pinfunction "Pin_1")
 			(pintype "passive")
@@
 			(size 3 1.5)
 			(layers "F.Cu" "F.Mask" "F.Paste")
-			(net 3 "/TX1")
+			(net 2 "/RX1")
 			(pinfunction "Pin_1")
 			(pintype "passive")
@@
 	(gr_poly
 		(pts
-			(xy 105.247749 86.127626) (xy 103.769188 88.835059) (xy 106.905732 88.835059)
+			(xy 98.181788 112.709085) (xy 96.703227 115.416518) (xy 99.839771 115.416518)
 		)
 		(stroke
@@
 	)
 	(gr_line
-		(start 63 98.67)
+		(start 63 99.5)
 		(end 63 124.33)
 		(stroke
@@
 	)
 	(gr_line
-		(start 115 98.67)
+		(start 115 99.5)
 		(end 115 106)
 		(stroke
@@
 		)
 	)
-	(gr_text "RX1"
+	(gr_text "TX1"
 		(at 65.5 110.768769 0)
 		(layer "F.SilkS")
@@
 		)
 	)
-	(gr_text "TX1\n"
+	(gr_text "RX1\n"
 		(at 65.5 107.868769 0)
 		(layer "F.SilkS")
@@
 	)
 	(gr_text "5V"
-		(at 74.351984 121.3 0)
+		(at 74.351984 120.6 0)
 		(layer "F.SilkS")
 		(effects
@@
 	)
 	(segment
-		(start 72.45 113.4)
-		(end 72.318769 113.268769)
-		(width 0.4)
-		(layer "F.Cu")
-		(net 1)
-	)
-	(segment
-		(start 69.080694 113.268769)
-		(end 70.261873 113.268769)
-		(width 0.4)
-		(layer "F.Cu")
-		(net 1)
-	)
-	(segment
-		(start 72.318769 113.268769)
-		(end 70.261873 113.268769)
+		(start 73.8 112.05)
+		(end 72.581231 113.268769)
 		(width 0.4)
 		(layer "F.Cu")
@@
 	)
 	(segment
-		(start 73.8 112.05)
-		(end 72.45 113.4)
+		(start 72.581231 113.268769)
+		(end 70.261873 113.268769)
 		(width 0.4)
 		(layer "F.Cu")
@@
 	(segment
 		(start 70.173891 107.268769)
-		(end 72.9 109.994878)
-		(width 0.2)
+		(end 74.587336 107.268769)
+		(width 0.3)
+		(layer "F.Cu")
+		(net 2)
+	)
+	(segment
+		(start 74.60498 107.251125)
+		(end 74.587336 107.268769)
+		(width 0.3)
+		(layer "F.Cu")
+		(net 2)
+	)
+	(segment
+		(start 74.587336 107.268769)
+		(end 74.50213 107.268769)
+		(width 0.3)
+		(layer "F.Cu")
+		(net 2)
+	)
+	(via
+		(at 74.587336 107.268769)
+		(size 0.5)
+		(drill 0.3)
+		(layers "F.Cu" "B.Cu")
+		(net 2)
+	)
+	(via
+		(at 74.587336 107.268769)
+		(size 0.5)
+		(drill 0.3)
+		(layers "F.Cu" "B.Cu")
+		(net 2)
+	)
+	(segment
+		(start 74.587336 107.268769)
+		(end 78.128769 107.268769)
+		(width 0.3)
+		(layer "B.Cu")
+		(net 2)
+	)
+	(segment
+		(start 78.128769 107.268769)
+		(end 92.86 122)
+		(width 0.3)
+		(layer "B.Cu")
+		(net 2)
+	)
+	(segment
+		(start 70.305863 110.268769)
+		(end 71.569175 110.268769)
+		(width 0.3)
 		(layer "F.Cu")
 		(net 3)
 	)
 	(segment
-		(start 72.9 109.994878)
-		(end 72.9 111.1)
-		(width 0.2)
+		(start 71.569175 110.268769)
+		(end 72.9772 111.676794)
+		(width 0.3)
 		(layer "F.Cu")
 		(net 3)
 	)
 	(via
-		(at 72.9 111.1)
+		(at 72.9772 111.676794)
 		(size 0.6)
 		(drill 0.3)
@@
 	)
 	(segment
+		(start 81.23696 119.936554)
+		(end 88.256554 119.936554)
+		(width 0.3)
+		(layer "B.Cu")
+		(net 3)
+	)
+	(segment
+		(start 72.9772 111.676794)
+		(end 81.23696 119.936554)
+		(width 0.3)
+		(layer "B.Cu")
+		(net 3)
+	)
+	(segment
+		(start 88.256554 119.936554)
+		(end 90.32 122)
+		(width 0.3)
+		(layer "B.Cu")
+		(net 3)
+	)
+	(segment
 		(start 93.466397 112.486703)
 		(end 93.591279 112.486703)
@@
 		(net 23)
 	)
+	(zone
+		(net 1)
+		(net_name "/GND")
+		(layer "F.Cu")
+		(hatch edge 0.5)
+		(connect_pads
+			(clearance 0.4)
+		)
+		(min_thickness 0.25)
+		(filled_areas_thickness no)
+		(fill yes
+			(thermal_gap 0.5)
+			(thermal_bridge_width 0.5)
+		)
+		(polygon
+			(pts
+				(xy 63 99.5) (xy 115 99.5) (xy 115 124.33) (xy 63 124.33)
+			)
+		)
+	)
 	(embedded_fonts no)

Commit message: modified:   kicad/feather/top/top.kicad_pro
Parts:
- J1, J2: moved to B.Cu
- moved J2 112.1 mm to (182.0, 97.5)
- moved J1 106.8 mm to (176.8, 117.5)
- moved GND_PAD19 73.9 mm to (144.1, 111.9)
- moved GND_PAD21 73.9 mm to (144.1, 104.6)
- moved Motor5 73.9 mm to (166.5, 105.4)
- moved POST_2 73.9 mm to (138.9, 96.5)
- moved GND_PAD18 73.9 mm to (144.2, 110.2)
- moved GND_PAD20 73.9 mm to (144.2, 107.3)
- moved J3 73.9 mm to (177.4, 108.1)
- moved POST_3 73.9 mm to (185.8, 117.5)
- moved POST_4 73.9 mm to (139.7, 117.8)
- moved PMW3901_PWR2 73.9 mm to (152.3, 104.2)
- moved POST_1 73.9 mm to (187.1, 96.5)
- moved POST_5 73.9 mm to (171.7, 102.5)
Connections:
- J1 pad 10: /RX1 -> (no net)
- J1 pad 11: /SCL -> /TX1
- J1 pad 12: /SDA -> /RX1
- J1 pad 13: (no net) -> /SCL
- J1 pad 14: (no net) -> /SDA
- J1 pad 9: /TX1 -> (no net)
- Motor5 pad 1: /SCL1 -> /SCL
- Motor5 pad 2: /SDA1 -> /SDA
Routing:
- net /SCL: track 0.00 -> 33.4 mm
- net /BOOT: track 7.39 -> 35.8 mm
- net /SDA: track 0.00 -> 27.6 mm
- net /5V: track 7.74 -> 30.0 mm
- net /GND: track 17.0 -> 37.6 mm, vias 2 -> 0
- net /SDA1: track 18.8 -> 0.00 mm
- net /SCL1: track 15.7 -> 0.00 mm
- net /RX1: track 28.9 -> 24.0 mm, vias 2 -> 0
- net /TX1: track 24.9 -> 21.9 mm, vias 1 -> 0
- net /3V3: track 41.0 -> 43.0 mm
Other:
- outline, holes or cut-outs redrawn
- board text removed: "SCL1"
- board text removed: "SDA1"
