File: kicad/teensy/top/top.kicad_sch (KiCad schematic)
At the start: 4 parts, among them J1 Conn_01x08_Socket, J2 Conn_01x08_Socket

Commit message: modified:   kicad/teensy/top/top.kicad_pcb
Parts:
- removed J1, J2: Conn_01x08_Socket, Connector_PinSocket_2.54mm:PinSocket_1x08_P2.54mm_Vertical, symbol Connector:Conn_01x08_Socket
- added J1: Conn_01x04_Socket, Connector_PinHeader_2.00mm:PinHeader_1x04_P2.00mm_Vertical, symbol Connector:Conn_01x04_Socket
- added J2: Conn_01x09_Socket, Connector_PinSocket_2.54mm:PinSocket_1x09_P2.54mm_Vertical, symbol Connector:Conn_01x09_Socket
- added J3: Conn_01x09_Socket, Connector_PinHeader_2.54mm:PinHeader_1x09_P2.54mm_Vertical, symbol Connector:Conn_01x09_Socket
Connections:
- net 3V3: now also J2.3 (Pin_3)
- net GND: now also J1.3 (Pin_3), J2.2 (Pin_2), J3.1 (Pin_1)
- net SCL0: now also J2.8 (Pin_8)
- net SDA0: now also J2.9 (Pin_9)
- new net 5V: J1.4 (Pin_4), J2.1 (Pin_1)
- new net RX5: J1.2 (Pin_2), J2.6 (Pin_6)
- new net TX5: J1.1 (Pin_1), J2.7 (Pin_7)
