File: kicad/teensy/bottom/bottom.kicad_pcb (KiCad board)
At the start: 2 copper layers, 27.5 x 21.7 mm, 5 parts, among them J1 Conn_01x04_Socket, J2 Conn_01x09_Socket, J3 Conn_01x09_Socket

Commit message: modified:   kicad/teensy/bottom/bottom.kicad_pro
Parts:
- removed J1: Conn_01x04_Socket, Connector_PinHeader_2.00mm:PinHeader_1x04_P2.00mm_Vertical
- removed J2, J3: Conn_01x09_Socket, Connector_PinHeader_2.54mm:PinHeader_1x09_P2.54mm_Vertical
- removed Motor5: Conn_01x03_Female, Connector_PinHeader_2.54mm:PinHeader_1x03_P2.54mm_Vertical
- removed PMW3901_PWR2: Conn_01x02_Female, Connector_PinHeader_2.54mm:PinHeader_1x02_P2.54mm_Vertical
- added J4: Conn_01x14_Socket, Connector_PinSocket_2.54mm:PinSocket_1x14_P2.54mm_Vertical, F.Cu at (167.5, 93.4)
- added J5: Conn_01x14_Socket, Connector_PinSocket_2.54mm:PinSocket_1x14_P2.54mm_Vertical, F.Cu at (167.5, 108.2)
Routing:
- net /GND: track 33.6 -> 0.00 mm
- net /3V3: track 25.9 -> 0.00 mm
- net /SDA0: track 19.7 -> 0.00 mm, vias 1 -> 0
- net /SCL0: track 17.5 -> 0.00 mm
- net /5V: track 8.79 -> 0.00 mm
- net /TX5: track 3.41 -> 0.00 mm
- net /RX5: track 3.18 -> 0.00 mm
- net /CS: track 0.00 -> 0.93 mm
- removed copper zone on F.Cu, net /GND
Other:
- board outline removed
- board text added: "CS"
- board text added: "MISO"
- board text added: "MOSI"
- board text added: "SCK"
- board text added: "SCL1"
- board text added: "SDA1"
- board text added: "USB"
- board text removed: "RX5"
- board text removed: "SCL"
- board text removed: "SDA"
- board text removed: "TX5"

Commit message: modified:   kicad/teensy/bottom/bottom.kicad_pcb
Parts:
- added J1: Conn_01x04_Socket, Connector_PinSocket_2.54mm:PinSocket_1x04_P2.54mm_Vertical, F.Cu at (137.8, 97.1)
- added J2: Conn_01x03_Socket, Connector_PinSocket_2.54mm:PinSocket_1x03_P2.54mm_Vertical, F.Cu at (153.0, 103.5)
- added J3: Conn_01x02_Socket, Connector_PinSocket_2.54mm:PinSocket_1x02_P2.54mm_Vertical, F.Cu at (144.5, 104.6)
- added J6: Conn_01x04_Socket, Connector_PinSocket_2.54mm:PinSocket_1x04_P2.54mm_Vertical, F.Cu at (149.2, 104.8)
- added J7: Conn_01x03_Socket, Connector_PinSocket_2.54mm:PinSocket_1x03_P2.54mm_Vertical, F.Cu at (162.9, 98.7)

Commit message: modified:   kicad/teensy/bottom/bottom.kicad_pro
Parts:
- added GND_PAD1: Conn_01x01, Connector_Wire:SolderWirePad_1x01_SMD_5x10mm, F.Cu at (149.0, 118.3)
- added M1: Conn_01x03_Socket, Connector_PinSocket_2.54mm:PinSocket_1x03_P2.54mm_Vertical, F.Cu at (170.0, 80.0)
- added M2: Conn_01x03_Socket, Connector_PinSocket_2.54mm:PinSocket_1x03_P2.54mm_Vertical, F.Cu at (173.5, 121.0)
- added M3: Conn_01x03_Socket, Connector_PinSocket_2.54mm:PinSocket_1x03_P2.54mm_Vertical, F.Cu at (128.5, 121.0)
- added M4: Conn_01x03_Socket, Connector_PinSocket_2.54mm:PinSocket_1x03_P2.54mm_Vertical, F.Cu at (132.0, 80.0)
- added VB_PAD1: Conn_01x01, Connector_Wire:SolderWirePad_1x01_SMD_5x10mm, F.Cu at (152.2, 118.0)
- moved J2 15.4 mm to (168.2, 105.5)
- moved J7 11.8 mm to (153.2, 105.5), turned to 180 degrees
- moved J1 3.60 mm to (135.0, 99.3)
- moved J6 2.34 mm to (150.0, 107.0)
- moved J3 2.26 mm to (145.0, 106.9)
- moved J5 2.26 mm to (168.0, 110.4)
- moved J4 2.26 mm to (168.0, 95.6)
Connections:
- J1 pad 1: /SCK -> unconnected-(J1-Pin_1-Pad1)
- J1 pad 4: unconnected-(J1-Pin_4-Pad4) -> /SCK
- J7 pad 2: /SDA1 -> /SCL1
- J7 pad 3: /SCL1 -> /SDA1
Other:
- board text added: "M1"
- board text added: "M2"
- board text added: "M3"
- board text added: "VBAT"
- board text removed: "USB"

Commit message: modified:   kicad/teensy/bottom/bottom.kicad_pcb
Parts:
- added J8: Conn_01x04_Socket, Connector_PinSocket_2.54mm:PinSocket_1x04_P2.54mm_Vertical, F.Cu at (141.8, 114.5)
- moved J4 15.1 mm to (168.0, 110.8)
- moved J5 14.7 mm to (168.0, 95.8)
- moved M4 8.73 mm to (135.5, 88.0)
- moved M1 8.54 mm to (167.0, 88.0)
- moved M2 8.49 mm to (167.5, 115.0)
- moved M3 7.91 mm to (133.0, 114.5)
Connections:
- J4 pad 13: unconnected-(J4-Pin_13-Pad13) -> /M3
- J4 pad 2: /3V3 -> /GND
- J4 pad 3: /GND -> /3V3
- J4 pad 4: unconnected-(J4-Pin_4-Pad4) -> /M2
- J4 pad 6: unconnected-(J4-Pin_6-Pad6) -> /RX5
- J4 pad 7: unconnected-(J4-Pin_7-Pad7) -> /TX5
- J4 pad 8: unconnected-(J4-Pin_8-Pad8) -> /SCL0
- J4 pad 9: unconnected-(J4-Pin_9-Pad9) -> /SDA0
- J5 pad 11: unconnected-(J5-Pin_11-Pad11) -> /M4
- J5 pad 2: unconnected-(J5-Pin_2-Pad2) -> /M1
- M3 pad 1: /M3 -> /GND
- M3 pad 3: /GND -> /M3
- M4 pad 1: /M4 -> /GND
- M4 pad 3: /GND -> /M4
Routing:
- net /VBAT: track 0.00 -> 113.3 mm, vias 0 -> 1
- net /GND: track 0.00 -> 77.4 mm, vias 0 -> 1
- net /3V3: track 0.00 -> 32.3 mm
- net /SDA1: track 0.00 -> 28.6 mm, vias 0 -> 1
- net /5V: track 0.00 -> 28.3 mm, vias 0 -> 2
- net /SCL1: track 0.00 -> 21.0 mm
- net /MISO: track 0.00 -> 19.7 mm
- net /MOSI: track 0.00 -> 16.8 mm
- net /CS: track 0.93 -> 12.5 mm
- net /SCK: track 0.00 -> 3.87 mm
- net unconnected-(J4-Pin_12-Pad12): track 0.00 -> 0.93 mm
- net /M4: track 0.00 -> 0.65 mm
- added copper zone on F.Cu, net /GND
Other:
- board outline added: 43.5 x 39.5 mm
- board text added: "GD"
- board text added: "M4"
- board text added: "SI"
- board text added: "SO"
- board text added: "VB"
- board text removed: "MISO"
- board text removed: "MOSI"

Commit message: modified:   kicad/teensy/bottom/bottom.kicad_pcb
Parts:
- moved M3 10.5 mm to (132.9, 125.0), turned to -135 degrees
- moved M2 7.30 mm to (170.8, 121.5)
- moved M1 7.00 mm to (167.0, 81.0)
- moved M4 6.77 mm to (129.7, 84.5), turned to 135 degrees
Connections:
- M2 pad 1: /M2 -> /GND
- M2 pad 3: /GND -> /M2
- M3 pad 1: /GND -> /M3
- M3 pad 3: /M3 -> /GND
Routing:
- net /GND: track 77.4 -> 161.6 mm
- net /M4: track 0.65 -> 19.3 mm
- net /M2: track 0.25 -> 17.4 mm
- net /M3: track 0.00 -> 16.5 mm
- net /M1: track 0.00 -> 15.4 mm
- net /VBAT: track 113.3 -> 124.3 mm, vias 1 -> 0
- net /5V: track 28.3 -> 27.7 mm
Other:
- board size 43.5 x 39.5 mm -> 47.6 x 51 mm
- board text added: "PMW3901"
- board text added: "USB"
- board text added: "VL53L1X"
