File: kicad/teensy2/teensy2.kicad_pcb (KiCad board)
At the start: 2 copper layers, 6 parts, among them J1 Conn_01x14_Socket, J2 Conn_01x14_Socket

Commit message: modified:   kicad/teensy2/teensy2.kicad_pcb
Parts:
- added J3: Conn_01x04_Socket, Connector_PinHeader_2.54mm:PinHeader_1x04_P2.54mm_Vertical, F.Cu at (148.4, 97.8)
- added J4: Conn_01x03_Socket, Connector_PinHeader_2.54mm:PinHeader_1x03_P2.54mm_Vertical, F.Cu at (150.3, 64.6)
- added J5: Conn_01x06_Pin, Connector_PinHeader_2.00mm:PinHeader_1x06_P2.00mm_Vertical, F.Cu at (148.1, 60.8)
- moved J1 1.00 mm to (162.0, 76.2)
- moved J2 1.00 mm to (162.0, 91.2)
Routing:
- net /GND: track 16.1 -> 0.00 mm
Other:
- board text added: "GND"
- board text added: "M1"
- board text added: "M2"
- board text added: "M3"
- board text added: "M4"
- board text added: "VBAT"

Commit message: modified:   kicad/teensy2/teensy2.kicad_pcb
Parts:
- added J6: Conn_01x04_Socket, Connector_PinHeader_2.00mm:PinHeader_1x04_P2.00mm_Vertical, F.Cu at (127.9, 65.3)
Other:
- board text added: "RX"
- board text added: "TX"
Changed lines of the file:
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@@
 	(net 31 "/M1")
 	(net 32 "/M4")
+	(net 33 "/TX")
+	(net 34 "/RX")
 	(footprint "MountingHole:MountingHole_2.5mm"
 		(layer "F.Cu")
@@
 		(embedded_fonts no)
 	)
+	(footprint "Connector_PinHeader_2.00mm:PinHeader_1x04_P2.00mm_Vertical"
+		(layer "F.Cu")
+		(at 127.908715 65.299896)
+		(descr "Through hole straight pin header, 1x04, 2.00mm pitch, single row")
+		(tags "Through hole pin header THT 1x04 2.00mm single row")
+		(property "Reference" "J6"
+			(at 0 -2.11 0)
+			(layer "F.SilkS")
+			(hide yes)
+			(effects
+				(font
+					(size 1 1)
+					(thickness 0.15)
+				)
+			)
+		)
+		(property "Value" "Conn_01x04_Socket"
+			(at 0 8.11 0)
+			(layer "F.Fab")
+			(hide yes)
+			(effects
+				(font
+					(size 1 1)
+					(thickness 0.15)
+				)
+			)
+		)
+		(property "Datasheet" "~"
+			(at 0 0 0)
+			(layer "F.Fab")
+			(hide yes)
+			(effects
+				(font
+					(size 1.27 1.27)
+					(thickness 0.15)
+				)
+			)
+		)
+		(property "Description" "Generic connector, single row, 01x04, script generated"
+			(at 0 0 0)
+			(layer "F.Fab")
+			(hide yes)
+			(effects
+				(font
+					(size 1.27 1.27)
+					(thickness 0.15)
+				)
+			)
+		)
+		(property ki_fp_filters "Connector*:*_1x??_*")
+		(sheetname "/")
+		(sheetfile "teensy2.kicad_sch")
+		(attr through_hole)
+		(fp_line
+			(start -1 -0.5)
+			(end -0.5 -1)
+			(stroke
+				(width 0.1)
+				(type solid)
+			)
+			(layer "F.Fab")
+		)
+		(fp_line
+			(start -1 7)
+			(end -1 -0.5)
+			(stroke
+				(width 0.1)
+				(type solid)
+			)
+			(layer "F.Fab")
+		)
+		(fp_line
+			(start -0.5 -1)
+			(end 1 -1)
+			(stroke
+				(width 0.1)
+				(type solid)
+			)
+			(layer "F.Fab")
+		)
+		(fp_line
+			(start 1 -1)
+			(end 1 7)
+			(stroke
+				(width 0.1)
+				(type solid)
+			)
+			(layer "F.Fab")
+		)
+		(fp_line
+			(start 1 7)
+			(end -1 7)
+			(stroke
+				(width 0.1)
+				(type solid)
+			)
+			(layer "F.Fab")
+		)
+		(pad "1" thru_hole rect
+			(at 0 0)
+			(size 1.35 1.35)
+			(drill 0.8)
+			(layers "*.Cu" "*.Mask")
+			(remove_unused_layers no)
+			(net 33 "/TX")
+			(pinfunction "Pin_1")
+			(pintype "passive")
+		)
+		(pad "2" thru_hole circle
+			(at 0 2)
+			(size 1.35 1.35)
+			(drill 0.8)
+			(layers "*.Cu" "*.Mask")
+			(remove_unused_layers no)
+			(net 34 "/RX")
+			(pinfunction "Pin_2")
+			(pintype "passive")
+		)
+		(pad "3" thru_hole circle
+			(at 0 4)
+			(size 1.35 1.35)
+			(drill 0.8)
+			(layers "*.Cu" "*.Mask")
+			(remove_unused_layers no)
+			(net 4 "/GND")
+			(pinfunction "Pin_3")
+			(pintype "passive")
+		)
+		(pad "4" thru_hole circle
+			(at 0 6)
+			(size 1.35 1.35)
+			(drill 0.8)
+			(layers "*.Cu" "*.Mask")
+			(remove_unused_layers no)
+			(net 19 "/5V")
+			(pinfunction "Pin_4")
+			(pintype "passive")
+		)
+		(embedded_fonts no)
+		(model "${KICAD9_3DMODEL_DIR}/Connector_PinHeader_2.00mm.3dshapes/PinHeader_1x04_P2.00mm_Vertical.step"
+			(offset
+				(xyz 0 0 0)
+			)
+			(scale
+				(xyz 1 1 1)
+			)
+			(rotate
+				(xyz 0 0 0)
+			)
+		)
+	)
 	(footprint "Connector_PinHeader_2.54mm:PinHeader_1x03_P2.54mm_Vertical"
 		(layer "F.Cu")
@@
 		)
 	)
+	(gr_text "5V"
+		(at 128.908715 72.299896 0)
+		(layer "F.SilkS")
+		(effects
+			(font
+				(size 1 1)
+				(thickness 0.15)
+			)
+			(justify left bottom)
+		)
+	)
 	(gr_text "CS"
 		(at 134.663521 79.941875 90)
@@
 		)
 	)
+	(gr_text "TX"
+		(at 128.908715 65.702803 0)
+		(layer "F.SilkS")
+		(effects
+			(font
+				(size 1 1)
+				(thickness 0.15)
+			)
+			(justify left bottom)
+		)
+	)
 	(gr_text "VBAT"
 		(at 152.974597 70.729429 0)
@@
 		(layer "F.SilkS")
 		(effects
+			(font
+				(size 1 1)
+				(thickness 0.15)
+			)
+			(justify left bottom)
+		)
+	)
+	(gr_text "RX"
+		(at 128.908715 67.677518 0)
+		(layer "F.SilkS")
+		(effects
+			(font
+				(size 1 1)
+				(thickness 0.15)
+			)
+			(justify left bottom)
+		)
+	)
+	(gr_text "GD"
+		(at 128.908715 69.919087 0)
+		(layer "F.SilkS")
+		(effects

Commit message: modified:   kicad/hoverdeck/hoverdeck.kicad_pcb
Other:
- board text added: "COMMS"
- board text added: "IMU"
- board text added: "MOTORS"
- board text added: "REG"
Changed lines of the file:
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@@
 	)
 	(gr_text "USB"
-		(at 163.851644 87.088137 90)
+		(at 161.7 81.375 270)
 		(layer "F.SilkS")
 		(effects
@@
 		)
 	)
+	(gr_text "REG"
+		(at 157.05 64.65 270)
+		(layer "F.SilkS")
+		(effects
+			(font
+				(size 2 2)
+				(thickness 0.15)
+			)
+			(justify left bottom)
+		)
+	)
 	(gr_text "GD"
 		(at 148.644013 59.808556 90)
@@
 		)
 	)
+	(gr_text "IMU"
+		(at 153.5 100.3 270)
+		(layer "F.SilkS")
+		(effects
+			(font
+				(size 2 2)
+				(thickness 0.15)
+			)
+			(justify left bottom)
+		)
+	)
 	(gr_text "GD"
 		(at 159.887997 89.98 90)
@@
 			(font
 				(size 1 1)
+				(thickness 0.15)
+			)
+			(justify left bottom)
+		)
+	)
+	(gr_text "COMMS"
+		(at 123.875 63.425 270)
+		(layer "F.SilkS")
+		(effects
+			(font
+				(size 2 2)
 				(thickness 0.15)
 			)
@@
 				(thickness 0.15)
 			)
+			(justify left bottom)
+		)
+	)
+	(gr_text "MOTORS"
+		(at 137.325 56.625 0)
+		(layer "F.SilkS")
+		(effects
+			(font
+				(size 2 2)
+				(thickness 0.15)
+			)

Commit message: modified:   kicad/teensy2/teensy2.kicad_pcb
Parts:
- added J7: Conn_01x08_Pin, Connector_PinSocket_2.00mm:PinSocket_1x08_P2.00mm_Vertical, F.Cu at (152.1, 87.8)
- moved J6 34.4 mm to (133.0, 99.3)
- moved J5 18.6 mm to (149.8, 79.3)
- moved J3 2.13 mm to (150.2, 99.0)
Other:
- board text added: "HOVER"
- board text added: "VB"
