File: kicad/teensy2/teensy2.kicad_sch (KiCad schematic)
At the start: 6 parts, among them J1 Conn_01x14_Socket, J2 Conn_01x14_Socket

Commit message: modified:   kicad/teensy2/teensy2.kicad_pcb
Parts:
- added J3: Conn_01x04_Socket, Connector_PinHeader_2.54mm:PinHeader_1x04_P2.54mm_Vertical, symbol Connector:Conn_01x04_Socket
- added J4: Conn_01x03_Socket, Connector_PinHeader_2.54mm:PinHeader_1x03_P2.54mm_Vertical, symbol Connector:Conn_01x03_Socket
- added J5: Conn_01x06_Pin, Connector_PinHeader_2.00mm:PinHeader_1x06_P2.00mm_Vertical, symbol Connector:Conn_01x06_Pin
Connections:
- net 3V3: now also J3.4 (Pin_4)
- net 5V: now also J4.1 (Pin_1)
- net GND: now also J3.3 (Pin_3), J4.2 (Pin_2), J5.1 (Pin_1)
- net SCL0: now also J3.1 (Pin_1)
- net SDA0: now also J3.2 (Pin_2)
- new net M1: J5.3 (Pin_3)
- new net M2: J5.4 (Pin_4)
- new net M3: J5.5 (Pin_5)
- new net M4: J5.6 (Pin_6)
- new net VBAT: J4.3 (Pin_3), J5.2 (Pin_2)

Commit message: modified:   kicad/teensy2/teensy2.kicad_pcb
Parts:
- added J6: Conn_01x04_Socket, Connector_PinHeader_2.00mm:PinHeader_1x04_P2.00mm_Vertical, symbol Connector:Conn_01x04_Socket
Connections:
- net 5V: now also J6.4 (Pin_4)
- net GND: now also J6.3 (Pin_3)
- new net RX: J6.2 (Pin_2)
- new net TX: J6.1 (Pin_1)
Changed lines of the file:
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@@
+	(wire
+		(pts
+			(xy 162.56 101.6) (xy 167.64 101.6)
+		)
+		(stroke
+			(width 0)
+			(type default)
+		)
+	)
+	(wire
+		(pts
+			(xy 162.56 106.68) (xy 167.64 106.68)
+		)
+		(stroke
+			(width 0)
+			(type default)
+		)
+	)
 	(wire
 		(pts
@@
 	(wire
 		(pts
+			(xy 162.56 104.14) (xy 167.64 104.14)
+		)
+		(stroke
+			(width 0)
+			(type default)
+		)
+	)
+	(wire
+		(pts
 			(xy 91.44 132.08) (xy 96.52 132.08)
 		)
@@
 		(pts
 			(xy 91.44 104.14) (xy 96.52 104.14)
+		)
+		(stroke
+			(width 0)
+			(type default)
+		)
+	)
+	(wire
+		(pts
+			(xy 162.56 99.06) (xy 167.64 99.06)
 		)
 		(stroke
@@
 		)
 	)
+	(label "TX"
+		(at 163.83 99.06 0)
+		(effects
+			(font
+				(size 1.27 1.27)
+			)
+			(justify left bottom)
+		)
+	)
 	(label "GND"
 		(at 120.65 101.6 0)
@@
 		)
 	)
+	(label "5V"
+		(at 163.83 106.68 0)
+		(effects
+			(font
+				(size 1.27 1.27)
+			)
+			(justify left bottom)
+		)
+	)
 	(label "MISO"
 		(at 91.44 132.08 0)
@@
 		)
 	)
+	(label "RX"
+		(at 163.83 101.6 0)
+		(effects
+			(font
+				(size 1.27 1.27)
+			)
+			(justify left bottom)
+		)
+	)
 	(label "MOSI"
 		(at 91.44 129.54 0)
@@
 	(label "GND"
 		(at 144.78 105.41 0)
+		(effects
+			(font
+				(size 1.27 1.27)
+			)
+			(justify left bottom)
+		)
+	)
+	(label "GND"
+		(at 163.83 104.14 0)
 		(effects
 			(font
@@
 					(unit 1)
 				)
+			)
+		)
+	)
+	(symbol
+		(lib_id "Connector:Conn_01x04_Socket")
+		(at 172.72 101.6 0)
+		(unit 1)
+		(exclude_from_sim no)
+		(in_bom yes)
+		(on_board yes)
+		(dnp no)
+		(fields_autoplaced yes)
+		(property "Reference" "J6"
+			(at 173.99 101.5999 0)
+			(effects
+				(font
+					(size 1.27 1.27)
+				)
+				(justify left)
+				(hide yes)
+			)
+		)
+		(property "Value" "Conn_01x04_Socket"
+			(at 173.99 104.1399 0)
+			(effects
+				(font
+					(size 1.27 1.27)
+				)
+				(justify left)
+				(hide yes)
+			)
+		)
+		(property "Footprint" "Connector_PinHeader_2.00mm:PinHeader_1x04_P2.00mm_Vertical"
+			(at 172.72 101.6 0)
+			(effects
+				(font
+					(size 1.27 1.27)
+				)
+				(hide yes)
+			)
+		)
+		(property "Datasheet" "~"
+			(at 172.72 101.6 0)
+			(effects
+				(font
+					(size 1.27 1.27)
+				)
+				(hide yes)
+			)
+		)
+		(property "Description" "Generic connector, single row, 01x04, script generated"
+			(at 172.72 101.6 0)
+			(effects
+				(font
+					(size 1.27 1.27)
+				)
+				(hide yes)
+			)
+		)
+		(pin "2"
+		)
+		(pin "1"
+		)
+		(pin "3"
+		)
+		(pin "4"
+		)
+		(instances
+			(project ""
+				(path "/2b1f0318-b347-4cb8-9bbf-78e69ec66761"
+					(reference "J6")
+					(unit 1)
+				)

Commit message: modified:   kicad/teensy2/teensy2.kicad_pcb
Parts:
- added J7: Conn_01x08_Pin, Connector_PinSocket_2.00mm:PinSocket_1x08_P2.00mm_Vertical, symbol Connector:Conn_01x08_Pin
Connections:
- net 3V3: now also J7.8 (Pin_8)
- net CS: now also J7.5 (Pin_5)
- net GND: now also J7.7 (Pin_7)
- net MISO: now also J7.3 (Pin_3)
- net MOSI: now also J7.4 (Pin_4)
- net SCK: now also J7.6 (Pin_6)
- net SCL1: now also J7.2 (Pin_2)
- net SDA1: now also J7.1 (Pin_1)
Other:
- note added: "COMMS"
- note added: "HOVER"
- note added: "IMU"
- note added: "MOTORS"
- note added: "REG"
