File: kicad/teensy2-bottom/teensy2-bottom.kicad_sch (KiCad schematic)
At the start: 11 parts, among them J1 Conn_01x14_Socket, J2 Conn_01x14_Socket, J3 Conn_01x04_Socket, J4 Conn_01x03_Socket, J5 Conn_01x06_Pin, J6 Conn_01x04_Socket, J7 Conn_01x08_Pin

Commit message: new file:   kicad/teensy2 -top/teensy2-top.kicad_pcb
Parts:
- removed J6: Conn_01x04_Socket, Connector_PinHeader_2.00mm:PinHeader_1x04_P2.00mm_Vertical, symbol Connector:Conn_01x04_Socket
Connections:
- net RX2: no longer names the net of J1.9 (Pin_9)
- net RX3: no longer names the net of J2.12 (Pin_12)
- net RX5: no longer names the net of J2.6 (Pin_6)
- net TX2: no longer names the net of J1.10 (Pin_10)
- net TX3: no longer names the net of J2.13 (Pin_13)
- net TX5: no longer names the net of J2.7 (Pin_7)
Other:
- note removed: "COMMS"
Changed lines of the file:
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@@
-		)
-	)
-	(text "COMMS"
-		(exclude_from_sim no)
-		(at 167.386 109.474 0)
-		(effects
-			(font
-				(size 1.27 1.27)
-			)
 		)
 	)
@@
 	(wire
 		(pts
-			(xy 162.56 101.6) (xy 167.64 101.6)
-		)
-		(stroke
-			(width 0)
-			(type default)
-		)
-	)
-	(wire
-		(pts
-			(xy 162.56 106.68) (xy 167.64 106.68)
-		)
-		(stroke
-			(width 0)
-			(type default)
-		)
-	)
-	(wire
-		(pts
 			(xy 168.91 81.28) (xy 173.99 81.28)
 		)
@@
 	(wire
 		(pts
-			(xy 162.56 104.14) (xy 167.64 104.14)
-		)
-		(stroke
-			(width 0)
-			(type default)
-		)
-	)
-	(wire
-		(pts
 			(xy 81.28 85.09) (xy 87.63 85.09)
 		)
@@
 	(wire
 		(pts
-			(xy 162.56 99.06) (xy 167.64 99.06)
-		)
-		(stroke
-			(width 0)
-			(type default)
-		)
-	)
-	(wire
-		(pts
 			(xy 91.44 109.22) (xy 96.52 109.22)
 		)
@@
 			(width 0)
 			(type default)
-		)
-	)
-	(label "RX5"
-		(at 119.38 111.76 0)
-		(effects
-			(font
-				(size 1.27 1.27)
-			)
-			(justify left bottom)
 		)
 	)
@@
 		)
 	)
-	(label "TX5"
-		(at 119.38 114.3 0)
-		(effects
-			(font
-				(size 1.27 1.27)
-			)
-			(justify left bottom)
-		)
-	)
-	(label "RX2"
-		(at 91.44 119.38 0)
-		(effects
-			(font
-				(size 1.27 1.27)
-			)
-			(justify left bottom)
-		)
-	)
 	(label "GND"
 		(at 92.71 99.06 0)
@@
 		)
 	)
-	(label "TX"
-		(at 163.83 99.06 0)
-		(effects
-			(font
-				(size 1.27 1.27)
-			)
-			(justify left bottom)
-		)
-	)
 	(label "GND"
 		(at 120.65 101.6 0)
@@
 		)
 	)
-	(label "5V"
-		(at 163.83 106.68 0)
-		(effects
-			(font
-				(size 1.27 1.27)
-			)
-			(justify left bottom)
-		)
-	)
 	(label "MISO"
 		(at 91.44 132.08 0)
@@
 		)
 	)
-	(label "TX3"
-		(at 119.38 129.54 0)
-		(effects
-			(font
-				(size 1.27 1.27)
-			)
-			(justify left bottom)
-		)
-	)
 	(label "VBAT"
 		(at 168.91 76.2 0)
@@
 		)
 	)
-	(label "RX"
-		(at 163.83 101.6 0)
-		(effects
-			(font
-				(size 1.27 1.27)
-			)
-			(justify left bottom)
-		)
-	)
 	(label "SCL1"
 		(at 81.28 69.85 0)
@@
 		)
 	)
-	(label "GND"
-		(at 163.83 104.14 0)
-		(effects
-			(font
-				(size 1.27 1.27)
-			)
-			(justify left bottom)
-		)
-	)
 	(label "5V"
 		(at 120.65 99.06 0)
@@
 		)
 	)
-	(label "TX2"
-		(at 91.44 121.92 0)
-		(effects
-			(font
-				(size 1.27 1.27)
-			)
-			(justify left bottom)
-		)
-	)
 	(label "3V3"
 		(at 140.97 104.14 0)
@@
 	(label "SDA1"
 		(at 119.38 121.92 0)
-		(effects
-			(font
-				(size 1.27 1.27)
-			)
-			(justify left bottom)
-		)
-	)
-	(label "RX3"
-		(at 119.38 127 0)
 		(effects
 			(font
@@
 					(unit 1)
 				)
-			)
-		)
-	)
-	(symbol
-		(lib_id "Connector:Conn_01x04_Socket")
-		(at 172.72 101.6 0)
-		(unit 1)
-		(exclude_from_sim no)
-		(in_bom yes)
-		(on_board yes)
-		(dnp no)
-		(fields_autoplaced yes)
-		(property "Reference" "J6"
-			(at 173.99 101.5999 0)
-			(effects
-				(font
-					(size 1.27 1.27)
-				)
-				(justify left)
-				(hide yes)
-			)
-		)
-		(property "Value" "Conn_01x04_Socket"
-			(at 173.99 104.1399 0)
-			(effects
-				(font
-					(size 1.27 1.27)
-				)
-				(justify left)
-				(hide yes)
-			)
-		)
-		(property "Footprint" "Connector_PinHeader_2.00mm:PinHeader_1x04_P2.00mm_Vertical"
-			(at 172.72 101.6 0)
-			(effects
-				(font
-					(size 1.27 1.27)
-				)
-				(hide yes)
-			)
-		)
-		(property "Datasheet" "~"
-			(at 172.72 101.6 0)
-			(effects
-				(font
-					(size 1.27 1.27)
-				)
-				(hide yes)
-			)
-		)
-		(property "Description" "Generic connector, single row, 01x04, script generated"
-			(at 172.72 101.6 0)
-			(effects
-				(font
-					(size 1.27 1.27)
-				)
-				(hide yes)
-			)
-		)
-		(pin "2"
-		)
-		(pin "1"
-		)
-		(pin "3"
-		)
-		(pin "4"
-		)
-		(instances
-			(project ""
-				(path "/2b1f0318-b347-4cb8-9bbf-78e69ec66761"
-					(reference "J6")
-					(unit 1)
-				)

Commit message: modified:   kicad/teensy2-bottom/teensy2-bottom.kicad_pcb
Connections:
- net M1: now also J2.6 (Pin_6)
- net M2: now also J2.7 (Pin_7)
- net M3: now also J2.12 (Pin_12)
- net M4: now also J2.13 (Pin_13)
- net SCL0: now also J7.2 (Pin_2); no longer J3.1 (Pin_1)
- net SCL1: now also J3.1 (Pin_1); no longer J7.2 (Pin_2)
- net SDA0: now also J7.1 (Pin_1); no longer J3.2 (Pin_2)
- net SDA1: now also J3.2 (Pin_2); no longer J7.1 (Pin_1)
- net Rin: now reaches J2.4 (Pin_4)
Changed lines of the file:
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@@
+		)
+	)
+	(label "M1"
+		(at 120.65 111.76 0)
+		(effects
+			(font
+				(size 1.27 1.27)
+			)
+			(justify left bottom)
+		)
+	)
+	(label "SDA0"
+		(at 119.38 119.38 0)
+		(effects
+			(font
+				(size 1.27 1.27)
+			)
+			(justify left bottom)
 		)
 	)
@@
 		)
 	)
+	(label "M4"
+		(at 119.38 129.54 0)
+		(effects
+			(font
+				(size 1.27 1.27)
+			)
+			(justify left bottom)
+		)
+	)
 	(label "CS"
 		(at 91.44 127 0)
@@
 		)
 	)
+	(label "SCL0"
+		(at 81.28 69.85 0)
+		(effects
+			(font
+				(size 1.27 1.27)
+			)
+			(justify left bottom)
+		)
+	)
 	(label "CS"
 		(at 81.28 77.47 0)
@@
 		)
 	)
+	(label "SCL1"
+		(at 140.97 96.52 0)
+		(effects
+			(font
+				(size 1.27 1.27)
+			)
+			(justify left bottom)
+		)
+	)
 	(label "MISO"
 		(at 91.44 132.08 0)
@@
 		)
 	)
-	(label "SDA0"
-		(at 119.38 119.38 0)
-		(effects
-			(font
-				(size 1.27 1.27)
-			)
-			(justify left bottom)
-		)
-	)
-	(label "SCL1"
-		(at 81.28 69.85 0)
+	(label "SDA1"
+		(at 140.97 99.06 0)
 		(effects
 			(font
@@
 		)
 	)
-	(label "SCL0"
-		(at 140.97 96.52 0)
-		(effects
-			(font
-				(size 1.27 1.27)
-			)
-			(justify left bottom)
-		)
-	)
 	(label "GND"
 		(at 140.97 101.6 0)
+		(effects
+			(font
+				(size 1.27 1.27)
+			)
+			(justify left bottom)
+		)
+	)
+	(label "Rin"
+		(at 120.65 106.68 0)
 		(effects
 			(font
@@
 		)
 	)
+	(label "M3"
+		(at 119.38 127 0)
+		(effects
+			(font
+				(size 1.27 1.27)
+			)
+			(justify left bottom)
+		)
+	)
+	(label "SDA0"
+		(at 81.28 67.31 0)
+		(effects
+			(font
+				(size 1.27 1.27)
+			)
+			(justify left bottom)
+		)
+	)
 	(label "3V3"
 		(at 140.97 104.14 0)
@@
 		)
 	)
-	(label "SDA0"
-		(at 140.97 99.06 0)
-		(effects
-			(font
-				(size 1.27 1.27)
-			)
-			(justify left bottom)
-		)
-	)
 	(label "GND"
 		(at 168.91 73.66 0)
@@
 		)
 	)
-	(label "SDA1"
-		(at 81.28 67.31 0)
-		(effects
-			(font
+	(label "M2"
+		(at 120.65 114.3 0)
+		(effects
+			(font
