File: kicad/main/main.kicad_sch (KiCad schematic)
At the start: 13 parts, among them J1 Conn_01x14, J2 Conn_01x14_Socket, J4 Conn_01x03_Socket, J5 Conn_01x06, J6 Conn_01x08, J7 Conn_01x07, J8 Conn_01x09

Commit message: modified:   kicad/main/main.kicad_pcb
Connections:
- net 3V3: now also J6.1 (Pin_1); no longer J6.8 (Pin_8)
- net CS: now also J6.7 (Pin_7); no longer J6.4 (Pin_4)
- net GND: now also J6.2 (Pin_2); no longer J6.7 (Pin_7)
- net MISO: now also J6.5 (Pin_5); no longer J6.2 (Pin_2)
- net MOSI: now also J6.6 (Pin_6); no longer J6.3 (Pin_3)
- net SCK: now also J6.8 (Pin_8); no longer J6.1 (Pin_1)
- net SCL1: now also J6.4 (Pin_4); no longer J6.5 (Pin_5)
- net SDA1: now also J6.3 (Pin_3); no longer J6.6 (Pin_6)
Changed lines of the file:
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@@
 		)
 	)
-	(label "MISO"
+	(label "GND"
 		(at 50.8 123.19 0)
 		(effects
@@
 		)
 	)
-	(label "SCK"
+	(label "3V3"
 		(at 50.8 120.65 0)
 		(effects
@@
 		)
 	)
-	(label "SDA1"
+	(label "MOSI"
 		(at 50.8 133.35 0)
 		(effects
@@
 		)
 	)
-	(label "3V3"
+	(label "SCK"
 		(at 50.8 138.43 0)
 		(effects
@@
 		)
 	)
-	(label "MOSI"
+	(label "SDA1"
 		(at 50.8 125.73 0)
 		(effects
@@
 		)
 	)
-	(label "CS"
+	(label "SCL1"
 		(at 50.8 128.27 0)
 		(effects
@@
 		)
 	)
-	(label "SCL1"
+	(label "MISO"
 		(at 50.8 130.81 0)
 		(effects
@@
 		)
 	)
-	(label "GND"
+	(label "CS"
 		(at 50.8 135.89 0)
 		(effects
