File: kicad/smd/smd.kicad_sch (KiCad schematic)
At the start: 13 parts, among them J1 Conn_01x14, J2 Conn_01x14_Socket, J4 Conn_01x03_Socket, J5 Conn_01x06, J6 Conn_01x08, J7 Conn_01x07, J8 Conn_01x09

Commit message: modified:   kicad/smd/smd.kicad_pcb
Parts:
- removed J7: Conn_01x07, Connector_PinHeader_1.27mm:PinHeader_1x07_P1.27mm_Vertical, symbol Connector_Generic:Conn_01x07
- removed J8: Conn_01x09, Connector_PinHeader_1.27mm:PinHeader_1x09_P1.27mm_Vertical, symbol Connector_Generic:Conn_01x09
- added C1: C, Capacitor_SMD:C_0603_1608Metric, symbol Device:C
- added U1: BMI088, Package_LGA:Bosch_LGA-16_4.5x3mm_P0.5mm_LayoutBorder7x1y_ClockwisePinNumbering, symbol Sensor_Motion:BMI088
- D1: footprint LED_THT:LED_D3.0mm_FlatTop -> LED_SMD:LED_0603_1608Metric
- R1: footprint Resistor_THT:R_Axial_DIN0204_L3.6mm_D1.6mm_P7.62mm_Horizontal -> Resistor_SMD:R_0603_1608Metric
Connections:
- net 3V3: now also C1.2, U1.3 (VDD), U1.7 (PS)
- net GND: now also C1.1, U1.10 (SDO2), U1.15 (SDO1), U1.2 (GNDA), U1.4 (GNDA), U1.6 (GNDIO)
- net SCL0: now also U1.8 (SCK/SCL)
- net SDA0: now also U1.9 (SDI/SDA)

Commit message: modified:   kicad/hover/hover.kicad_pcb, kicad/smd/smd.kicad_pcb
Connections:
- net 3V3: now also J6.1 (Pin_1); no longer J6.8 (Pin_8)
- net CS: now also J6.7 (Pin_7); no longer J6.4 (Pin_4)
- net GND: now also J6.2 (Pin_2); no longer J6.7 (Pin_7)
- net MISO: now also J6.5 (Pin_5); no longer J6.2 (Pin_2)
- net MOSI: now also J6.6 (Pin_6); no longer J6.3 (Pin_3)
- net SCK: now also J6.8 (Pin_8); no longer J6.1 (Pin_1)
- net SCL1: now also J6.4 (Pin_4); no longer J6.5 (Pin_5)
- net SDA1: now also J6.3 (Pin_3); no longer J6.6 (Pin_6)
Changed lines of the file:
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@@
 		)
 	)
-	(label "MISO"
+	(label "GND"
 		(at 50.8 123.19 0)
 		(effects
@@
 		)
 	)
-	(label "SCK"
-		(at 50.8 120.65 0)
-		(effects
-			(font
-				(size 1.27 1.27)
-			)
-			(justify left bottom)
-		)
-	)
 	(label "MISO"
 		(at 91.44 132.08 0)
@@
 		)
 	)
-	(label "SDA1"
+	(label "MOSI"
 		(at 50.8 133.35 0)
 		(effects
@@
 		)
 	)
-	(label "3V3"
+	(label "SCK"
 		(at 50.8 138.43 0)
 		(effects
@@
 		)
 	)
-	(label "MOSI"
+	(label "SDA1"
 		(at 50.8 125.73 0)
 		(effects
@@
 		)
 	)
-	(label "CS"
+	(label "SCL1"
 		(at 50.8 128.27 0)
 		(effects
@@
 		)
 	)
-	(label "SCL1"
+	(label "MISO"
 		(at 50.8 130.81 0)
 		(effects
@@
 		)
 	)
-	(label "GND"
+	(label "CS"
 		(at 50.8 135.89 0)
 		(effects
 			(font
+				(size 1.27 1.27)
+			)
+			(justify left bottom)
+		)
+	)
+	(label "3V3"
+		(at 50.8 120.65 0)
+		(effects
+			(font

Commit message: modified:   kicad/smd/smd.kicad_pcb
Parts:
- removed H1, H2, H3, H4: MountingHole, MountingHole:MountingHole_2.5mm, symbol Mechanical:MountingHole
