File: kicad/2-inch-Apex-frame/main.kicad_sch (KiCad schematic)
At the start: 13 parts, among them J1 Conn_01x14, J2 Conn_01x14_Socket, J4 Conn_01x03_Socket, J5 Conn_01x06, J6 Conn_01x08, J7 Conn_01x07, J8 Conn_01x09

Commit message: modified:   kicad/2-inch-Apex-frame/main.kicad_pcb
Parts:
- H1, H2, H3, H4: footprint MountingHole:MountingHole_2.5mm -> MountingHole:MountingHole_2.1mm
