File: kicad/apex-main/main.kicad_pcb (KiCad board)
At the start: 2 copper layers, 41 x 55.5 mm, 17 parts, among them J1 Conn_01x14, J2 Conn_01x14_Socket, J4 Conn_01x03_Socket, J5 Conn_01x06, J6 Conn_01x08, J7 Conn_01x07, J8 Conn_01x09

Commit message: new file:   pcb.png
Parts:
- removed G***: LOGO, Logo:logo
Other:
- board text added: "BMI088"
- board text added: "Teensy 4.0"
- board text added: "To ESC"
- board text added: "To HoverDeck"
