File: kicad/hover-jst/hover.kicad_pcb (KiCad board)
At the start: 2 copper layers, 25.6 x 27 mm, 8 parts, among them J1 Conn_01x07_Socket, J2 Conn_01x07_Socket, J3 Conn_01x02_Socket, J4 Conn_01x08_Socket

Commit message: modified:   kicad/hover-jst/hover.kicad_pcb
Parts:
- J4: footprint Connector_JST:JST_SHL_SM08B-SHLS-TF_1x08-1MP_P1.00mm_Horizontal -> Connector_JST:JST_ZH_B8B-ZR_1x08_P1.50mm_Vertical
- moved J4 5.07 mm to (141.1, 95.4)
Routing:
- net /3V3: track 22.3 -> 25.2 mm
- net /SDA: track 6.70 -> 9.42 mm
- net /GND: track 23.2 -> 25.9 mm
- net /SCL: track 8.60 -> 11.1 mm
- net /CS: track 14.5 -> 17.0 mm
- net /SCK: track 19.9 -> 22.2 mm
- net /MOSI: track 17.5 -> 19.8 mm
- net /MISO: track 20.5 -> 22.6 mm
Other:
- board text added: "GND"
- board text added: "MISO"
- board text added: "MOSI"
- board text removed: "GD"
- board text removed: "SI"
- board text removed: "SO"
