File: kicad/main-tinypico/main.kicad_pcb (KiCad board)
At the start: 2 copper layers, 41 x 48 mm, 16 parts, among them J1 Conn_01x14, J2 Conn_01x14_Socket, J3 Conn_01x04_Socket, J4 Conn_01x03_Socket, J5 Conn_01x06, J6 Conn_01x08, J8 Conn_01x07, J9 Conn_01x07

Commit message: modified:   kicad/main-tinypico/main.kicad_pcb
Parts:
- added J10: Conn_01x01_Pin, Connector_Wire:SolderWirePad_1x01_SMD_1x2mm, F.Cu at (152.6, 81.2)
- added J11: Conn_01x01_Pin, Connector_Wire:SolderWirePad_1x01_SMD_1x2mm, F.Cu at (152.6, 83.8)
- added J12: Conn_01x01_Pin, Connector_Wire:SolderWirePad_1x01_SMD_1x2mm, F.Cu at (152.6, 86.3)
- added J13: Conn_01x01_Pin, Connector_Wire:SolderWirePad_1x01_SMD_1x2mm, F.Cu at (152.6, 88.9)
- added J7: Conn_01x01_Pin, Connector_Wire:SolderWirePad_1x01_SMD_1x2mm, F.Cu at (137.6, 81.2)
- added U1: TinyPICO_Nano, footprints:TinyPICO_Nano, B.Cu at (159.4, 90.8)
- J3: value Conn_01x04_Socket -> Conn_01x01_Pin; footprint Connector_PinHeader_2.54mm:PinHeader_1x04_P2.54mm_Vertical -> Connector_Wire:SolderWirePad_1x01_SMD_1x2mm
- J8, J9: value Conn_01x07 -> Conn_01x01_Pin; footprint Connector_PinHeader_2.54mm:PinHeader_1x07_P2.54mm_Vertical -> Connector_Wire:SolderWirePad_1x01_SMD_1x2mm
- moved H3 26.5 mm to (155.0, 70.9)
- moved J8 24.8 mm to (137.6, 86.3), turned to -90 degrees
- moved H2 19.3 mm to (147.1, 84.5)
- moved H4 17.8 mm to (126.9, 68.7)
- moved R2 12.7 mm to (158.4, 70.2), turned to 180 degrees
- moved R3 11.5 mm to (154.5, 72.8)
- moved J3 11.3 mm to (137.6, 83.8), turned to 90 degrees
- moved J9 6.98 mm to (137.6, 88.9), turned to -90 degrees
- moved J6 2.64 mm to (138.2, 97.8)
- moved J4 2.53 mm to (155.4, 89.7)
- moved H1 1.39 mm to (143.9, 70.9)
Connections:
- J3 pad 1: /3V3 -> /GND
Routing:
- net /5V: track 37.8 -> 13.9 mm
- net /TX3: track 22.7 -> 0.00 mm
- net /RX3: track 22.7 -> 0.00 mm
- net /A9: track 20.2 -> 28.0 mm
- net /MISO: track 38.7 -> 33.8 mm
- net /MOSI: track 28.8 -> 25.4 mm
- net /SCL1: track 19.5 -> 16.7 mm
- net /SDA1: track 19.8 -> 17.0 mm
- net /VBAT: track 36.8 -> 34.7 mm
- net /SDA0: track 13.3 -> 14.9 mm, vias 0 -> 2
- net /CS: track 32.4 -> 30.9 mm
- net /3V3: track 43.4 -> 44.7 mm, vias 0 -> 1
- net /GND: track 78.9 -> 80.2 mm, vias 0 -> 1
- net /SCK: track 23.7 -> 22.7 mm
- net /SCL0: track 13.3 -> 12.4 mm
Other:
- board size 41 x 48 mm -> 41 x 41.5 mm
- board text removed: "Teensy4"
- board text removed: "Xiao ESP32"
