File: kicad/main-xiao-bottom/main.kicad_pcb (KiCad board)
At the start: 2 copper layers, 41 x 41.5 mm, 22 parts, among them J1 Conn_01x14, J10 Conn_01x01_Pin, J11 Conn_01x01_Pin, J12 Conn_01x01_Pin, J13 Conn_01x01_Pin, J2 Conn_01x14_Socket, J3 Conn_01x01_Pin, J4 Conn_01x03_Socket, J5 Conn_01x06, J6 Conn_01x08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

Commit message: modified:   kicad/main-xiao-bottom/main.kicad_pcb
Parts:
- removed U1: TinyPICO_Nano, footprints:TinyPICO_Nano
- added J14: Conn_01x05_Socket, Connector_PinHeader_2.54mm:PinHeader_1x05_P2.54mm_Vertical, F.Cu at (151.0, 74.2)
- moved J5 3.18 mm to (151.0, 70.1)
- moved R2 0.07 mm to (158.4, 70.2), turned to 150 degrees
Connections:
- J1 pad 10: unconnected-(J1-Pin_10-Pad10) -> /TX2
- J1 pad 9: unconnected-(J1-Pin_9-Pad9) -> /RX2
Routing:
- net /5V: track 13.9 -> 41.8 mm, vias 0 -> 2
- net /GND: track 80.2 -> 95.7 mm
- net /RX2: track 0.00 -> 4.30 mm
- net /TX2: track 0.00 -> 4.30 mm
- net /M2: track 8.86 -> 12.6 mm
- net /M4: track 7.48 -> 11.1 mm
- net /M1: track 8.71 -> 12.0 mm
- net /M3: track 7.78 -> 10.6 mm
- net /A9: track 28.0 -> 29.1 mm
- removed copper zone on F.Cu, net /GND
Other:
- board text added: "RX1"
- board text added: "RX2"
- board text added: "TX1"
- board text added: "TX2"
- board text added: "Xiao"

Commit message: modified:   kicad/main-xiao-bottom/main.kicad_pcb
Parts:
- added G***: LOGO, LOGO, F.Cu at (138.1, 102.3)
Other:
- board text added: "tindie.com/stores/bobbiebots"

Commit message: modified:   webots/protos/SevJr.proto
Parts:
- moved G*** 15.4 mm to (153.4, 102.2)
Changed lines of the file:
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@@
 	(footprint "LOGO"
 		(layer "F.Cu")
-		(at 138.05 102.35)
+		(at 153.43 102.2)
 		(property "Reference" "G***"
 			(at 0 0 0)
@@
 	)
 	(gr_text "tindie.com/stores/bobbiebots"
-		(at 140.9 101.25 0)
+		(at 155.86 103.9 49)
 		(layer "F.SilkS")
 		(effects
@@
 	)
 	(gr_text "5V"
-		(at 162.65 95.75 90)
+		(at 164.11 93.64 90)
 		(layer "F.SilkS")
 		(effects

Commit message: modified:   webots/protos/SevJr.proto
Parts:
- moved G*** 0.78 mm to (152.7, 102.2)

Commit message: modified:   kicad/main-xiao-bottom/main.kicad_pcb
Parts:
- moved G*** 14.7 mm to (138.0, 102.2)

Commit message: modified:   kicad/main-xiao-bottom/main.kicad_pcb
Parts:
- moved J10 0.63 mm to (152.0, 81.2)
- moved J12 0.63 mm to (152.0, 86.3)
- moved J13 0.63 mm to (152.0, 88.9)
- moved J3 0.37 mm to (138.0, 83.8)
- moved J7 0.37 mm to (138.0, 81.2)
- moved J8 0.37 mm to (138.0, 86.3)
- moved J9 0.37 mm to (138.0, 88.9)
Changed lines of the file:
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@@
 	(footprint "Connector_Wire:SolderWirePad_1x01_SMD_1x2mm"
 		(layer "F.Cu")
-		(at 152.63 81.25 -90)
+		(at 152 81.25 -90)
 		(descr "Wire Pad, Square, SMD Pad,  1mm x 2mm")
 		(tags "MeasurementPoint Square SMDPad 1mmx2mm ")
@@
 	(footprint "Connector_Wire:SolderWirePad_1x01_SMD_1x2mm"
 		(layer "F.Cu")
-		(at 152.63 88.87 -90)
+		(at 152 88.87 -90)
 		(descr "Wire Pad, Square, SMD Pad,  1mm x 2mm")
 		(tags "MeasurementPoint Square SMDPad 1mmx2mm ")
@@
 	(footprint "Connector_Wire:SolderWirePad_1x01_SMD_1x2mm"
 		(layer "F.Cu")
-		(at 137.63 83.79 90)
+		(at 138 83.79 90)
 		(descr "Wire Pad, Square, SMD Pad,  1mm x 2mm")
 		(tags "MeasurementPoint Square SMDPad 1mmx2mm ")
@@
 	(footprint "Connector_Wire:SolderWirePad_1x01_SMD_1x2mm"
 		(layer "F.Cu")
-		(at 137.63 81.25 -90)
+		(at 138 81.25 -90)
 		(descr "Wire Pad, Square, SMD Pad,  1mm x 2mm")
 		(tags "MeasurementPoint Square SMDPad 1mmx2mm ")
@@
 		)
 		(pad "1" smd roundrect
-			(at 0 0 270)
+			(at 0 0.63 270)
 			(size 1 2)
 			(layers "F.Cu" "F.Mask")
@@
 	(footprint "Connector_Wire:SolderWirePad_1x01_SMD_1x2mm"
 		(layer "F.Cu")
-		(at 137.63 88.87 -90)
+		(at 138 88.87 -90)
 		(descr "Wire Pad, Square, SMD Pad,  1mm x 2mm")
 		(tags "MeasurementPoint Square SMDPad 1mmx2mm ")
@@
 	(footprint "Connector_Wire:SolderWirePad_1x01_SMD_1x2mm"
 		(layer "F.Cu")
-		(at 137.63 86.33 -90)
+		(at 138 86.33 -90)
 		(descr "Wire Pad, Square, SMD Pad,  1mm x 2mm")
 		(tags "MeasurementPoint Square SMDPad 1mmx2mm ")
@@
 	(footprint "Connector_Wire:SolderWirePad_1x01_SMD_1x2mm"
 		(layer "F.Cu")
-		(at 152.63 86.33 -90)
+		(at 152 86.33 -90)
 		(descr "Wire Pad, Square, SMD Pad,  1mm x 2mm")
 		(tags "MeasurementPoint Square SMDPad 1mmx2mm ")
@@
 	)
 	(segment
-		(start 144.145 92.275)
-		(end 144.145 92.725)
+		(start 144.145 91.645)
+		(end 152 83.79)
 		(width 0.2)
 		(layer "F.Cu")
@@
 	)
 	(segment
-		(start 152.63 83.79)
-		(end 144.145 92.275)
+		(start 144.145 92.725)
+		(end 144.145 91.645)
 		(width 0.2)
 		(layer "F.Cu")

Commit message: modified:   kicad/main-xiao-bottom/main.kicad_pcb
Routing:
- added copper zone on F.Cu, net /GND
Changed lines of the file:
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@@
 		(net "/SDA0")
+	)
+	(zone
+		(net "/GND")
+		(layer "F.Cu")
+		(hatch edge 0.5)
+		(connect_pads
+			(clearance 0.5)
+		)
+		(min_thickness 0.25)
+		(fill yes
+			(thermal_gap 0.5)
+			(thermal_bridge_width 0.5)
+			(island_removal_mode 0)
+		)
+		(polygon
+			(pts
+				(xy 135.06 64.55) (xy 155.01 64.55) (xy 166.02 74.01) (xy 166.28 93.95) (xy 155.79 105.84) (xy 135.58 105.84)
+				(xy 125 93.87) (xy 125 74.18) (xy 135.13 64.53)
+			)
+		)
 	)
 	(embedded_fonts no)
