File: kicad/fc-41/main.kicad_sch (KiCad schematic)
At the start: 26 parts, among them J1 Conn_01x14, J10 Conn_01x01_Pin, J11 Conn_01x01_Pin, J12 Conn_01x01_Pin, J13 Conn_01x01_Pin, J14 Conn_01x01_Pin, J15 Conn_01x02, J16 Conn_01x04, J17 Conn_01x01_Pin, J18 Conn_01x01_Pin, J2 Conn_01x14_Socket, J3 Conn_01x01_Pin, J4 Conn_01x03_Socket, J5 Conn_01x01_Pin, J6 Conn_01x08, J7 Conn_01x01_Pin, J8 Conn_01x01_Pin, J9 Conn_01x01_Pin

Commit message: modified:   kicad/fc-41/main.kicad_pcb
Parts:
- removed J15: Conn_01x02, Connector_PinSocket_2.00mm:PinSocket_1x02_P2.00mm_Vertical, symbol Connector_Generic:Conn_01x02
- removed J16: Conn_01x04, Connector_PinSocket_2.00mm:PinSocket_1x04_P2.00mm_Vertical, symbol Connector_Generic:Conn_01x04
- added J19: Conn_01x06, Connector_PinSocket_2.00mm:PinSocket_1x06_P2.00mm_Vertical, symbol Connector_Generic:Conn_01x06
Connections:
- net GND: now also J19.1 (Pin_1)
- net M1: now also J19.3 (Pin_3)
- net M2: now also J19.4 (Pin_4)
- net M3: now also J19.5 (Pin_5)
- net M4: now also J19.6 (Pin_6)
- net VBAT: now also J19.2 (Pin_2)
- net A9 renamed DIV

Commit message: modified:   kicad/fc-41/main.kicad_pcb
Parts:
- added J16, J20: Conn_01x03_Socket, Connector_PinHeader_2.54mm:PinHeader_1x03_P2.54mm_Vertical, symbol Connector:Conn_01x03_Socket
Connections:
- net RX3: no longer names the net of J2.12 (Pin_12)
- net RX3: no longer J17.1 (Pin_1)
- net TX3: no longer names the net of J2.13 (Pin_13)
- net TX3: no longer J18.1 (Pin_1)
- new net RX8: J18.1 (Pin_1), J20.3 (Pin_3)
- new net TX8: J17.1 (Pin_1), J20.2 (Pin_2)
