File: kicad/tx/tx.kicad_sch (KiCad schematic)
At the start: 34 parts, among them J10 Conn_01x01_Pin, J11 Conn_01x01_Pin, J12 Conn_01x01_Pin, J13 Conn_01x01_Pin, J14 Conn_01x01_Pin, J15 Conn_01x01_Pin, J16 Conn_01x01_Pin, J17 Conn_01x01_Pin, J18 Conn_01x01_Pin, J20 Conn_01x01_Pin, J22 Conn_01x01_Pin, J24 Conn_01x01_Pin, J25 Conn_01x01_Pin, J26 Conn_01x01_Pin, J27 Conn_01x01_Pin, J28 Conn_01x01_Pin, J29 Conn_01x01_Pin, J30 Conn_01x01_Pin, J31 Conn_01x01_Pin, J4 Conn_01x04_Socket, J5 Conn_01x01_Pin, J6 Conn_01x01_Pin, J7 Conn_01x01_Pin, J8 Conn_01x01_Pin, J9 Conn_01x01_Pin, U1 NanoS3

Commit message: modified:   kicad/tx/tx.kicad_pcb
Connections:
- net 3V3: no longer J24.1 (Pin_1), J26.1 (Pin_1)
- net GND: now also J24.1 (Pin_1), J26.1 (Pin_1)
Changed lines of the file:
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@@
 		)
 	)
-	(label "3V3"
+	(label "GND"
 		(at 102.87 143.51 0)
 		(effects
@@
 		)
 	)
-	(label "3V3"
+	(label "GND"
 		(at 119.38 143.51 0)
 		(effects

Commit message: modified:   kicad/tx/tx.kicad_pro
Connections:
- net A0_YAW: now reaches U1.33 (IO1)
- net A0_YAW: now also J16.1 (Pin_1)
- net ARM: no longer names the net of J18.1 (Pin_1)
- net AUT renamed D8_AUT
- net DIV renamed A4_DIV
- net A4_DIV: now also U1.22 (IO5); no longer U1.36 (IO4)
- net HOV renamed D9_HOV
- net PIT renamed A1_THR
- net A1_THR: now also J13.1 (Pin_1); no longer J15.1 (Pin_1)
- net ROL renamed A2_ROL
- removed net THR: J13.1 (Pin_1), U1.22 (IO5)
- net YAW: no longer names the net of U1.21 (IO6)
- net YAW: no longer J16.1 (Pin_1)
- new net A3_PIT: J15.1 (Pin_1), U1.36 (IO4)

Commit message: modified:   kicad/tx/tx.kicad_pcb
Parts:
- removed J28, J29, J30, J31: Conn_01x01_Pin, Connector_PinSocket_2.54mm:PinSocket_1x01_P2.54mm_Vertical, symbol Connector:Conn_01x01_Pin
Connections:
- net D35_ARM: now also J18.1 (Pin_1), U1.23 (IO35)
- net D8_AUT: now also U1.28 (IO8)
- net D9_HOV: now also U1.27 (IO9)

Commit message: modified:   kicad/tx/tx.kicad_pcb
Connections:
- net LED renamed D33_LED
Changed lines of the file:
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@@
+	(wire
+		(pts
+			(xy 161.29 127) (xy 170.18 127)
+		)
+		(stroke
+			(width 0)
+			(type default)
+		)
+	)
 	(wire
 		(pts
@@
 	(wire
 		(pts
-			(xy 163.83 127) (xy 170.18 127)
-		)
-		(stroke
-			(width 0)
-			(type default)
-		)
-	)
-	(wire
-		(pts
 			(xy 87.63 142.24) (xy 92.71 142.24)
 		)
@@
 	(wire
 		(pts
-			(xy 137.16 77.47) (xy 142.24 77.47)
+			(xy 137.16 77.47) (xy 147.32 77.47)
 		)
 		(stroke
@@
 		)
 	)
-	(label "LED"
-		(at 163.83 127 0)
-		(effects
-			(font
-				(size 1.27 1.27)
-			)
-			(justify left bottom)
-		)
-	)
 	(label "D-"
 		(at 139.7 134.62 0)
@@
 		)
 	)
+	(label "D33_LED"
+		(at 137.16 77.47 0)
+		(effects
+			(font
+				(size 1.27 1.27)
+			)
+			(justify left bottom)
+		)
+	)
 	(label "VBAT"
 		(at 180.34 77.47 0)
@@
 		)
 	)
-	(label "LED"
-		(at 137.16 77.47 0)
-		(effects
-			(font
-				(size 1.27 1.27)
-			)
-			(justify left bottom)
-		)
-	)
 	(label "GND"
 		(at 119.38 143.51 0)
 		(effects
 			(font
+				(size 1.27 1.27)
+			)
+			(justify left bottom)
+		)
+	)
+	(label "D33_LED"
+		(at 162.56 127 0)
+		(effects
+			(font

Commit message: modified:   kicad/tx/tx.kicad_pcb
Connections:
- net 3V3: no longer J17.1 (Pin_1)
- net GND: now also J17.1 (Pin_1)
- net A5_ARM: now reaches U1.21 (IO6)
- net A5_ARM: now also J18.1 (Pin_1)
- net D35_ARM: no longer names the net of U1.23 (IO35)
- net D35_ARM: no longer J18.1 (Pin_1)
- net D8_AUT renamed A7_AUT
- net D9_HOV renamed A8_HOV
Changed lines of the file:
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@@
+	(wire
+		(pts
+			(xy 200.66 139.7) (xy 205.74 139.7)
+		)
+		(stroke
+			(width 0)
+			(type default)
+		)
+	)
 	(wire
 		(pts
@@
 	(wire
 		(pts
-			(xy 48.26 118.11) (xy 53.34 118.11)
+			(xy 49.53 118.11) (xy 54.61 118.11)
 		)
 		(stroke
@@
 	(wire
 		(pts
-			(xy 160.02 109.22) (xy 170.18 109.22)
-		)
-		(stroke
-			(width 0)
-			(type default)
-		)
-	)
-	(wire
-		(pts
 			(xy 163.83 77.47) (xy 172.72 77.47)
 		)
@@
 			(width 0)
 			(type default)
+		)
+	)
+	(label "GND"
+		(at 49.53 123.19 0)
+		(effects
+			(font
+				(size 1.27 1.27)
+			)
+			(justify left bottom)
 		)
 	)
@@
 		)
 	)
-	(label "D9_HOV"
-		(at 119.38 147.32 0)
-		(effects
-			(font
-				(size 1.27 1.27)
-			)
-			(justify left bottom)
-		)
-	)
 	(label "GND"
 		(at 114.3 77.47 0)
@@
 		)
 	)
-	(label "D9_HOV"
-		(at 162.56 119.38 0)
+	(label "A5_ARM"
+		(at 49.53 118.11 0)
 		(effects
 			(font
@@
 		)
 	)
+	(label "A7_AUT"
+		(at 162.56 121.92 0)
+		(effects
+			(font
+				(size 1.27 1.27)
+			)
+			(justify left bottom)
+		)
+	)
 	(label "GND"
 		(at 152.4 77.47 0)
@@
 		)
 	)
-	(label "D8_AUT"
-		(at 33.02 123.19 0)
+	(label "A8_HOV"
+		(at 162.56 119.38 0)
 		(effects
 			(font
@@
 		)
 	)
-	(label "D35_ARM"
-		(at 160.02 109.22 0)
-		(effects
-			(font
-				(size 1.27 1.27)
-			)
-			(justify left bottom)
-		)
-	)
-	(label "D35_ARM"
-		(at 48.26 118.11 0)
-		(effects
-			(font
-				(size 1.27 1.27)
-			)
-			(justify left bottom)
-		)
-	)
 	(label "A1_THR"
 		(at 87.63 149.86 0)
@@
 		)
 	)
+	(label "A7_AUT"
+		(at 33.02 123.19 0)
+		(effects
+			(font
+				(size 1.27 1.27)
+			)
+			(justify left bottom)
+		)
+	)
+	(label "A8_HOV"
+		(at 119.38 147.32 0)
+		(effects
+			(font
+				(size 1.27 1.27)
+			)
+			(justify left bottom)
+		)
+	)
 	(label "A0_YAW"
 		(at 86.36 125.73 0)
@@
 		)
 	)
-	(label "D8_AUT"
-		(at 162.56 121.92 0)
-		(effects
-			(font
-				(size 1.27 1.27)
-			)
-			(justify left bottom)
-		)
-	)
 	(label "D+"
 		(at 190.5 96.52 0)
@@
 		)
 	)
+	(label "A5_ARM"
+		(at 201.93 139.7 0)
+		(effects
+			(font
+				(size 1.27 1.27)
+			)
+			(justify left bottom)
+		)
+	)
 	(label "GND"
 		(at 86.36 118.11 0)
-		(effects
-			(font
-				(size 1.27 1.27)
-			)
-			(justify left bottom)
-		)
-	)
-	(label "3V3"
-		(at 49.53 123.19 0)
 		(effects
 			(font
@@
 	(symbol
 		(lib_id "Connector:Conn_01x01_Pin")
-		(at 43.18 118.11 0)
+		(at 44.45 118.11 0)
 		(unit 1)
 		(body_style 1)
@@
 		(fields_autoplaced yes)
 		(property "Reference" "J18"
-			(at 43.815 113.03 0)
+			(at 45.085 113.03 0)
 			(hide yes)
 			(show_name no)
@@
 		)
 		(property "Value" "Conn_01x01_Pin"
-			(at 43.815 115.57 0)
+			(at 45.085 115.57 0)
 			(hide yes)
 			(show_name no)
@@
 		)
 		(property "Footprint" "Connector_Wire:SolderWirePad_1x01_SMD_2x4mm"
-			(at 43.18 118.11 0)
+			(at 44.45 118.11 0)
 			(hide yes)
 			(show_name no)
@@
 		)
 		(property "Datasheet" ""
-			(at 43.18 118.11 0)
+			(at 44.45 118.11 0)
 			(hide yes)
 			(show_name no)
@@
 		)
 		(property "Description" "Generic connector, single row, 01x01, script generated"
-			(at 43.18 118.11 0)
-			(hide yes)
-			(show_name no)
+			(at 44.45 118.11 0)
+			(hide yes)
+			(show_name no)

Commit message: modified:   kicad/tx/tx.kicad_pcb
Connections:
- net A6_YAW: now reaches U1.20 (IO7)
- net A6_YAW: now also J16.1 (Pin_1)
- net A0_YAW: no longer names the net of U1.33 (IO1)
- net A0_YAW: no longer J16.1 (Pin_1)
- net A1_THR renamed A1_ARM
- net A1_ARM: now also J18.1 (Pin_1); no longer J13.1 (Pin_1)
- net A5_ARM renamed A5_THR
- net A5_THR: now also J13.1 (Pin_1); no longer J18.1 (Pin_1)
Changed lines of the file:
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@@
-	(wire
-		(pts
-			(xy 163.83 134.62) (xy 170.18 134.62)
-		)
-		(stroke
-			(width 0)
-			(type default)
-		)
-	)
 	(wire
 		(pts
@@
 		(pts
 			(xy 86.36 125.73) (xy 91.44 125.73)
+		)
+		(stroke
+			(width 0)
+			(type default)
+		)
+	)
+	(wire
+		(pts
+			(xy 200.66 137.16) (xy 205.74 137.16)
 		)
 		(stroke
@@
 		)
 	)
-	(label "A5_ARM"
-		(at 49.53 118.11 0)
-		(effects
-			(font
-				(size 1.27 1.27)
-			)
-			(justify left bottom)
-		)
-	)
-	(label "A1_THR"
+	(label "A1_ARM"
 		(at 163.83 137.16 0)
 		(effects
@@
 		)
 	)
-	(label "A0_YAW"
-		(at 163.83 134.62 0)
-		(effects
-			(font
-				(size 1.27 1.27)
-			)
-			(justify left bottom)
-		)
-	)
 	(label "A8_HOV"
 		(at 162.56 119.38 0)
@@
 		)
 	)
-	(label "A1_THR"
-		(at 87.63 149.86 0)
+	(label "A6_YAW"
+		(at 201.93 137.16 0)
 		(effects
 			(font
@@
 		)
 	)
+	(label "A1_ARM"
+		(at 49.53 118.11 0)
+		(effects
+			(font
+				(size 1.27 1.27)
+			)
+			(justify left bottom)
+		)
+	)
 	(label "A7_AUT"
 		(at 33.02 123.19 0)
@@
 		)
 	)
-	(label "A0_YAW"
-		(at 86.36 125.73 0)
-		(effects
-			(font
-				(size 1.27 1.27)
-			)
-			(justify left bottom)
-		)
-	)
 	(label "VBAT"
 		(at 201.93 109.22 0)
@@
 		)
 	)
+	(label "A5_THR"
+		(at 87.63 149.86 0)
+		(effects
+			(font
+				(size 1.27 1.27)
+			)
+			(justify left bottom)
+		)
+	)
 	(label "5V"
 		(at 139.7 132.08 0)
@@
 		)
 	)
-	(label "A5_ARM"
+	(label "A5_THR"
 		(at 201.93 139.7 0)
 		(effects
@@
 		(effects
 			(font
+				(size 1.27 1.27)
+			)
+			(justify left bottom)
+		)
+	)
+	(label "A6_YAW"
+		(at 86.36 125.73 0)
+		(effects
+			(font

Commit message: modified:   kicad/tx/tx.kicad_pcb
Parts:
- removed J4: Conn_01x04_Socket, Connector_PinSocket_2.54mm:PinSocket_1x04_P2.54mm_Vertical, symbol Connector:Conn_01x04_Socket
- removed U1: NanoS3, um-s3-footprints:NanoS3, symbol NanoS3:NanoS3
- added J1: Conn_01x12_Socket, Connector_PinHeader_2.54mm:PinHeader_1x12_P2.54mm_Vertical, symbol Connector:Conn_01x12_Socket
- added J2: Conn_01x11_Socket, Connector_PinHeader_2.54mm:PinHeader_1x11_P2.54mm_Vertical, symbol Connector:Conn_01x11_Socket
Connections:
- net 3V3: now also J2.4 (Pin_4)
- net 5V: now also J2.3 (Pin_3)
- net GND: now also J1.10 (Pin_10), J2.2 (Pin_2)
- net VBAT: now also J2.1 (Pin_1)
- new net A0: J2.5 (Pin_5)
- new net A1: J2.6 (Pin_6)
- new net A2: J2.7 (Pin_7)
- new net A3: J2.8 (Pin_8)
- new net A4: J2.9 (Pin_9)
- new net A5: J1.8 (Pin_8)
- new net A6: J1.7 (Pin_7)
- new net A7: J1.6 (Pin_6)
- new net A8: J1.5 (Pin_5)
Other:
- note removed: "USB"

Commit message: modified:   kicad/tx/tx.kicad_pcb
Connections:
- net A3 is gone; now on net A3_ROL: J2.8 (Pin_8)
- net A3_PIT is gone; now on net A2_PIT: J15.1 (Pin_1)
- net A5_THR is gone; now on net A4_THR: J13.1 (Pin_1)
- net A6 is gone; now on net A6_DIV: J1.7 (Pin_7)
- net A6_YAW is gone; now on net A1_YAW: J16.1 (Pin_1)
- net A7 is gone; now on net A7_AUT: J1.6 (Pin_6)
- net A8 is gone; now on net A8_ARM: J1.5 (Pin_5)
- net A8_HOV is gone; now on net A0_HOV: J27.1 (Pin_1)
- net D33_LED is gone; now on net LED_HI: R1.2
- net LED_HI: now reaches J2.10 (Pin_10)
- net A0 renamed A0_HOV
- net A1 renamed A1_YAW
- net A1_ARM renamed A8_ARM
- net A2 renamed A2_PIT
- net A2_ROL renamed A3_ROL
- net A4 renamed A4_THR
- net A4_DIV renamed A6_DIV
Other:
- moved on the sheet: J1, J2
