File: kicad/fc/main.kicad_pcb (KiCad board)
At the start: 2 copper layers, 41 x 41.5 mm, 26 parts, among them J1 Conn_01x14, J10 Conn_01x01_Pin, J11 Conn_01x01_Pin, J12 Conn_01x01_Pin, J13 Conn_01x01_Pin, J14 Conn_01x01_Pin, J15 Conn_01x02, J16 Conn_01x04, J17 Conn_01x01_Pin, J18 Conn_01x01_Pin, J2 Conn_01x14_Socket, J3 Conn_01x01_Pin, J4 Conn_01x03_Socket, J5 Conn_01x01_Pin, J6 Conn_01x08, J7 Conn_01x01_Pin, J8 Conn_01x01_Pin, J9 Conn_01x01_Pin

Commit message: modified:   kicad/fc/main.kicad_pcb
Parts:
- turned J14 to 0 degrees
- turned J17 to 0 degrees
- turned J18 to 0 degrees
- turned J5 to 0 degrees
Changed lines of the file:
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@@
 	(footprint "Connector_Wire:SolderWirePad_1x01_SMD_1x2mm"
 		(layer "F.Cu")
-		(at 137.6 102.4 30)
+		(at 137.6 102.4)
 		(descr "Wire Pad, Square, SMD Pad,  1mm x 2mm")
 		(tags "MeasurementPoint Square SMDPad 1mmx2mm ")
 		(property "Reference" "J17"
-			(at -0.000001 -2 30)
+			(at -0.000001 -2 0)
 			(layer "F.SilkS")
 			(hide yes)
@@
 		)
 		(property "Value" "Conn_01x01_Pin"
-			(at 0 2.54 30)
+			(at 0 2.54 0)
 			(layer "F.Fab")
 			(hide yes)
@@
 		)
 		(property "Datasheet" ""
-			(at 0 0 30)
+			(at 0 0 0)
 			(unlocked yes)
 			(layer "F.Fab")
@@
 		)
 		(property "Description" "Generic connector, single row, 01x01, script generated"
-			(at 0 0 30)
+			(at 0 0 0)
 			(unlocked yes)
 			(layer "F.Fab")
@@
 		)
 		(pad "1" smd roundrect
-			(at 0 0 30)
+			(at 0 0)
 			(size 1 2)
 			(layers "F.Cu" "F.Mask")
@@
 	(footprint "Connector_Wire:SolderWirePad_1x01_SMD_1x2mm"
 		(layer "F.Cu")
-		(at 139.7 102.4 30)
+		(at 139.7 102.4)
 		(descr "Wire Pad, Square, SMD Pad,  1mm x 2mm")
 		(tags "MeasurementPoint Square SMDPad 1mmx2mm ")
 		(property "Reference" "J5"
-			(at -0.000001 -2 30)
+			(at -0.000001 -2 0)
 			(layer "F.SilkS")
 			(hide yes)
@@
 		)
 		(property "Value" "Conn_01x01_Pin"
-			(at 0 2.54 30)
+			(at 0 2.54 0)
 			(layer "F.Fab")
 			(hide yes)
@@
 		)
 		(property "Datasheet" ""
-			(at 0 0 30)
+			(at 0 0 0)
 			(unlocked yes)
 			(layer "F.Fab")
@@
 		)
 		(property "Description" "Generic connector, single row, 01x01, script generated"
-			(at 0 0 30)
+			(at 0 0 0)
 			(unlocked yes)
 			(layer "F.Fab")
@@
 		)
 		(pad "1" smd roundrect
-			(at 0 0 30)
+			(at 0 0)
 			(size 1 2)
 			(layers "F.Cu" "F.Mask")
@@
 	(footprint "Connector_Wire:SolderWirePad_1x01_SMD_1x2mm"
 		(layer "F.Cu")
-		(at 135.5 102.4 30)
+		(at 135.5 102.4)
 		(descr "Wire Pad, Square, SMD Pad,  1mm x 2mm")
 		(tags "MeasurementPoint Square SMDPad 1mmx2mm ")
 		(property "Reference" "J18"
-			(at -0.000001 -2 30)
+			(at -0.000001 -2 0)
 			(layer "F.SilkS")
 			(hide yes)
@@
 		)
 		(property "Value" "Conn_01x01_Pin"
-			(at 0 2.54 30)
+			(at 0 2.54 0)
 			(layer "F.Fab")
 			(hide yes)
@@
 		)
 		(property "Datasheet" ""
-			(at 0 0 30)
+			(at 0 0 0)
 			(unlocked yes)
 			(layer "F.Fab")
@@
 		)
 		(property "Description" "Generic connector, single row, 01x01, script generated"
-			(at 0 0 30)
+			(at 0 0 0)
 			(unlocked yes)
 			(layer "F.Fab")
@@
 		)
 		(pad "1" smd roundrect
-			(at 0 0 30)
+			(at 0 0)
 			(size 1 2)
 			(layers "F.Cu" "F.Mask")
@@
 	(footprint "Connector_Wire:SolderWirePad_1x01_SMD_1x2mm"
 		(layer "F.Cu")
-		(at 141.9 102.4 30)
+		(at 141.9 102.4)
 		(descr "Wire Pad, Square, SMD Pad,  1mm x 2mm")
 		(tags "MeasurementPoint Square SMDPad 1mmx2mm ")
 		(property "Reference" "J14"
-			(at 0 -1.999999 30)
+			(at 0 -1.999999 0)
 			(layer "F.SilkS")
 			(hide yes)
@@
 		)
 		(property "Value" "Conn_01x01_Pin"
-			(at -0.000001 2.54 30)
+			(at -0.000001 2.54 0)
 			(layer "F.Fab")
 			(hide yes)
@@
 		)
 		(property "Datasheet" ""
-			(at 0 0 30)
+			(at 0 0 0)
 			(unlocked yes)
 			(layer "F.Fab")
@@
 		)
 		(property "Description" "Generic connector, single row, 01x01, script generated"
-			(at 0 0 30)
+			(at 0 0 0)
 			(unlocked yes)
 			(layer "F.Fab")
@@
 		)
 		(pad "1" smd roundrect
-			(at 0 0 30)
+			(at 0 0)
 			(size 1 2)
 			(layers "F.Cu" "F.Mask")

Commit message: modified:   kicad/fc/main.kicad_pro
Parts:
- added J19: Conn_01x01_Pin, Connector_Wire:SolderWirePad_1x01_SMD_1x2mm, F.Cu at (155.3, 103.0)
- added J20: Conn_01x01_Pin, Connector_Wire:SolderWirePad_1x01_SMD_1x2mm, F.Cu at (153.2, 103.0)
- added J21: Conn_01x01_Pin, Connector_Wire:SolderWirePad_1x01_SMD_1x2mm, F.Cu at (151.1, 103.0)
- added J22: Conn_01x01_Pin, Connector_Wire:SolderWirePad_1x01_SMD_1x2mm, F.Cu at (149.0, 103.0)
Connections:
- J2 pad 6: unconnected-(J2-Pin_6-Pad6) -> /RX5
- J2 pad 7: unconnected-(J2-Pin_7-Pad7) -> /TX5
Routing:
- net /TX5: track 0.00 -> 11.4 mm, vias 0 -> 1
- net /RX5: track 0.00 -> 11.1 mm, vias 0 -> 1
- net /GND: track 101.4 -> 109.3 mm, vias 1 -> 2
- net /5V: track 62.8 -> 64.7 mm, vias 2 -> 4
Other:
- board text added: "RX5"
- board text added: "TX5"

Commit message: modified:   kicad/fc/main.kicad_pcb
Parts:
- moved J19 2.10 mm to (153.2, 103.0)
- moved J20 2.10 mm to (155.3, 103.0)
Routing:
- net /5V: track 64.7 -> 66.4 mm
- net /GND: track 109.3 -> 108.4 mm, vias 2 -> 1
Changed lines of the file:
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@@
 	(footprint "Connector_Wire:SolderWirePad_1x01_SMD_1x2mm"
 		(layer "F.Cu")
-		(at 155.3 103)
+		(at 153.2 103)
 		(descr "Wire Pad, Square, SMD Pad,  1mm x 2mm")
 		(tags "MeasurementPoint Square SMDPad 1mmx2mm ")
@@
 	(footprint "Connector_Wire:SolderWirePad_1x01_SMD_1x2mm"
 		(layer "F.Cu")
-		(at 153.2 103)
+		(at 155.3 103)
 		(descr "Wire Pad, Square, SMD Pad,  1mm x 2mm")
 		(tags "MeasurementPoint Square SMDPad 1mmx2mm ")
@@
 	)
 	(segment
-		(start 140.15 99.89)
-		(end 140.15 97.85)
+		(start 153.2 104.658067)
+		(end 153.2 103)
 		(width 0.4)
 		(layer "F.Cu")
@@
 	(segment
 		(start 140.15 99.89)
-		(end 139.7 100.34)
+		(end 140.15 97.85)
 		(width 0.4)
 		(layer "F.Cu")
@@
 	)
 	(segment
-		(start 145.99 83.79)
-		(end 137.63 83.79)
+		(start 140.15 99.89)
+		(end 139.7 100.34)
 		(width 0.4)
 		(layer "F.Cu")
@@
 	)
 	(segment
-		(start 140.44 100.18)
-		(end 140.15 99.89)
+		(start 139.7 102.4)
+		(end 142.31 105.01)
 		(width 0.4)
 		(layer "F.Cu")
@@
 	)
 	(segment
-		(start 139.7 102.4)
-		(end 142.31 105.01)
+		(start 145.99 83.79)
+		(end 137.63 83.79)
 		(width 0.4)
 		(layer "F.Cu")
@@
 	)
 	(segment
-		(start 156.73495 102.310958)
-		(end 155.989042 102.310958)
+		(start 152.848067 105.01)
+		(end 153.2 104.658067)
 		(width 0.4)
 		(layer "F.Cu")
@@
 	)
 	(segment
-		(start 153.29 105.01)
-		(end 155.3 103)
+		(start 140.44 100.18)
+		(end 140.15 99.89)
 		(width 0.4)
 		(layer "F.Cu")
@@
 	)
 	(segment
-		(start 159.385 92.725)
-		(end 158.67 93.44)
+		(start 152.250992 99.859008)
+		(end 152.250992 102.050992)
 		(width 0.4)
 		(layer "F.Cu")
@@
 	(segment
 		(start 142.31 105.01)
-		(end 153.29 105.01)
+		(end 152.848067 105.01)
 		(width 0.4)
 		(layer "F.Cu")
@@
 	)
 	(segment
+		(start 152.250992 102.050992)
+		(end 153.2 103)
+		(width 0.4)
+		(layer "F.Cu")
+		(net "/GND")
+	)
+	(segment
 		(start 154.05 73.25)
 		(end 154.49 72.81)
@@
 	)
 	(segment
-		(start 155.989042 102.310958)
-		(end 155.3 103)
+		(start 159.385 92.725)
+		(end 152.250992 99.859008)
 		(width 0.4)
 		(layer "F.Cu")
@@
 		(net "/GND")
 	)
-	(via
-		(at 156.73495 102.310958)
-		(size 0.6)
-		(drill 0.3)
-		(layers "F.Cu" "B.Cu")
-		(net "/GND")
-	)
 	(segment
 		(start 157.98 91.32)
@@
 	)
 	(segment
-		(start 159.385 92.725)
-		(end 159.385 99.660908)
-		(width 0.4)
-		(layer "B.Cu")
-		(net "/GND")
-	)
-	(segment
 		(start 154.49 72.81)
 		(end 157.01 72.81)
@@
 	)
 	(segment
-		(start 159.385 99.660908)
-		(end 156.73495 102.310958)
-		(width 0.4)
-		(layer "B.Cu")
-		(net "/GND")
-	)
-	(segment
 		(start 150.02 79.76)
 		(end 162.24 79.76)
@@
 	(segment
 		(start 161.925 92.725)
-		(end 153.65 101)
+		(end 155.122412 99.527588)
 		(width 0.4)
 		(layer "F.Cu")
@@
 	)
 	(segment
+		(start 155.122412 99.527588)
+		(end 153.65 101)
+		(width 0.4)
+		(layer "F.Cu")
+		(net "/5V")
+	)
+	(segment
 		(start 158.75 74.15)
 		(end 157.4 75.5)
@@
 	)
 	(segment
-		(start 153.2 101.073961)
-		(end 153.2 103)
+		(start 155.22073 99.625907)
+		(end 155.3 99.705176)
 		(width 0.4)
 		(layer "F.Cu")
@@
 	)
 	(segment
+		(start 155.122412 99.527588)
+		(end 155.22073 99.625907)
+		(width 0.4)
+		(layer "F.Cu")
+		(net "/5V")
+	)
+	(segment
 		(start 161.925 87.475)
 		(end 161.925 92.725)
@@
 		(width 0.4)
 		(layer "F.Cu")
+		(net "/5V")
+	)
+	(segment
+		(start 155.3 99.705176)
+		(end 155.3 103)
+		(width 0.4)
+		(layer "F.Cu")
