File: kicad/fc/main.kicad_sch (KiCad schematic)
At the start: 26 parts, among them J1 Conn_01x14, J10 Conn_01x01_Pin, J11 Conn_01x01_Pin, J12 Conn_01x01_Pin, J13 Conn_01x01_Pin, J14 Conn_01x01_Pin, J15 Conn_01x02, J16 Conn_01x04, J17 Conn_01x01_Pin, J18 Conn_01x01_Pin, J2 Conn_01x14_Socket, J3 Conn_01x01_Pin, J4 Conn_01x03_Socket, J5 Conn_01x01_Pin, J6 Conn_01x08, J7 Conn_01x01_Pin, J8 Conn_01x01_Pin, J9 Conn_01x01_Pin

Commit message: modified:   kicad/fc/main.kicad_pro
Parts:
- added J19, J20, J21, J22: Conn_01x01_Pin, Connector_Wire:SolderWirePad_1x01_SMD_1x2mm, symbol Connector:Conn_01x01_Pin
Connections:
- net 5V: now also J20.1 (Pin_1)
- net GND: now also J19.1 (Pin_1)
- net RX5: now reaches J2.6 (Pin_6)
- net RX5: now also J21.1 (Pin_1)
- net TX5: now reaches J2.7 (Pin_7)
- net TX5: now also J22.1 (Pin_1)
Other:
- note added: "FPGA"

Commit message: Added IMU interrupt INT pin to FC board
Connections:
- net INT: now reaches J2.5 (Pin_5)
- net INT: now also J13.1 (Pin_1)
Changed lines of the file:
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@@
 		)
+	)
+	(junction
+		(at 129.54 87.63)
+		(diameter 0)
+		(color 0 0 0 0)
 	)
 	(wire
@@
 	(wire
 		(pts
+			(xy 129.54 87.63) (xy 130.81 87.63)
+		)
+		(stroke
+			(width 0)
+			(type default)
+		)
+	)
+	(wire
+		(pts
 			(xy 96.52 92.71) (xy 101.6 92.71)
 		)
@@
 		(pts
 			(xy 147.32 99.06) (xy 152.4 99.06)
+		)
+		(stroke
+			(width 0)
+			(type default)
+		)
+	)
+	(wire
+		(pts
+			(xy 124.46 87.63) (xy 129.54 87.63)
 		)
 		(stroke
@@
 		)
 	)
+	(label "INT"
+		(at 124.46 87.63 0)
+		(effects
+			(font
+				(size 1.27 1.27)
+			)
+			(justify left bottom)
+		)
+	)
 	(label "GND"
 		(at 147.32 139.7 0)
@@
 		(effects
 			(font
+				(size 1.27 1.27)
+			)
+			(justify left bottom)
+		)
+	)
+	(label "INT"
+		(at 119.38 142.24 0)
+		(effects
+			(font

Commit message: Cleanup
Connections:
- net INT: no longer names the net of J2.5 (Pin_5)
- net INT: no longer J13.1 (Pin_1)
Changed lines of the file:
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@@
 		)
-	)
-	(junction
-		(at 129.54 87.63)
-		(diameter 0)
-		(color 0 0 0 0)
 	)
 	(wire
@@
 	(wire
 		(pts
-			(xy 118.11 142.24) (xy 123.19 142.24)
-		)
-		(stroke
-			(width 0)
-			(type default)
-		)
-	)
-	(wire
-		(pts
 			(xy 147.32 93.98) (xy 152.4 93.98)
 		)
@@
 		(pts
 			(xy 147.32 99.06) (xy 152.4 99.06)
-		)
-		(stroke
-			(width 0)
-			(type default)
-		)
-	)
-	(wire
-		(pts
-			(xy 124.46 87.63) (xy 129.54 87.63)
 		)
 		(stroke
@@
 		)
 	)
-	(label "INT"
-		(at 124.46 87.63 0)
-		(effects
-			(font
-				(size 1.27 1.27)
-			)
-			(justify left bottom)
-		)
-	)
 	(label "GND"
 		(at 147.32 139.7 0)
@@
 		(effects
 			(font
-				(size 1.27 1.27)
-			)
-			(justify left bottom)
-		)
-	)
-	(label "INT"
-		(at 119.38 142.24 0)
-		(effects
-			(font
