File: kicad/1s/main.kicad_pcb (KiCad board)
At the start: 2 copper layers, 41 x 41.5 mm, 30 parts, among them J1 Conn_01x14, J10 Conn_01x01_Pin, J11 Conn_01x01_Pin, J12 Conn_01x01_Pin, J13 Conn_01x01_Pin, J14 Conn_01x01_Pin, J15 Conn_01x02, J16 Conn_01x04, J17 Conn_01x01_Pin, J18 Conn_01x01_Pin, J19 Conn_01x01_Pin, J2 Conn_01x14_Socket, J20 Conn_01x01_Pin, J21 Conn_01x01_Pin, J22 Conn_01x01_Pin, J3 Conn_01x01_Pin, J4 Conn_01x03_Socket, J5 Conn_01x01_Pin, J6 Conn_01x08, J7 Conn_01x01_Pin, J8 Conn_01x01_Pin, J9 Conn_01x01_Pin

Commit message: modified:   kicad/1s/main.kicad_pcb
Parts:
- added J23: Conn_01x03_Socket, Connector_PinHeader_2.54mm:PinHeader_1x03_P2.54mm_Vertical, F.Cu at (132.1, 103.1)
- added J24: Conn_01x03_Socket, Connector_PinHeader_2.54mm:PinHeader_1x03_P2.54mm_Vertical, F.Cu at (128.6, 71.5)
- J15: value Conn_01x02 -> Conn_01x03_Socket; footprint Connector_PinSocket_2.00mm:PinSocket_1x02_P2.00mm_Vertical -> Connector_PinHeader_2.54mm:PinHeader_1x03_P2.54mm_Vertical
- J16: value Conn_01x04 -> Conn_01x03_Socket; footprint Connector_PinSocket_2.00mm:PinSocket_1x04_P2.00mm_Vertical -> Connector_PinHeader_2.54mm:PinHeader_1x03_P2.54mm_Vertical
- moved J15 31.6 mm to (164.0, 99.3), turned to -45 degrees
- moved J16 18.6 mm to (160.6, 68.0), turned to 45 degrees
Connections:
- J1 pad 6: /M3 -> unconnected-(J1-Pin_6-Pad6)
- J1 pad 7: /M4 -> unconnected-(J1-Pin_7-Pad7)
- J15 pad 1: /GND -> /M1
- J16 pad 1: /M1 -> /M2
- J16 pad 2: /M2 -> /VBAT
- J16 pad 3: /M3 -> /GND
- J2 pad 4: /A9 -> /M1
- J2 pad 5: unconnected-(J2-Pin_5-Pad5) -> /A8
- R2 pad 1: /A9 -> /A8
- R3 pad 2: /A9 -> /A8
Routing:
- net /A8: track 0.00 -> 30.4 mm
- net /A9: track 29.5 -> 0.00 mm
- net /GND: track 108.4 -> 88.8 mm, vias 1 -> 2
- net /M4: track 17.0 -> 0.00 mm
- net /M2: track 18.5 -> 1.60 mm
- net /M3: track 16.5 -> 0.00 mm
- net /VBAT: track 33.8 -> 48.0 mm
- net unconnected-(J1-Pin_7-Pad7): track 0.00 -> 1.15 mm
- net /M1: track 17.0 -> 16.2 mm, vias 0 -> 2
- removed copper zone on F.Cu, net /GND
Other:
- board size 41 x 41.5 mm -> 40.2 x 41.1 mm

Commit message: modified:   kicad/1s/main.kicad_pcb
Routing:
- net /GND: track 88.8 -> 87.1 mm
Other:
- board size 40.2 x 41.1 mm -> 40.2 x 46.1 mm
- board text added: "A8"
Changed lines of the file:
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@@
 	)
 	(gr_line
-		(start 137 106.02)
+		(start 136.998914 106)
 		(end 134.228775 103.249535)
 		(stroke
@@
 	)
 	(gr_line
-		(start 155.278763 106.02)
-		(end 137 106.02)
-		(stroke
-			(width 0.2)
-			(type solid)
-		)
-		(layer "Edge.Cuts")
-	)
-	(gr_line
-		(start 155.280996 106.014145)
+		(start 142.042403 106)
+		(end 136.998914 106)
+		(stroke
+			(width 0.2)
+			(type solid)
+		)
+		(layer "Edge.Cuts")
+	)
+	(gr_line
+		(start 142.042403 111)
+		(end 142.042403 106)
+		(stroke
+			(width 0.2)
+			(type solid)
+		)
+		(layer "Edge.Cuts")
+	)
+	(gr_line
+		(start 142.042403 111)
+		(end 150.3 111)
+		(stroke
+			(width 0.2)
+			(type solid)
+		)
+		(layer "Edge.Cuts")
+	)
+	(gr_line
+		(start 150.3 111)
+		(end 150.3 106)
+		(stroke
+			(width 0.2)
+			(type solid)
+		)
+		(layer "Edge.Cuts")
+	)
+	(gr_line
+		(start 155.3 106)
+		(end 150.3 106)
+		(stroke
+			(width 0.2)
+			(type solid)
+		)
+		(layer "Edge.Cuts")
+	)
+	(gr_line
+		(start 155.3 106)
 		(end 158.26323 103.067896)
 		(stroke
@@
 	)
 	(gr_text ">LED"
-		(at 128.75 73.8 0)
+		(at 129.25962 74.129423 0)
 		(layer "F.SilkS")
 		(effects
@@
 		)
 	)
-	(gr_text "A9"
-		(at 156.61 68.99 0)
+	(gr_text "A8"
+		(at 156.207532 70.892542 0)
 		(layer "F.SilkS")
 		(effects
@@
 		)
 	)
-	(gr_text "A9"
+	(gr_text "A8"
 		(at 162.65 74.85 0)
+		(layer "F.SilkS")
+		(effects
+			(font
+				(size 0.8 0.8)
+				(thickness 0.15)
+			)
+			(justify left bottom)
+		)
+	)
+	(gr_text "M4"
+		(at 129.430798 73.562297 45)
+		(layer "F.SilkS")
+		(effects
+			(font
+				(size 0.8 0.8)
+				(thickness 0.15)
+			)
+			(justify left bottom)
+		)
+	)
+	(gr_text "VB"
+		(at 131.308955 71.698538 45)
+		(layer "F.SilkS")
+		(effects
+			(font
+				(size 0.8 0.8)
+				(thickness 0.15)
+			)
+			(justify left bottom)
+		)
+	)
+	(gr_text "GD"
+		(at 132.974339 70.004357 45)
 		(layer "F.SilkS")
 		(effects
@@
 	)
 	(gr_text "GD"
-		(at 159.317438 103.082581 45)
+		(at 159.184346 102.797911 45)
 		(layer "F.SilkS")
 		(effects
@@
 	)
 	(gr_text "VB"
-		(at 161.128035 101.341622 45)
+		(at 161.038718 101.000469 45)
 		(layer "F.SilkS")
 		(effects
@@
 	)
 	(gr_text "M1"
-		(at 162.747126 99.687711 45)
+		(at 162.671576 99.29696 45)
 		(layer "F.SilkS")
 		(effects
@@
 	(gr_text "5V"
 		(at 164.11 93.64 90)
+		(layer "F.SilkS")
+		(effects
+			(font
+				(size 0.8 0.8)
+				(thickness 0.15)
+			)
+			(justify left bottom)
+		)
+	)
+	(gr_text "GD"
+		(at 128.496968 98.165761 315)
+		(layer "F.SilkS")
+		(effects
+			(font
+				(size 0.8 0.8)
+				(thickness 0.15)
+			)
+			(justify left bottom)
+		)
+	)
+	(gr_text "VB"
+		(at 130.392122 99.939431 315)
+		(layer "F.SilkS")
+		(effects
+			(font
+				(size 0.8 0.8)
+				(thickness 0.15)
+			)
+			(justify left bottom)
+		)
+	)
+	(gr_text "M3"
+		(at 132.26298 101.672607 315)
+		(layer "F.SilkS")
+		(effects
+			(font
+				(size 0.8 0.8)
+				(thickness 0.15)
+			)
+			(justify left bottom)
+		)
+	)
+	(gr_text "M2"
+		(at 158.661515 68.997387 315)
+		(layer "F.SilkS")
+		(effects
+			(font
+				(size 0.8 0.8)
+				(thickness 0.15)
+			)
+			(justify left bottom)
+		)
+	)
+	(gr_text "VB"
+		(at 160.556669 70.771057 315)
+		(layer "F.SilkS")
+		(effects
+			(font
+				(size 0.8 0.8)
+				(thickness 0.15)
+			)
+			(justify left bottom)
+		)
+	)
+	(gr_text "GD"
+		(at 162.670496 72.666212 315)
 		(layer "F.SilkS")
 		(effects
@@
 	)
 	(segment
-		(start 159.385 98.178659)
-		(end 159.385 102.082045)
-		(width 1)
-		(layer "F.Cu")
-		(net "/GND")
-	)
-	(segment
 		(start 140.44 100.18)
 		(end 140.15 99.89)
@@
 	)
 	(segment
-		(start 159.385 102.082045)
-		(end 160.620709 103.317754)
-		(width 1)
-		(layer "F.Cu")
-		(net "/GND")
-	)
-	(segment
 		(start 142.31 105.01)
 		(end 152.848067 105.01)
 		(width 0.4)
+		(layer "F.Cu")
+		(net "/GND")
+	)
+	(segment
+		(start 159.385 98.178659)
+		(end 159.385 101.869361)
+		(width 1)
 		(layer "F.Cu")
 		(net "/GND")
@@
 		(layer "F.Cu")
 		(net "/GND")
+	)
+	(segment
+		(start 160.39191 102.876271)
+		(end 160.39191 103.088955)
+		(width 1)
+		(layer "F.Cu")
+		(net "/GND")

Commit message: modified:   kicad/1s/main.kicad_pro
Parts:
- added J25: Conn_01x01_Pin, Connector_Wire:SolderWirePad_1x01_SMD_2x4mm, F.Cu at (144.2, 108.3)
- added J26: Conn_01x01_Pin, Connector_Wire:SolderWirePad_1x01_SMD_2x4mm, F.Cu at (148.3, 108.3)
- moved R3 7.01 mm to (147.5, 72.2)
- moved R2 5.19 mm to (153.5, 68.7), turned to 180 degrees
Connections:
- J1 pad 10: unconnected-(J1-Pin_10-Pad10) -> /M3
- J1 pad 2: unconnected-(J1-Pin_2-Pad2) -> /M2
- J1 pad 4: /M1 -> unconnected-(J1-Pin_4-Pad4)
- J1 pad 5: /M2 -> unconnected-(J1-Pin_5-Pad5)
- J1 pad 9: unconnected-(J1-Pin_9-Pad9) -> /M4
- J24 pad 3: unconnected-(J24-Pin_3-Pad3) -> /GND
Routing:
- net /VBAT: track 48.0 -> 133.5 mm, vias 0 -> 1
- net /GND: track 87.1 -> 152.5 mm
- net /5V: track 66.4 -> 35.8 mm, vias 4 -> 2
- net /M3: track 0.00 -> 28.3 mm, vias 0 -> 2
- net /M4: track 0.00 -> 16.5 mm
- net /A8: track 30.4 -> 14.7 mm
- net /M2: track 1.60 -> 10.2 mm, vias 0 -> 1
- net /CS: track 30.9 -> 24.8 mm, vias 0 -> 2
- net /SCK: track 22.7 -> 26.1 mm, vias 0 -> 2
- net /M1: track 16.2 -> 12.9 mm, vias 2 -> 0
- net /3V3: track 44.7 -> 43.8 mm
- net unconnected-(J1-Pin_5-Pad5): track 0.00 -> 0.69 mm
- net /RX3: track 11.2 -> 11.8 mm, vias 0 -> 1
- net /TX3: track 11.4 -> 11.5 mm, vias 0 -> 1
Other:
- board text removed: "A9"
- board text removed: "RX1"
- board text removed: "TX1"

Commit message: modified:   kicad/1s/main.kicad_pcb
Parts:
- moved R2 3.26 mm to (156.8, 68.5)
Routing:
- net /A8: track 14.7 -> 27.0 mm, vias 0 -> 1
- net /VBAT: track 133.5 -> 136.1 mm
- net /GND: track 152.5 -> 154.3 mm
- added copper zone on F.Cu, net /GND
Other:
- board text added: "+"
- board text added: "-"
- board text removed: "RX2"
- board text removed: "TX2"
