File: kicad/fc/1s/main.kicad_sch (KiCad schematic)
At the start: 34 parts, among them J1 Conn_01x14, J10 Conn_01x01_Pin, J11 Conn_01x01_Pin, J12 Conn_01x01_Pin, J13 Conn_01x01_Pin, J14 Conn_01x01_Pin, J15 Conn_01x03_Socket, J16 Conn_01x03_Socket, J17 Conn_01x01_Pin, J18 Conn_01x01_Pin, J19 Conn_01x01_Pin, J2 Conn_01x14_Socket, J20 Conn_01x01_Pin, J21 Conn_01x01_Pin, J22 Conn_01x01_Pin, J23 Conn_01x03_Socket, J24 Conn_01x03_Socket, J25 Conn_01x01_Pin, J26 Conn_01x01_Pin, J3 Conn_01x01_Pin, J4 Conn_01x03_Socket, J5 Conn_01x01_Pin, J6 Conn_01x08, J7 Conn_01x01_Pin, J8 Conn_01x01_Pin, J9 Conn_01x01_Pin

Commit message: modified:   fc/1s/main.kicad_pcb
Parts:
- removed J6: Conn_01x08, Connector_PinSocket_2.00mm:PinSocket_1x08_P2.00mm_Vertical, symbol Connector_Generic:Conn_01x08
- added J27: Conn_02x04_Odd_Even, Connector_PinHeader_2.54mm:PinHeader_2x04_P2.54mm_Vertical, symbol Connector_Generic:Conn_02x04_Odd_Even
Connections:
- net 3V3: now also J27.1 (Pin_1)
- net CS: now also J27.4 (Pin_4)
- net GND: now also J27.2 (Pin_2)
- net MISO: now also J27.6 (Pin_6)
- net MOSI: now also J27.3 (Pin_3)
- net SCK: now also J27.5 (Pin_5)
- net SCL1: now also J27.8 (Pin_8)
- net SDA1: now also J27.7 (Pin_7)
Other:
- note removed: "Hover"

Commit message: modified:   kicad/fc/1s/main.kicad_pcb
Parts:
- removed J27: Conn_02x04_Odd_Even, Connector_PinHeader_2.54mm:PinHeader_2x04_P2.54mm_Vertical, symbol Connector_Generic:Conn_02x04_Odd_Even
- added J27, J6: Conn_01x04_Socket, Connector_PinHeader_2.54mm:PinHeader_1x04_P2.54mm_Vertical, symbol Connector:Conn_01x04_Socket
Connections:
- net 3V3: now also J27.4 (Pin_4)
- net CS: now also J6.1 (Pin_1)
- net GND: now also J27.3 (Pin_3)
- net MISO: now also J6.3 (Pin_3)
- net MOSI: now also J6.2 (Pin_2)
- net SCK: now also J6.4 (Pin_4)
- net SCL1: now also J27.1 (Pin_1)
- net SDA1: now also J27.2 (Pin_2)
