File: kicad/fc/1s/main.kicad_pcb (KiCad board)
At the start: 2 copper layers, 40.2 x 46.1 mm, 34 parts, among them J1 Conn_01x14, J10 Conn_01x01_Pin, J11 Conn_01x01_Pin, J12 Conn_01x01_Pin, J13 Conn_01x01_Pin, J14 Conn_01x01_Pin, J15 Conn_01x03_Socket, J16 Conn_01x03_Socket, J17 Conn_01x01_Pin, J18 Conn_01x01_Pin, J19 Conn_01x01_Pin, J2 Conn_01x14_Socket, J20 Conn_01x01_Pin, J21 Conn_01x01_Pin, J22 Conn_01x01_Pin, J23 Conn_01x03_Socket, J24 Conn_01x03_Socket, J25 Conn_01x01_Pin, J26 Conn_01x01_Pin, J27 Conn_02x04_Odd_Even, J3 Conn_01x01_Pin, J4 Conn_01x03_Socket, J5 Conn_01x01_Pin, J7 Conn_01x01_Pin, J8 Conn_01x01_Pin, J9 Conn_01x01_Pin

Commit message: modified:   kicad/fc/1s/main.kicad_pcb
Parts:
- moved R1 17.9 mm to (148.8, 74.9), turned to 180 degrees
Routing:
- net Net-(D1-A): track 8.40 -> 19.3 mm
- net /LED: track 13.0 -> 8.07 mm, vias 0 -> 1
Changed lines of the file:
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@@
 	(footprint "Resistor_THT:R_Axial_DIN0204_L3.6mm_D1.6mm_P7.62mm_Horizontal"
 		(layer "F.Cu")
-		(at 132.675 82.79 -90)
+		(at 148.791324 74.924901 180)
 		(descr "Resistor, Axial_DIN0204 series, Axial, Horizontal, pin pitch=7.62mm, 0.167W, length*diameter=3.6*1.6mm^2, http://cdn-reichelt.de/documents/datenblatt/B400/1_4W%23YAG.pdf")
 		(tags "Resistor Axial_DIN0204 series Axial Horizontal pin pitch 7.62mm 0.167W length 3.6mm diameter 1.6mm")
 		(property "Reference" "R1"
-			(at 3.81 0 90)
+			(at 3.81 0 0)
 			(layer "F.SilkS")
 			(hide yes)
@@
 		)
 		(property "Value" "R_LED"
-			(at 3.81 1.92 90)
+			(at 3.81 1.92 0)
 			(layer "F.Fab")
 			(hide yes)
@@
 		)
 		(property "Datasheet" ""
-			(at 0 0 90)
+			(at 0 0 0)
 			(layer "F.Fab")
 			(hide yes)
@@
 		)
 		(property "Description" "Resistor"
-			(at 0 0 90)
+			(at 0 0 0)
 			(layer "F.Fab")
 			(hide yes)
@@
 		(duplicate_pad_numbers_are_jumpers no)
 		(pad "1" thru_hole circle
-			(at -1.25 0 270)
+			(at -1.25 0 180)
 			(size 1.4 1.4)
 			(drill 0.7)
@@
 		)
 		(pad "2" thru_hole circle
-			(at 6.37 0 270)
+			(at 6.37 0 180)
 			(size 1.4 1.4)
 			(drill 0.7)
@@
 	)
 	(gr_text ">LED"
-		(at 128.3 82.7 0)
-		(layer "F.SilkS")
-		(effects
-			(font
-				(size 0.8 0.8)
-				(thickness 0.15)
-			)
-			(justify left bottom)
-		)
-	)
-	(gr_text "LED>"
-		(at 129.26 88.57 0)
+		(at 129.499815 74.938153 0)
 		(layer "F.SilkS")
 		(effects
@@
 		)
 	)
-	(gr_text ">LED"
-		(at 129.499815 74.938153 0)
+	(gr_text "GD"
+		(at 135 84.21 0)
 		(layer "F.SilkS")
 		(effects
@@
 	)
 	(gr_text "GD"
-		(at 135 84.21 0)
+		(at 137.1 73.9 0)
 		(layer "F.SilkS")
 		(effects
@@
 		)
 	)
-	(gr_text "GD"
-		(at 137.1 73.9 0)
+	(gr_text "M3"
+		(at 138.119148 79.9 0)
 		(layer "F.SilkS")
 		(effects
@@
 		)
 	)
-	(gr_text "M3"
-		(at 138.119148 79.9 0)
+	(gr_text "M4"
+		(at 140.663107 79.971888 0)
 		(layer "F.SilkS")
 		(effects
@@
 		)
 	)
-	(gr_text "M4"
-		(at 140.663107 79.971888 0)
+	(gr_text "LED>"
+		(at 140.755653 73.980584 0)
 		(layer "F.SilkS")
 		(effects
@@
 		)
 	)
+	(gr_text ">LED"
+		(at 150.943372 75.378899 0)
+		(layer "F.SilkS")
+		(effects
+			(font
+				(size 0.8 0.8)
+				(thickness 0.15)
+			)
+			(justify left bottom)
+		)
+	)
 	(gr_text "3V3"
 		(at 153.2 82 0)
@@
 		)
 	)
+	(gr_text "R 100Ω"
+		(at 148.609151 75.511735 0)
+		(layer "B.SilkS")
+		(effects
+			(font
+				(size 0.8 0.8)
+				(thickness 0.15)
+			)
+			(justify left bottom mirror)
+		)
+	)
 	(gr_text "5V"
 		(at 156 88.5 0)
@@
 		)
 	)
-	(gr_text "R 100Ω"
-		(at 133.15 82.95 90)
-		(layer "B.SilkS")
-		(effects
-			(font
-				(size 0.8 0.8)
-				(thickness 0.15)
-			)
-			(justify left bottom mirror)
-		)
-	)
 	(gr_text "CS"
 		(at 134.51 78.9 90)
@@
 	)
 	(segment
+		(start 144.145 91.645)
+		(end 152 83.79)
+		(width 0.2)
+		(layer "F.Cu")
+		(net "/SCL0")
+	)
+	(segment
+		(start 144.145 92.725)
+		(end 144.145 91.645)
+		(width 0.2)
+		(layer "F.Cu")
+		(net "/SCL0")
+	)
+	(segment
+		(start 131.445 77.725)
+		(end 145.535 91.815)
+		(width 0.2)
+		(layer "B.Cu")
+		(net "/MOSI")
+	)
+	(segment
+		(start 145.535 91.815)
+		(end 145.535 94.115961)
+		(width 0.2)
+		(layer "B.Cu")
+		(net "/MOSI")
+	)
+	(segment
+		(start 145.535 94.115961)
+		(end 146.668695 95.249656)
+		(width 0.2)
+		(layer "B.Cu")
+		(net "/MOSI")
+	)
+	(segment
 		(start 133.993688 86.558557)
 		(end 134.057247 86.622117)
@@
 	)
 	(segment
-		(start 131.445 77.725)
-		(end 145.535 91.815)
+		(start 134.630131 90.523599)
+		(end 137.565258 90.523599)
+		(width 0.2)
+		(layer "F.Cu")
+		(net "/SCK")
+	)
+	(segment
+		(start 137.565258 90.523599)
+		(end 137.580262 90.508595)
+		(width 0.2)
+		(layer "F.Cu")
+		(net "/SCK")
+	)
+	(via
+		(at 134.630131 90.523599)
+		(size 0.6)
+		(drill 0.3)
+		(layers "F.Cu" "B.Cu")
+		(net "/SCK")
+	)
+	(via
+		(at 137.580262 90.508595)
+		(size 0.6)
+		(drill 0.3)
+		(layers "F.Cu" "B.Cu")
+		(net "/SCK")
+	)
+	(segment
+		(start 141.014941 90.508595)
+		(end 137.580262 90.508595)
 		(width 0.2)
 		(layer "B.Cu")
-		(net "/MOSI")
+		(net "/SCK")
 	)
 	(segment
-		(start 145.535 91.815)
-		(end 145.535 94.115961)
+		(start 134.630131 90.523599)
+		(end 134.669611 90.523599)
 		(width 0.2)
 		(layer "B.Cu")
-		(net "/MOSI")
+		(net "/SCK")
 	)
 	(segment
-		(start 145.535 94.115961)
-		(end 146.668695 95.249656)
+		(start 131.106401 90.523599)
+		(end 134.630131 90.523599)
 		(width 0.2)
 		(layer "B.Cu")
-		(net "/MOSI")
+		(net "/SCK")
+	)
+	(segment
+		(start 142.995 92.488654)
+		(end 141.014941 90.508595)
+		(width 0.2)
+		(layer "B.Cu")
+		(net "/SCK")
+	)
+	(segment
+		(start 128.905 92.725)
+		(end 131.106401 90.523599)
+		(width 0.2)
+		(layer "B.Cu")
+		(net "/SCK")
+	)
+	(segment
+		(start 142.995 94.115961)
+		(end 142.995 92.488654)
+		(width 0.2)
+		(layer "B.Cu")
+		(net "/SCK")
+	)
+	(segment
+		(start 144.128695 95.249656)
+		(end 142.995 94.115961)
+		(width 0.2)
+		(layer "B.Cu")
+		(net "/SCK")
 	)
 	(segment
@@
 	)
 	(segment
-		(start 134.630131 90.523599)
-		(end 137.565258 90.523599)
-		(width 0.2)
-		(layer "F.Cu")
-		(net "/SCK")
-	)
-	(segment
-		(start 137.565258 90.523599)
-		(end 137.580262 90.508595)
+		(start 141.588695 95.248695)
+		(end 141.588695 95.249656)
 		(width 0.2)
 		(layer "F.Cu")
-		(net "/SCK")
-	)
-	(via
-		(at 134.630131 90.523599)
-		(size 0.6)
-		(drill 0.3)
-		(layers "F.Cu" "B.Cu")
-		(net "/SCK")
-	)
-	(via
-		(at 137.580262 90.508595)
-		(size 0.6)
-		(drill 0.3)
-		(layers "F.Cu" "B.Cu")
-		(net "/SCK")
-	)
-	(segment
-		(start 141.014941 90.508595)
-		(end 137.580262 90.508595)
-		(width 0.2)
-		(layer "B.Cu")
-		(net "/SCK")
-	)
-	(segment
-		(start 134.630131 90.523599)
-		(end 134.669611 90.523599)
-		(width 0.2)
-		(layer "B.Cu")
-		(net "/SCK")
-	)
-	(segment
-		(start 131.106401 90.523599)
-		(end 134.630131 90.523599)
-		(width 0.2)
-		(layer "B.Cu")
-		(net "/SCK")
-	)
-	(segment
-		(start 142.995 92.488654)
-		(end 141.014941 90.508595)
-		(width 0.2)
-		(layer "B.Cu")
-		(net "/SCK")
-	)
-	(segment
-		(start 128.905 92.725)
-		(end 131.106401 90.523599)
-		(width 0.2)
-		(layer "B.Cu")
-		(net "/SCK")
-	)
-	(segment
-		(start 142.995 94.115961)
-		(end 142.995 92.488654)
-		(width 0.2)
-		(layer "B.Cu")
-		(net "/SCK")
+		(net "/SDA1")
 	)
 	(segment
-		(start 144.128695 95.249656)
-		(end 142.995 94.115961)
+		(start 139.065 92.725)
+		(end 141.588695 95.248695)
 		(width 0.2)
 		(layer "B.Cu")
-		(net "/SCK")
+		(net "/SDA1")
 	)
 	(segment
@@
 	)
 	(segment
-		(start 141.588695 95.248695)
-		(end 141.588695 95.249656)
-		(width 0.2)
-		(layer "F.Cu")
-		(net "/SDA1")
-	)
-	(segment
-		(start 139.065 92.725)
-		(end 141.588695 95.248695)
-		(width 0.2)
-		(layer "B.Cu")
-		(net "/SDA1")
-	)
-	(segment
-		(start 144.145 91.645)
-		(end 152 83.79)
-		(width 0.2)
-		(layer "F.Cu")
-		(net "/SCL0")
-	)
-	(segment
-		(start 144.145 92.725)
-		(end 144.145 91.645)
-		(width 0.2)
-		(layer "F.Cu")
-		(net "/SCL0")
-	)
-	(segment
 		(start 147.902579 93.942579)
 		(end 147.902579 101.902579)
@@
 	)
 	(segment
-		(start 132.675 74.035)
-		(end 132.675 81.54)
+		(start 146.103439 72.2)
+		(end 148.82834 74.924901)
 		(width 0.2)
-		(layer "F.Cu")
+		(layer "B.Cu")
+		(net "Net-(D1-A)")
+	)
+	(segment
+		(start 148.82834 74.924901)
+		(end 150.041324 74.924901)
+		(width 0.2)
+		(layer "B.Cu")
+		(net "Net-(D1-A)")
+	)
+	(segment
+		(start 134.51 72.2)
+		(end 146.103439 72.2)
+		(width 0.2)
+		(layer "B.Cu")
+		(net "Net-(D1-A)")
+	)
+	(segment
+		(start 133.31 73.4)
+		(end 134.51 72.2)
+		(width 0.2)
+		(layer "B.Cu")
 		(net "Net-(D1-A)")
 	)
@@
 	(segment
 		(start 136.525 77.725)
-		(end 135.675 78.575)
+		(end 136.525 75.996062)
 		(width 0.2)
 		(layer "F.Cu")
@@
 	)
 	(segment
-		(start 135.675 86.16)
-		(end 132.675 89.16)
+		(start 136.525 75.996062)
+		(end 136.914829 75.606233)
 		(width 0.2)
 		(layer "F.Cu")
 		(net "/LED")
 	)
+	(via
+		(at 136.914829 75.606233)
+		(size 0.6)
+		(drill 0.3)
+		(layers "F.Cu" "B.Cu")
+		(net "/LED")
+	)
 	(segment
-		(start 135.675 78.575)
-		(end 135.675 86.16)
+		(start 136.914829 75.606233)
+		(end 137.596161 74.924901)
 		(width 0.2)
-		(layer "F.Cu")
+		(layer "B.Cu")
+		(net "/LED")
+	)
+	(segment
+		(start 137.596161 74.924901)
+		(end 142.421324 74.924901)
+		(width 0.2)
+		(layer "B.Cu")
 		(net "/LED")
 	)

Commit message: modified:   kicad/fc/1s/main.kicad_pcb
Parts:
- added J6: Conn_01x04_Socket, Connector_PinHeader_2.54mm:PinHeader_1x04_P2.54mm_Vertical, F.Cu at (133.5, 81.8)
- J27: value Conn_02x04_Odd_Even -> Conn_01x04_Socket; footprint Connector_PinHeader_2.54mm:PinHeader_2x04_P2.54mm_Vertical -> Connector_PinHeader_2.54mm:PinHeader_1x04_P2.54mm_Vertical
- moved J4 23.4 mm to (151.0, 112.5), turned to 180 degrees
- moved J27 16.3 mm to (158.5, 81.8), turned to 0 degrees
- moved J26 9.31 mm to (144.3, 116.7)
- moved J25 9.20 mm to (148.2, 116.6)
Connections:
- J27 pad 1: /3V3 -> /SCL1
- J27 pad 2: /GND -> /SDA1
- J27 pad 3: /MOSI -> /GND
- J27 pad 4: /CS -> /3V3
Routing:
- net /CS: track 28.0 -> 4.90 mm, vias 1 -> 0
- net /SDA1: track 3.57 -> 23.3 mm
- net /SCL1: track 7.16 -> 26.5 mm
- net /MOSI: track 23.8 -> 7.50 mm
- net /MISO: track 35.2 -> 21.7 mm, vias 1 -> 0
- net /GND: track 163.9 -> 150.6 mm, vias 2 -> 4
- net /SCK: track 19.1 -> 6.15 mm, vias 2 -> 0
- net /VBAT: track 136.1 -> 148.4 mm, vias 1 -> 2
- net /3V3: track 31.3 -> 26.0 mm
- net /M1: track 12.9 -> 15.2 mm
- net /5V: track 35.7 -> 37.6 mm
- net /M3: track 28.3 -> 29.3 mm
Other:
- board size 40.2 x 46.1 mm -> 40.2 x 55.1 mm
- board text removed: "GND"

Commit message: modified:   kicad/hover/1s/main.kicad_pcb
Parts:
- added G***: LOGO, LOGO, B.Cu at (145.0, 84.6)
- moved J27 0.50 mm to (158.0, 81.8)
- moved J6 0.50 mm to (134.0, 81.8)
Routing:
- net /CS: track 4.90 -> 4.17 mm
Other:
- board text added: "tindie.com/stores/bobbiebots"

Commit message: modified:   kicad/fc/1s/main.kicad_pcb
Parts:
- moved J25 1.91 mm to (148.2, 118.5)
- moved J26 1.77 mm to (144.4, 118.5)
- moved J4 1.22 mm to (151.0, 113.7)
Routing:
- net /GND: track 150.6 -> 148.5 mm
- net /5V: track 37.6 -> 39.1 mm
- net /VBAT: track 148.4 -> 147.7 mm
Other:
- board size 40.2 x 55.1 mm -> 40.2 x 57.1 mm
Changed lines of the file:
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@@
 	(footprint "Connector_Wire:SolderWirePad_1x01_SMD_2x4mm"
 		(layer "F.Cu")
-		(at 148.202235 116.592822)
+		(at 148.247162 118.5)
 		(descr "Wire Pad, Square, SMD Pad,  2mm x 4mm")
 		(tags "MeasurementPoint Square SMDPad 2mmx4mm ")
@@
 	(footprint "Connector_Wire:SolderWirePad_1x01_SMD_2x4mm"
 		(layer "F.Cu")
-		(at 144.301756 116.72849)
+		(at 144.383803 118.5)
 		(descr "Wire Pad, Square, SMD Pad,  2mm x 4mm")
 		(tags "MeasurementPoint Square SMDPad 2mmx4mm ")
@@
 	(footprint "Connector_PinHeader_2.54mm:PinHeader_1x03_P2.54mm_Vertical"
 		(layer "F.Cu")
-		(at 151 112.505798 180)
+		(at 150.986915 113.727771 180)
 		(descr "Through hole straight pin header, 1x03, 2.54mm pitch, single row")
 		(tags "Through hole pin header THT 1x03 2.54mm single row")
@@
 	)
 	(gr_line
-		(start 139.532766 114)
+		(start 139.532766 115.5)
 		(end 139.5 106)
 		(stroke
@@
 	)
 	(gr_line
-		(start 142.042403 114)
-		(end 139.532766 114)
+		(start 142.042403 115.5)
+		(end 139.532766 115.5)
 		(stroke
 			(width 0.2)
@@
 	)
 	(gr_line
-		(start 142.042403 120)
-		(end 142.042403 114)
+		(start 142.042403 122)
+		(end 142.042403 115.5)
 		(stroke
 			(width 0.2)
@@
 	)
 	(gr_line
-		(start 142.042403 120)
-		(end 150.3 120)
+		(start 142.042403 122)
+		(end 150.3 122)
 		(stroke
 			(width 0.2)
@@
 	)
 	(gr_line
-		(start 150.3 120)
-		(end 150.3 114.055781)
+		(start 150.3 122)
+		(end 150.3 115.5)
 		(stroke
 			(width 0.2)
@@
 	)
 	(gr_line
-		(start 152.767543 114.055781)
-		(end 150.29937 114.055781)
+		(start 152.767543 115.5)
+		(end 150.3 115.5)
 		(stroke
 			(width 0.2)
@@
 	)
 	(gr_line
-		(start 152.767543 114.055781)
+		(start 152.767543 115.5)
 		(end 152.75 106)
 		(stroke
@@
 		)
 	)
-	(gr_text "+"
-		(at 143.757336 119.773223 0)
-		(layer "F.SilkS")
-		(effects
-			(font
-				(size 0.8 0.8)
-				(thickness 0.15)
-			)
-			(justify left bottom)
-		)
-	)
 	(gr_text "GD"
 		(at 144.758158 72.615837 0)
@@
 		)
 	)
-	(gr_text "-"
-		(at 147.744911 120 0)
-		(layer "F.SilkS")
-		(effects
-			(font
-				(size 0.8 0.8)
-				(thickness 0.15)
-			)
-			(justify left bottom)
-		)
-	)
-	(gr_text "VB"
-		(at 148.365342 67.661203 0)
+	(gr_text "GD"
+		(at 148.148656 112.139166 0)
 		(layer "F.SilkS")
 		(effects
@@
 		)
 	)
-	(gr_text "GD"
-		(at 148.46503 110.54203 0)
+	(gr_text "5V"
+		(at 148.202235 114.64617 0)
 		(layer "F.SilkS")
 		(effects
@@
 	)
 	(gr_text "VB"
-		(at 148.561447 108.146878 0)
+		(at 148.220804 109.545928 0)
 		(layer "F.SilkS")
 		(effects
@@
 		)
 	)
-	(gr_text "5V"
-		(at 148.577235 113.331137 0)
+	(gr_text "VB"
+		(at 148.365342 67.661203 0)
 		(layer "F.SilkS")
 		(effects
@@
 		)
 	)
+	(gr_text "+"
+		(at 143.457116 121.755736 0)
+		(layer "F.SilkS")
+		(effects
+			(font
+				(size 1.2 1.2)
+				(thickness 0.15)
+			)
+			(justify left bottom)
+		)
+	)
+	(gr_text "-"
+		(at 147.320475 121.721847 0)
+		(layer "F.SilkS")
+		(effects
+			(font
+				(size 1.2 1.2)
+				(thickness 0.15)
+			)
+			(justify left bottom)
+		)
+	)
 	(gr_text "USB"
 		(at 163.464881 87.074287 270)
@@
 	)
 	(gr_text "REG"
-		(at 141.258507 111.182177 0)
+		(at 141.23086 112.377552 0)
 		(layer "F.SilkS")
 		(effects
@@
 	)
 	(segment
-		(start 161.754921 95.925425)
-		(end 161.754921 100.647182)
+		(start 151 108.92)
+		(end 146.302682 108.92)
 		(width 1)
 		(layer "F.Cu")
@@
 	)
 	(segment
-		(start 147.796884 107.425798)
-		(end 144.301756 110.920926)
+		(start 161.754921 95.925425)
+		(end 161.754921 100.647182)
 		(width 1)
 		(layer "F.Cu")
@@
 	)
 	(segment
-		(start 147.796884 107.425798)
-		(end 151 107.425798)
+		(start 146.302682 108.92)
+		(end 144.301756 110.920926)
 		(width 1)
 		(layer "F.Cu")
@@
 	)
 	(segment
+		(start 149.716284 111.46)
+		(end 151 111.46)
+		(width 1)
+		(layer "F.Cu")
+		(net "/GND")
+	)
+	(segment
 		(start 147.507675 72.190022)
 		(end 147.507675 73.147176)
@@
 	)
 	(segment
-		(start 128.50052 99.55082)
-		(end 131.17634 96.875)
+		(start 148.202235 112.974049)
+		(end 149.716284 111.46)
 		(width 1)
 		(layer "F.Cu")
@@
 	)
 	(segment
-		(start 132.202409 67.859972)
-		(end 135.85 71.507563)
-		(width 0.4)
-		(layer "F.Cu")
-		(net "/GND")
-	)
-	(segment
-		(start 148.202235 110.299052)
-		(end 148.202235 116.560375)
+		(start 128.50052 99.55082)
+		(end 131.17634 96.875)
 		(width 1)
 		(layer "F.Cu")
@@
 	)
 	(segment
-		(start 148.535489 109.965798)
-		(end 148.202235 110.299052)
-		(width 1)
+		(start 132.202409 67.859972)
+		(end 135.85 71.507563)
+		(width 0.4)
 		(layer "F.Cu")
 		(net "/GND")
@@
 	)
 	(segment
-		(start 148.535489 109.965798)
-		(end 151 109.965798)
-		(width 1)
-		(layer "F.Cu")
-		(net "/GND")
-	)
-	(segment
 		(start 152.07241 97.123203)
 		(end 152.07241 97.072327)
@@
 	)
 	(segment
+		(start 148.202235 112.974049)
+		(end 148.202235 116.560375)
+		(width 1)
+		(layer "F.Cu")
+		(net "/GND")
+	)
+	(segment
 		(start 163.585732 72.215135)
 		(end 161.925 73.875868)
@@
 	)
 	(segment
-		(start 148.57057 105.755565)
-		(end 149.264693 105.061442)
+		(start 148.57057 111.57057)
+		(end 151 114)
 		(width 0.4)
 		(layer "B.Cu")
@@
 	)
 	(segment
-		(start 148.57057 110.076368)
-		(end 148.57057 105.755565)
+		(start 148.57057 105.755565)
+		(end 148.57057 111.57057)
 		(width 0.4)
 		(layer "B.Cu")
@@
 	)
 	(segment
-		(start 149.264693 105.061442)
-		(end 154.622453 105.061442)
+		(start 148.57057 105.755565)
+		(end 149.264693 105.061442)
 		(width 0.4)
 		(layer "B.Cu")
@@
 	)
 	(segment
-		(start 151 112.505798)
-		(end 148.57057 110.076368)
+		(start 149.264693 105.061442)
+		(end 154.622453 105.061442)
 		(width 0.4)
 		(layer "B.Cu")
@@
 			(pts
 				(xy 136.874564 64.918718) (xy 155.996967 64.980008) (xy 160.716278 65.838064) (xy 166.538805 71.599301)
-				(xy 166.232356 99.42485) (xy 160.22596 105.247376) (xy 151.956672 120.588417) (xy 141.628882 120.690169)
+				(xy 166.232356 99.42485) (xy 160.22596 105.247376) (xy 154.942146 124.410002) (xy 139.132873 124.308335)
 				(xy 132.093963 105.431246) (xy 126.577885 99.547429) (xy 125.903698 95.502305) (xy 126.577885 71.292853)
 				(xy 132.058903 65.520769) (xy 136.933835 64.931581)
