File: kicad/fc/1s/main.kicad_pcb (KiCad board)
At the start: 2 copper layers, 40.2 x 57.1 mm, 36 parts, among them J1 Conn_01x14, J10 Conn_01x01_Pin, J11 Conn_01x01_Pin, J12 Conn_01x01_Pin, J13 Conn_01x01_Pin, J14 Conn_01x01_Pin, J15 Conn_01x03_Socket, J16 Conn_01x03_Socket, J17 Conn_01x01_Pin, J18 Conn_01x01_Pin, J19 Conn_01x01_Pin, J2 Conn_01x14_Socket, J20 Conn_01x01_Pin, J21 Conn_01x01_Pin, J22 Conn_01x01_Pin, J23 Conn_01x03_Socket, J24 Conn_01x03_Socket, J25 Conn_01x01_Pin, J26 Conn_01x01_Pin, J27 Conn_01x04_Socket, J3 Conn_01x01_Pin, J4 Conn_01x03_Socket, J5 Conn_01x01_Pin, J6 Conn_01x04_Socket, J7 Conn_01x01_Pin, J8 Conn_01x01_Pin, J9 Conn_01x01_Pin

Commit message: modified:   kicad/fc/1s/main.kicad_pcb
Parts:
- moved J27 1.00 mm to (158.0, 82.8)
- moved J6 1.00 mm to (134.0, 82.8)
Routing:
- net /MOSI: track 7.50 -> 8.67 mm
- net /MISO: track 21.7 -> 22.9 mm
- net /SCL1: track 26.5 -> 25.6 mm
- net /CS: track 4.17 -> 5.08 mm
- net /3V3: track 26.0 -> 25.2 mm
- net /GND: track 148.5 -> 147.7 mm
- net /SDA1: track 23.3 -> 22.7 mm
- net /M3: track 29.3 -> 28.7 mm
Changed lines of the file:
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@@
 	(footprint "Connector_PinHeader_2.54mm:PinHeader_1x04_P2.54mm_Vertical"
 		(layer "F.Cu")
-		(at 134 81.8)
+		(at 134 82.8)
 		(descr "Through hole straight pin header, 1x04, 2.54mm pitch, single row")
 		(tags "Through hole pin header THT 1x04 2.54mm single row")
@@
 	(footprint "Connector_PinHeader_2.54mm:PinHeader_1x04_P2.54mm_Vertical"
 		(layer "F.Cu")
-		(at 158 81.8)
+		(at 158 82.8)
 		(descr "Through hole straight pin header, 1x04, 2.54mm pitch, single row")
 		(tags "Through hole pin header THT 1x04 2.54mm single row")
@@
 	)
 	(gr_text "SCK"
-		(at 130.529453 89.959262 0)
+		(at 130.436635 90.989539 0)
 		(layer "F.SilkS")
 		(effects
@@
 	)
 	(gr_text "CS"
-		(at 131 82.22939 0)
+		(at 130.907182 83.259667 0)
 		(layer "F.SilkS")
 		(effects
@@
 	)
 	(gr_text "SO"
-		(at 131 87.316971 0)
+		(at 130.907182 88.347248 0)
 		(layer "F.SilkS")
 		(effects
@@
 	)
 	(gr_text "SI"
-		(at 131.5 84.747743 0)
+		(at 131.407182 85.77802 0)
 		(layer "F.SilkS")
 		(effects
@@
 	)
 	(gr_text "GD"
-		(at 135 84.21 0)
+		(at 137.1 73.9 0)
 		(layer "F.SilkS")
 		(effects
@@
 		)
 	)
-	(gr_text "GD"
-		(at 137.1 73.9 0)
+	(gr_text "M3"
+		(at 138.119148 79.9 0)
 		(layer "F.SilkS")
 		(effects
@@
 		)
 	)
-	(gr_text "M3"
-		(at 138.119148 79.9 0)
+	(gr_text "GD"
+		(at 139.299014 84.275543 0)
 		(layer "F.SilkS")
 		(effects
@@
 		)
 	)
-	(gr_text "CL1"
-		(at 159 82.320269 0)
+	(gr_text "DA1"
+		(at 158.895591 85.726697 0)
 		(layer "F.SilkS")
 		(effects
@@
 		)
 	)
-	(gr_text "DA1"
-		(at 159 84.906961 0)
+	(gr_text "CL1"
+		(at 159.098479 83.323259 0)
 		(layer "F.SilkS")
 		(effects
@@
 	)
 	(gr_text "GD"
-		(at 159 87.444848 0)
+		(at 159.108883 88.57406 0)
 		(layer "F.SilkS")
 		(effects
@@
 	)
 	(gr_text "3V3"
-		(at 159 89.937544 0)
+		(at 159.176513 91.157843 0)
 		(layer "F.SilkS")
 		(effects
@@
 	)
 	(gr_text "BMI088"
-		(at 139.619108 85.899108 0)
+		(at 139.634352 87.363767 0)
 		(layer "F.SilkS")
 		(effects
@@
 	)
 	(gr_text "SO"
-		(at 132.827834 87.350641 0)
+		(at 132.735016 88.380918 0)
 		(layer "B.SilkS")
 		(effects
@@
 	)
 	(gr_text "SCK"
-		(at 132.847115 89.924679 0)
+		(at 132.754297 90.954956 0)
 		(layer "B.SilkS")
 		(effects
@@
 	)
 	(gr_text "SI"
-		(at 132.93388 84.766961 0)
+		(at 132.841062 85.797238 0)
 		(layer "B.SilkS")
 		(effects
@@
 	)
 	(gr_text "CS"
-		(at 132.943521 82.279688 0)
+		(at 132.850703 83.309965 0)
 		(layer "B.SilkS")
 		(effects
@@
 	)
 	(gr_text "GD"
-		(at 160.855049 87.401254 0)
+		(at 160.816955 88.626084 0)
 		(layer "B.SilkS")
 		(effects
@@
 	)
 	(gr_text "DA1"
-		(at 161.158728 84.863367 0)
+		(at 161.205389 85.804731 0)
 		(layer "B.SilkS")
 		(effects
@@
 	)
 	(gr_text "CL1"
-		(at 161.245493 82.30379 0)
+		(at 161.43949 83.245225 0)
 		(layer "B.SilkS")
 		(effects
@@
 	)
 	(gr_text "3V3"
-		(at 161.375641 89.982523 0)
+		(at 161.495848 91.107556 0)
 		(layer "B.SilkS")
 		(effects
@@
 	)
 	(segment
-		(start 157.738542 89.42)
-		(end 156.845 90.313542)
+		(start 150.65 81.25)
+		(end 152.63 81.25)
 		(width 0.4)
 		(layer "F.Cu")
@@
 	)
 	(segment
-		(start 150.65 81.25)
-		(end 152.63 81.25)
+		(start 156.845 91.575)
+		(end 158 90.42)
 		(width 0.4)
 		(layer "F.Cu")
@@
 	)
 	(segment
-		(start 156.845 90.313542)
-		(end 156.845 92.725)
+		(start 156.845 92.725)
+		(end 156.845 91.575)
 		(width 0.4)
 		(layer "F.Cu")
@@
 	)
 	(segment
-		(start 160.235 91.875)
-		(end 159.385 92.725)
-		(width 0.4)
-		(layer "F.Cu")
-		(net "/GND")
-	)
-	(segment
 		(start 139.7 100.724827)
 		(end 139.7 102.4)
@@
 	)
 	(segment
-		(start 135.85 73.4)
-		(end 147.760499 73.4)
-		(width 0.4)
+		(start 160.235 91.875)
+		(end 160.235 90.115)
+		(width 1)
 		(layer "F.Cu")
 		(net "/GND")
 	)
 	(segment
-		(start 158.5 86.88)
-		(end 160.235 88.615)
+		(start 135.85 73.4)
+		(end 147.760499 73.4)
 		(width 0.4)
 		(layer "F.Cu")
@@
 	)
 	(segment
-		(start 136.013598 96.875)
-		(end 139.7 100.561402)
+		(start 160.235 90.115)
+		(end 158 87.88)
 		(width 1)
 		(layer "F.Cu")
@@
 	)
 	(segment
-		(start 160.235 88.615)
+		(start 159.385 92.725)
 		(end 160.235 91.875)
-		(width 0.4)
+		(width 1)
+		(layer "F.Cu")
+		(net "/GND")
+	)
+	(segment
+		(start 136.013598 96.875)
+		(end 139.7 100.561402)
+		(width 1)
 		(layer "F.Cu")
 		(net "/GND")
@@
 	)
 	(segment
+		(start 134 81.464992)
+		(end 134 82.8)
+		(width 0.2)
+		(layer "F.Cu")
+		(net "/CS")
+	)
+	(segment
 		(start 133.985 81.449992)
-		(end 133.671685 81.763307)
+		(end 134 81.464992)
 		(width 0.2)
 		(layer "F.Cu")
@@
 	)
 	(segment
-		(start 131.445 82.076622)
-		(end 133.671685 84.303307)
+		(start 131.445 82.785)
+		(end 134 85.34)
 		(width 0.2)
 		(layer "F.Cu")
@@
 	(segment
 		(start 131.445 77.725)
-		(end 131.445 82.076622)
+		(end 131.445 82.785)
 		(width 0.2)
 		(layer "F.Cu")
@@
 	)
 	(segment
-		(start 128.905 82.076622)
-		(end 133.671685 86.843307)
+		(start 128.905 77.725)
+		(end 128.905 82.785)
 		(width 0.2)
 		(layer "F.Cu")
@@
 	)
 	(segment
-		(start 128.905 77.725)
-		(end 128.905 82.076622)
+		(start 128.905 82.785)
+		(end 134 87.88)
 		(width 0.2)
 		(layer "F.Cu")
@@
 	)
 	(segment
-		(start 132.246693 89.383307)
-		(end 133.671685 89.383307)
+		(start 128.905 92.725)
+		(end 131.21 90.42)
 		(width 0.2)
 		(layer "F.Cu")
@@
 	)
 	(segment
-		(start 128.905 92.725)
-		(end 132.246693 89.383307)
+		(start 131.21 90.42)
+		(end 134 90.42)
 		(width 0.2)
 		(layer "F.Cu")
@@
 	)
 	(segment
-		(start 153.584206 87.915794)
+		(start 154.29 79.366346)
 		(end 154.29 87.21)
 		(width 0.2)
@@
 	)
 	(segment
-		(start 154.29 87.21)
-		(end 154.29 79.366346)
+		(start 153.584206 87.915794)
+		(end 154.29 87.21)
 		(width 0.2)
 		(layer "F.Cu")
@@
 	)
 	(segment
-		(start 134.467727 91.105813)
-		(end 132.835276 91.105813)
+		(start 135.375 92.961346)
+		(end 133.198227 95.138119)
+		(width 0.2)
+		(layer "F.Cu")
+		(net "/M3")
+	)
+	(segment
+		(start 136.7 88.677077)
+		(end 136.7 88.87354)
 		(width 0.2)
 		(layer "F.Cu")
@@
 	)
 	(segment
-		(start 136.7 80.09)
-		(end 136.7 88.87354)
+		(start 135.375 90.002077)
+		(end 135.375 92.961346)
 		(width 0.2)
 		(layer "F.Cu")
@@
 	)
 	(segment
-		(start 132.835 91.105537)
+		(start 133.198227 95.138119)
 		(end 132.835 95.138119)
 		(width 0.2)
@@
 	)
 	(segment
-		(start 132.835276 91.105813)
-		(end 132.835 91.105537)
+		(start 136.7 80.09)
+		(end 136.7 88.677077)
 		(width 0.2)
 		(layer "F.Cu")
@@
 	)
 	(segment
-		(start 136.7 88.87354)
-		(end 134.467727 91.105813)
+		(start 136.7 88.677077)
+		(end 135.375 90.002077)
 		(width 0.2)
 		(layer "F.Cu")
@@
 	(segment
 		(start 136.525 92.725)
-		(end 147.45 81.8)
+		(end 146.45 82.8)
 		(width 0.2)
 		(layer "B.Cu")
@@
 	)
 	(segment
-		(start 147.45 81.8)
-		(end 158.5 81.8)
+		(start 146.45 82.8)
+		(end 158 82.8)
 		(width 0.2)
 		(layer "B.Cu")
@@
 	)
 	(segment
-		(start 146.711471 84.34)
-		(end 139.065 91.986471)
+		(start 145.247919 85.34)
+		(end 158 85.34)
 		(width 0.2)
 		(layer "B.Cu")
@@
 	)
 	(segment
-		(start 158.5 84.34)
-		(end 146.711471 84.34)
+		(start 139.065 92.725)
+		(end 139.065 91.522919)
 		(width 0.2)
 		(layer "B.Cu")
@@
 	)
 	(segment
-		(start 139.065 91.986471)
-		(end 139.065 92.725)
+		(start 139.065 91.522919)
+		(end 145.247919 85.34)
 		(width 0.2)
 		(layer "B.Cu")

Commit message: modified:   kicad/fc/1s/main.kicad_pcb
Parts:
- moved J4 30.6 mm to (155.2, 83.5), turned to 0 degrees
- moved J25 9.47 mm to (148.3, 109.0)
- moved J26 9.47 mm to (144.5, 109.0)
Routing:
- net /GND: track 147.7 -> 170.3 mm, vias 4 -> 7
- net /VBAT: track 147.7 -> 135.0 mm
- net /5V: track 39.1 -> 47.2 mm
Other:
- board size 40.2 x 57.1 mm -> 40.2 x 48.1 mm

Commit message: modified:   kicad/fc/1s/main.kicad_pcb
Routing:
- net /GND: track 170.3 -> 166.9 mm
Changed lines of the file:
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@@
 		(sheetname "/")
 		(sheetfile "main.kicad_sch")
-		(units
-			(unit
-				(name "A")
-				(pins "1")
-			)
-		)
 		(duplicate_pad_numbers_are_jumpers no)
 		(fp_rect
@@
 		)
 		(pad "1" smd roundrect
-			(at 0 -0.032447)
-			(size 2 4)
+			(at 0.669864 0.468448)
+			(size 3 5)
 			(layers "F.Cu" "F.Mask")
 			(roundrect_rratio 0.25)
@@
 		(sheetname "/")
 		(sheetfile "main.kicad_sch")
-		(units
-			(unit
-				(name "A")
-				(pins "1")
-			)
-		)
 		(duplicate_pad_numbers_are_jumpers no)
 		(fp_rect
@@
 		)
 		(pad "1" smd roundrect
-			(at 0 0)
-			(size 2 4)
+			(at -0.466777 0.468448)
+			(size 3 5)
 			(layers "F.Cu" "F.Mask")
 			(roundrect_rratio 0.25)
@@
 	)
 	(gr_text "+"
-		(at 143.621402 106.64942 0)
+		(at 142.97414 106.839626 0)
 		(layer "F.SilkS")
 		(effects
 			(font
-				(size 1.2 1.2)
+				(size 1.5 1.5)
 				(thickness 0.15)
 			)
@@
 	)
 	(gr_text "-"
-		(at 147.788403 106.727454 0)
+		(at 147.808469 106.997482 0)
 		(layer "F.SilkS")
 		(effects
 			(font
-				(size 1.2 1.2)
+				(size 1.5 1.5)
 				(thickness 0.15)
 			)
@@
 	)
 	(segment
-		(start 141.829953 106.394728)
-		(end 144.466777 109.031552)
+		(start 162.187959 101.08022)
+		(end 161.754921 100.647182)
 		(width 1)
 		(layer "F.Cu")
@@
 	)
 	(segment
-		(start 162.187959 101.08022)
-		(end 161.754921 100.647182)
+		(start 164.549109 93.131237)
+		(end 161.754921 95.925425)
 		(width 1)
 		(layer "F.Cu")
@@
 	)
 	(segment
-		(start 164.549109 93.131237)
-		(end 161.754921 95.925425)
+		(start 141.829953 106.106927)
+		(end 141.829953 107.329953)
 		(width 1)
 		(layer "F.Cu")
@@
 	)
 	(segment
-		(start 141.829953 106.106927)
-		(end 141.829953 106.394728)
+		(start 141.829953 107.329953)
+		(end 144 109.5)
 		(width 1)
 		(layer "F.Cu")
@@
 	)
 	(segment
-		(start 150.727569 108.999105)
-		(end 150.757166 109.028702)
-		(width 1)
-		(layer "F.Cu")
-		(net "/GND")
-	)
-	(segment
 		(start 147.507675 72.190022)
 		(end 147.507675 73.147176)
@@
 	)
 	(segment
-		(start 148.330136 108.999105)
-		(end 150.727569 108.999105)
-		(width 1)
-		(layer "F.Cu")
-		(net "/GND")
-	)
-	(segment
 		(start 163.585732 72.215135)
 		(end 161.925 73.875868)
@@
 	)
 	(via
-		(at 150.757166 109.028702)
+		(at 153.668066 79.76)
 		(size 0.5)
 		(drill 0.3)
@@
 	)
 	(via
-		(at 153.668066 79.76)
+		(at 153.397256 87.599528)
 		(size 0.5)
 		(drill 0.3)
@@
 	)
 	(via
-		(at 153.397256 87.599528)
-		(size 0.5)
+		(at 159.385 96.684794)
+		(size 0.6)
 		(drill 0.3)
 		(layers "F.Cu" "B.Cu")
@@
 	)
 	(via
-		(at 159.385 96.684794)
+		(at 148.893726 109.010141)
 		(size 0.6)
 		(drill 0.3)
@@
 	)
 	(segment
-		(start 150.429493 109.028702)
-		(end 147.57057 106.169779)
-		(width 1)
-		(layer "B.Cu")
-		(net "/GND")
-	)
-	(segment
 		(start 150.461186 96.875)
 		(end 154.390639 96.875)
@@
 	)
 	(segment
-		(start 147.57057 106.169779)
+		(start 150.461186 101.707241)
 		(end 147.57057 104.597857)
 		(width 1)
@@
 	)
 	(segment
+		(start 147.57057 104.597857)
+		(end 147.57057 107.686985)
+		(width 1)
+		(layer "B.Cu")
+		(net "/GND")
+	)
+	(segment
 		(start 162.575 78.375)
 		(end 161.925 77.725)
@@
 	)
 	(segment
+		(start 150.461186 96.875)
+		(end 150.461186 101.707241)
+		(width 1)
+		(layer "B.Cu")
+		(net "/GND")
+	)
+	(segment
 		(start 150.02 79.76)
 		(end 153.668066 79.76)
@@
 	)
 	(segment
-		(start 150.757166 109.028702)
-		(end 150.429493 109.028702)
-		(width 1)
-		(layer "B.Cu")
-		(net "/GND")
-	)
-	(segment
 		(start 162.24 79.76)
 		(end 162.575 79.425)
@@
 	)
 	(segment
-		(start 147.57057 104.597857)
-		(end 150.461186 101.707241)
-		(width 1)
-		(layer "B.Cu")
-		(net "/GND")
-	)
-	(segment
 		(start 153.668066 79.76)
 		(end 162.24 79.76)
@@
 	)
 	(segment
-		(start 150.461186 101.707241)
+		(start 136.013598 96.875)
 		(end 150.461186 96.875)
 		(width 1)
@@
 	)
 	(segment
-		(start 136.013598 96.875)
-		(end 150.461186 96.875)
+		(start 147.57057 107.686985)
+		(end 148.893726 109.010141)
 		(width 1)
 		(layer "B.Cu")
