File: kicad/hover/1s/main.kicad_sch (KiCad schematic)
At the start: 5 parts, among them J27 Conn_02x04_Odd_Even

Commit message: modified:   kicad/hover/1s/main.kicad_pcb
Parts:
- removed H1, H2, H3, H4: MountingHole, MountingHole:MountingHole_2.5mm, symbol Mechanical:MountingHole
- removed J27: Conn_02x04_Odd_Even, Connector_PinHeader_2.54mm:PinHeader_2x04_P2.54mm_Vertical, symbol Connector_Generic:Conn_02x04_Odd_Even
- added J1: Conn_01x02_Socket, Connector_PinHeader_2.54mm:PinHeader_1x02_P2.54mm_Vertical, symbol Connector:Conn_01x02_Socket
- added J27, J28, J6, J7, J8: Conn_01x04_Socket, Connector_PinHeader_2.54mm:PinHeader_1x04_P2.54mm_Vertical, symbol Connector:Conn_01x04_Socket
Connections:
- net 3V3: now also J1.2 (Pin_2), J27.4 (Pin_4), J28.4 (Pin_4)
- net CS: now also J6.1 (Pin_1), J7.3 (Pin_3)
- net GND: now also J1.1 (Pin_1), J27.3 (Pin_3), J28.3 (Pin_3)
- net MISO: now also J6.3 (Pin_3), J7.1 (Pin_1)
- net MOSI: now also J6.2 (Pin_2), J7.2 (Pin_2)
- net SCK: now also J6.4 (Pin_4), J8.1 (Pin_1)
- new net SCL: J27.1 (Pin_1), J28.1 (Pin_1)
- new net SDA: J27.2 (Pin_2), J28.2 (Pin_2)
